File: azimuth_sheet.kicad_sch (KiCad schematic)
At the start: 6 parts, among them U4 74LS32, U5 ICM7555xP

Commit message: Elevation sheet mostly complete
Parts:
- removed C7: 10nF, symbol Device:C
- removed C8: 100nF, symbol Device:C
- removed R6: 820, symbol Device:R
- removed R8: 6.8k, symbol Device:R
- removed U4: 74LS32, symbol 74xx:74LS32
- removed U5: ICM7555xP, Package_DIP:DIP-8_W7.62mm, symbol Timer:ICM7555xP
Other:
- note removed: "Motor 2 Pulse Generation"

Commit message: Added Azimuth
Parts:
- added C6: 10nF, symbol Device:C
- added C7: 100nF, symbol Device:C
- added J3: DA15_Socket, Connector_Dsub:DSUB-15_Socket_Horizontal_P2.77x2.54mm_EdgePinOffset9.40mm, symbol Connector:DA15_Socket
- added Q3, Q4: PZT2222A, Package_TO_SOT_SMD:SOT-223-3_TabPin2, symbol Transistor_BJT:PZT2222A
- added R14, R15, R16, R17, R7, R8: 10k, symbol Device:R
- added R18: 820, symbol Device:R
- added R19: 6.8k, symbol Device:R
- added R9: 1k, symbol Device:R
- added SW3: SW_SPDT_312, symbol Switch:SW_SPDT_312
- added U2: 74LS08, symbol 74xx:74LS08
- added U3: 74LS32, symbol 74xx:74LS32
- added U5: ICM7555xP, Package_DIP:DIP-8_W7.62mm, symbol Timer:ICM7555xP
Connections:
- new net: R16.1, U2.8, U3.4
- new net: R17.1, U2.11, U3.5
- new net: U3.6, U5.4 (R)
- new net: R18.2, R19.2, U5.7 (DIS)
- new net: C7.1, R19.1, U5.2 (TR), U5.6 (THR)
- new net: Q4.1 (B), U5.3 (Q)
- new net: C6.1, U5.5 (CV)
- new net: R15.1, R8.1, SW3.2 (C), U2.13
- new net: Q3.1 (B), R9.2
- new net +5V: J3.5, J3.8, R18.1, SW3.1 (B), U5.8 (VCC)
- new net Dir: J3.9 (P9), Q3.2 (C)
- new net Dir Sig: R7.1, R9.1, SW3.3 (A), U2.10
- new net GND: C6.2, C7.2, J3.1, J3.15 (P15), Q3.3 (E), Q4.3 (E), R14.2, R15.2, R16.2, R17.2, R7.2, R8.2, U5.1 (GND)
- new net Limit Sw1: J3.10 (P10), R14.1, U2.9
- new net Limit Sw2: J3.3, U2.12
- new net Pul: J3.2, Q4.2 (C)
- no-connect marks 0 -> 7
Other:
- note added: "Azimuth Motor Pulse Generation"
- note added: "Azimuth Motor SPDT on-off-on switch Pulse enable and direction"
- note added: "Direction Signal Conditioning Provides 5V to Dir"
- note added: "N.C."
- note added: "Power"

Commit message: Latest versions
Parts:
- added J4: CRJ022-G-TH, CRJ022-G-TH:CUI_CRJ022-G-TH, symbol CRJ022-G-TH:CRJ022-G-TH
Changed lines of the file:
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@@
+	)
+	(symbol
+		(lib_id "CRJ022-G-TH:CRJ022-G-TH")
+		(at 271.78 113.03 0)
+		(unit 2)
+		(exclude_from_sim no)
+		(in_bom yes)
+		(on_board yes)
+		(dnp no)
+		(fields_autoplaced yes)
+		(property "Reference" "J4"
+			(at 280.67 113.0299 0)
+			(effects
+				(font
+					(size 1.27 1.27)
+				)
+				(justify left)
+			)
+		)
+		(property "Value" "CRJ022-G-TH"
+			(at 280.67 115.5699 0)
+			(effects
+				(font
+					(size 1.27 1.27)
+				)
+				(justify left)
+			)
+		)
+		(property "Footprint" "CRJ022-G-TH:CUI_CRJ022-G-TH"
+			(at 271.78 113.03 0)
+			(effects
+				(font
+					(size 1.27 1.27)
+				)
+				(justify bottom)
+				(hide yes)
+			)
+		)
+		(property "Datasheet" ""
+			(at 271.78 113.03 0)
+			(effects
+				(font
+					(size 1.27 1.27)
+				)
+				(hide yes)
+			)
+		)
+		(property "Description" ""
+			(at 271.78 113.03 0)
+			(effects
+				(font
+					(size 1.27 1.27)
+				)
+				(hide yes)
+			)
+		)
+		(property "PARTREV" "1.0"
+			(at 271.78 113.03 0)
+			(effects
+				(font
+					(size 1.27 1.27)
+				)
+				(justify bottom)
+				(hide yes)
+			)
+		)
+		(property "STANDARD" "Manufacturer Recommendations"
+			(at 271.78 113.03 0)
+			(effects
+				(font
+					(size 1.27 1.27)
+				)
+				(justify bottom)
+				(hide yes)
+			)
+		)
+		(property "MAXIMUM_PACKAGE_HEIGHT" "14.05mm"
+			(at 271.78 113.03 0)
+			(effects
+				(font
+					(size 1.27 1.27)
+				)
+				(justify bottom)
+				(hide yes)
+			)
+		)
+		(property "MANUFACTURER" "CUI Devices"
+			(at 271.78 113.03 0)
+			(effects
+				(font
+					(size 1.27 1.27)
+				)
+				(justify bottom)
+				(hide yes)
+			)
+		)
+		(pin "6R"
+		)
+		(pin "8R"
+		)
+		(pin "7R"
+		)
+		(pin "7L"
+		)
+		(pin "3L"
+		)
+		(pin "1R"
+		)
+		(pin "4R"
+		)
+		(pin "1L"
+		)
+		(pin "5L"
+		)
+		(pin "6L"
+		)
+		(pin "2R"
+		)
+		(pin "5R"
+		)
+		(pin "2L"
+		)
+		(pin "S1"
+		)
+		(pin "4L"
+		)
+		(pin "S2"
+		)
+		(pin "S3"
+		)
+		(pin "3R"
+		)
+		(pin "8L"
+		)
+		(instances
+			(project "simple_dish_manual_controller"
+				(path "/8648ccd3-30ce-4b98-baff-aeab56a7c9f5/809ce83c-7739-411d-92b7-06d9bcd34d12"
+					(reference "J4")
+					(unit 2)
+				)
+			)
+		)
 	)
 	(symbol
