File: Simple_Dish_Controller/azimuth_sheet.kicad_sch (KiCad schematic)
At the start: 19 parts, among them J6 Conn_01x03_Pin, J7 Azimuth DE-15, Q3 MMBT2222A, Q4 MMBT2222A, U2 74LS32, U3 74LS08, U5 NE555D

Commit message: Final version of the PCB.Production files were generated in -Production- folder
Parts:
- C10: LCSC Part (none) -> C13585
- C8: value 0.1uF -> 100nF; LCSC Part (none) -> C24497
- C9: LCSC Part (none) -> C24497
- Q3, Q4: LCSC Part (none) -> C8512
- R11: LCSC Part (none) -> C17984
- R12, R13, R15, R16, R17, R18: LCSC Part (none) -> C17902
- R14: LCSC Part (none) -> C2907522
- R19: LCSC Part (none) -> C4410
- U2: LCSC Part (none) -> C116812
- U3: LCSC Part (none) -> C6802
- U5: LCSC Part (none) -> C234230
Changed lines of the file:
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@@
 			)
 		)
-		(property "LCSC Part" ""
+		(property "LCSC Part" "C4410"
 			(at 55.88 142.24 0)
 			(effects
@@
 					(size 1.27 1.27)
 				)
+				(hide yes)
 			)
 		)
@@
 			)
 		)
-		(property "LCSC Part" ""
+		(property "LCSC Part" "C2907522"
 			(at 193.04 73.66 0)
 			(effects
@@
 					(size 1.27 1.27)
 				)
+				(hide yes)
 			)
 		)
@@
 			)
 		)
-		(property "LCSC Part" ""
+		(property "LCSC Part" "C6802"
 			(at 85.09 81.28 0)
 			(effects
@@
 					(size 1.27 1.27)
 				)
+				(hide yes)
 			)
 		)
@@
 			)
 		)
-		(property "Value" "0.1uF"
+		(property "Value" "100nF"
 			(at 163.83 54.6099 0)
 			(effects
@@
 			)
 		)
-		(property "LCSC Part" ""
+		(property "LCSC Part" "C24497"
 			(at 160.02 53.34 0)
 			(effects
@@
 					(size 1.27 1.27)
 				)
+				(hide yes)
 			)
 		)
@@
 			)
 		)
-		(property "LCSC Part" ""
+		(property "LCSC Part" "C116812"
 			(at 113.03 69.85 0)
 			(effects
@@
 					(size 1.27 1.27)
 				)
+				(hide yes)
 			)
 		)
@@
 			)
 		)
-		(property "LCSC Part" ""
+		(property "LCSC Part" "C6802"
 			(at 85.09 57.15 0)
 			(effects
@@
 					(size 1.27 1.27)
 				)
+				(hide yes)
 			)
 		)
@@
 			)
 		)
-		(property "LCSC Part" ""
+		(property "LCSC Part" "C17902"
 			(at 97.79 77.47 0)
 			(effects
@@
 					(size 1.27 1.27)
 				)
+				(hide yes)
 			)
 		)
@@
 			)
 		)
-		(property "LCSC Part" ""
+		(property "LCSC Part" "C8512"
 			(at 69.85 142.24 0)
 			(effects
@@
 					(size 1.27 1.27)
 				)
+				(hide yes)
 			)
 		)
@@
 			)
 		)
-		(property "LCSC Part" ""
+		(property "LCSC Part" "C13585"
 			(at 161.29 85.09 0)
 			(effects
@@
 					(size 1.27 1.27)
 				)
+				(hide yes)
 			)
 		)
@@
 			)
 		)
-		(property "LCSC Part" ""
+		(property "LCSC Part" "C8512"
 			(at 128.27 142.24 0)
 			(effects
@@
 					(size 1.27 1.27)
 				)
+				(hide yes)
 			)
 		)
@@
 			)
 		)
-		(property "LCSC Part" ""
+		(property "LCSC Part" "C17902"
 			(at 76.2 88.9 0)
 			(effects
@@
 					(size 1.27 1.27)
 				)
+				(hide yes)
 			)
 		)
@@
 			)
 		)
-		(property "LCSC Part" ""
+		(property "LCSC Part" "C17902"
 			(at 102.87 77.47 0)
 			(effects
@@
 					(size 1.27 1.27)
 				)
+				(hide yes)
 			)
 		)
@@
 			)
 		)
-		(property "LCSC Part" ""
+		(property "LCSC Part" "C24497"
 			(at 152.4 85.09 0)
 			(effects
@@
 					(size 1.27 1.27)
 				)
+				(hide yes)
 			)
 		)
@@
 			)
 		)
-		(property "LCSC Part" ""
+		(property "LCSC Part" "C17902"
 			(at 64.77 63.5 0)
 			(effects
@@
 					(size 1.27 1.27)
 				)
+				(hide yes)
 			)
 		)
@@
 			)
 		)
-		(property "LCSC Part" ""
+		(property "LCSC Part" "C17902"
 			(at 76.2 64.77 0)
 			(effects
@@
 					(size 1.27 1.27)
 				)
+				(hide yes)
 			)
 		)
@@
 			)
 		)
-		(property "LCSC Part" ""
+		(property "LCSC Part" "C17984"
 			(at 193.04 55.88 0)
 			(effects
@@
 					(size 1.27 1.27)
 				)
+				(hide yes)
 			)
 		)
@@
 			)
 		)
-		(property "LCSC Part" ""
+		(property "LCSC Part" "C17902"
 			(at 64.77 87.63 0)
 			(effects
@@
 					(size 1.27 1.27)
 				)
+				(hide yes)
 			)
 		)
@@
 			)
 		)
-		(property "LCSC Part" ""
+		(property "LCSC Part" "C234230"
 			(at 176.53 67.31 0)
 			(effects
@@
 					(size 1.27 1.27)
 				)
+				(hide yes)
 			)
 		)
