File: kicad/RS485.kicad_sch (KiCad schematic)
At the start: 50 parts, among them CN3 KF2EDGR-2.54-4P, CN4 KF2EDGR-2.54-4P, CN5 KF2EDGR-2.54-4P, U2 ISOW1432BDFMR, U3 ISOW1432BDFMR

Commit message: Updates to power
Parts:
- C20, C23, C28, C31, C32, C35, C40, C43: value 10uF -> GRM21BR6YA106KE43L
- C21, C24, C27, C30, C33, C36, C39, C42: value 1uF -> CL10A105KA8NNNC
- C22, C25, C26, C29: value 100nF -> CL05B104KO5NNNC
- C44, C45: value 10nF -> C43Q1103K40C80F
- L3, L4: value Choke -> SMW2012B371BTE
Changed lines of the file:
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@@
 			)
 		)
-		(property "Value" "100nF"
+		(property "Value" "CL05B104KO5NNNC"
 			(at 112.522 57.912 90)
 			(show_name no)
@@
 			)
 		)
-		(property "Value" "1uF"
+		(property "Value" "CL10A105KA8NNNC"
 			(at 258.318 58.166 90)
 			(show_name no)
@@
 			)
 		)
-		(property "Value" "10nF"
+		(property "Value" "C43Q1103K40C80F"
 			(at 119.634 135.3821 90)
 			(show_name no)
@@
 			)
 		)
-		(property "Value" "10uF"
+		(property "Value" "GRM21BR6YA106KE43L"
 			(at 32.258 52.324 0)
 			(show_name no)
@@
 			)
 		)
-		(property "Value" "10uF"
+		(property "Value" "GRM21BR6YA106KE43L"
 			(at 132.588 58.674 0)
 			(show_name no)
@@
 			)
 		)
-		(property "Value" "100nF"
+		(property "Value" "CL05B104KO5NNNC"
 			(at 50.292 51.562 90)
 			(show_name no)
@@
 			)
 		)
-		(property "Value" "1uF"
+		(property "Value" "CL10A105KA8NNNC"
 			(at 178.308 51.816 90)
 			(show_name no)
@@
 			)
 		)
-		(property "Value" "10uF"
+		(property "Value" "GRM21BR6YA106KE43L"
 			(at 168.148 52.324 0)
 			(show_name no)
@@
 			)
 		)
-		(property "Value" "Choke"
+		(property "Value" "SMW2012B371BTE"
 			(at 251.206 51.816 0)
 			(show_name no)
@@
 			)
 		)
-		(property "Value" "10uF"
+		(property "Value" "GRM21BR6YA106KE43L"
 			(at 180.848 72.644 0)
 			(show_name no)
@@
 			)
 		)
-		(property "Value" "10uF"
+		(property "Value" "GRM21BR6YA106KE43L"
 			(at 268.478 58.674 0)
 			(show_name no)
@@
 			)
 		)
-		(property "Value" "1uF"
+		(property "Value" "CL10A105KA8NNNC"
 			(at 42.418 51.816 90)
 			(show_name no)
@@
 			)
 		)
-		(property "Value" "1uF"
+		(property "Value" "CL10A105KA8NNNC"
 			(at 117.602 78.4859 90)
 			(show_name no)
@@
 			)
 		)
-		(property "Value" "10nF"
+		(property "Value" "C43Q1103K40C80F"
 			(at 143.51 135.8901 90)
 			(show_name no)
@@
 			)
 		)
-		(property "Value" "100nF"
+		(property "Value" "CL05B104KO5NNNC"
 			(at 186.182 51.562 90)
 			(show_name no)
@@
 			)
 		)
-		(property "Value" "Choke"
+		(property "Value" "SMW2012B371BTE"
 			(at 115.824 43.688 0)
 			(show_name no)
@@
 			)
 		)
-		(property "Value" "10uF"
+		(property "Value" "GRM21BR6YA106KE43L"
 			(at 262.128 78.994 0)
 			(show_name no)
@@
 			)
 		)
-		(property "Value" "1uF"
+		(property "Value" "CL10A105KA8NNNC"
 			(at 122.428 58.166 90)
 			(show_name no)
@@
 			)
 		)
-		(property "Value" "100nF"
+		(property "Value" "CL05B104KO5NNNC"
 			(at 248.412 57.912 90)
 			(show_name no)
@@
 			)
 		)
-		(property "Value" "1uF"
+		(property "Value" "CL10A105KA8NNNC"
 			(at 55.118 72.136 90)
 			(show_name no)
@@
 			)
 		)
-		(property "Value" "10uF"
+		(property "Value" "GRM21BR6YA106KE43L"
 			(at 44.958 72.644 0)
 			(show_name no)
@@
 			)
 		)
-		(property "Value" "1uF"
+		(property "Value" "CL10A105KA8NNNC"
 			(at 191.008 72.136 90)
 			(show_name no)
@@
 			)
 		)
-		(property "Value" "1uF"
+		(property "Value" "CL10A105KA8NNNC"
 			(at 253.492 78.4859 90)
 			(show_name no)
@@
 			)
 		)
-		(property "Value" "10uF"
+		(property "Value" "GRM21BR6YA106KE43L"
 			(at 126.238 78.994 0)
 			(show_name no)

Commit message: Working on CM4 IO
Parts:
- C20: value GRM21BR6YA106KE43L -> 10uF
- C21: value CL10A105KA8NNNC -> 1uF
- C44, C45: value C43Q1103K40C80F -> 10nF
Changed lines of the file:
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@@
 			)
 		)
-		(property "Value" "C43Q1103K40C80F"
+		(property "Value" "10nF"
 			(at 119.634 135.3821 90)
 			(show_name no)
@@
 			)
 		)
-		(property "Value" "GRM21BR6YA106KE43L"
+		(property "Value" "10uF"
 			(at 32.258 52.324 0)
 			(show_name no)
@@
 			)
 		)
-		(property "Value" "CL10A105KA8NNNC"
+		(property "Value" "1uF"
 			(at 42.418 51.816 90)
 			(show_name no)
@@
 	)
 	(symbol
+		(lib_name "C43Q1103K40C80F_1")
 		(lib_id "MyParts:C43Q1103K40C80F")
 		(at 140.97 135.89 90)
@@
 			)
 		)
-		(property "Value" "C43Q1103K40C80F"
+		(property "Value" "10nF"
 			(at 143.51 135.8901 90)
 			(show_name no)

Commit message: CM4 schematic changes, before renumbering
Parts:
- removed C20: 10uF, MyParts:C0805, symbol MyParts:GRM21BR6YA106KE43L
- removed C21: 1uF, MyParts:C0603, symbol MyParts:CL10A105KA8NNNC
- removed C22, C26: CL05B104KO5NNNC, MyParts:C0402, symbol MyParts:CL05B104KO5NNNC
- removed C27, C33, C39: CL10A105KA8NNNC, MyParts:C0603, symbol MyParts:CL10A105KA8NNNC
- removed C28, C32, C40: GRM21BR6YA106KE43L, MyParts:C0805, symbol MyParts:GRM21BR6YA106KE43L
- removed C34, C38: 10nF, MyParts:C0402, symbol MyParts:0402B103K500CT
- removed C44: 10nF, MyParts:CAP-TH_L13.0-W6.0-P10.00-D1.2, symbol MyParts:C43Q1103K40C80F
- removed CN3, CN4: KF2EDGR-2.54-4P, MyParts:CONN-TH_4P-P2.54_KF2EDGR-2.54-4P, symbol MyParts:KF2EDGR-2.54-4P
- removed D27: SM712_SOT23, Package_TO_SOT_SMD:SOT-23, symbol Diode:SM712_SOT23
- removed D28: SMAJ15CA, Diode_SMD:D_SMA, symbol Diode:SMAJ15CA
- removed H2: 210S-1*2P L=11.6MMGold-plated black, MyParts:HDR-TH_2P-P2.54-V-M-1, symbol MyParts:210S-1*2PL=11.6MMGold-platedblack
- removed L1, L5, L7, L9: BLM15EX331SN1D, MyParts:L0402, symbol MyParts:BLM15EX331SN1D
- removed L3: SMW2012B371BTE, MyParts:FILTER-SMD_4P-L2.0-W1.2-BL, symbol MyParts:SMW2012B371BTE
- removed R18: 5.1kΩ, PCM_JLCPCB:R_0402, symbol PCM_JLCPCB-Resistors:0402,5.1kΩ
- removed R46: 120Ω, PCM_JLCPCB:R_0805, symbol PCM_JLCPCB-Resistors:0805,120Ω
- removed U2: ISOW1432BDFMR, MyParts:SOIC-20_L12.8-W7.5-P1.27-LS10.3-BL, symbol MyParts:ISOW1432BDFMR
- CN5: MPN (none) -> KF2EDGR-2.54-4P; Manufacturer (none) -> KEFA(科发)
Connections:
- no-connect marks 4 -> 2
Other:
- note added: "RS485"
- note added: "There is one RS485 interfaces. The MCU is an RS485 lead, able to send commands to other followers such as a servo driver."
- note removed: "Isolated RS485"
- note removed: "RS485 terminator, 2.54mm"
- note removed: "RS485_1 To Host"
- note removed: "RS485_1_CHASSIS"
- note removed: "RS485_1_GND"
- note removed: "RS485_1_RX"
- note removed: "RS485_1_TX"
- note removed: "There are 2 RS485 interfaces. 1 - To the Host computer, where the MCU is the follower. 2 - The MCU is an RS485 lead, able to send commands to other followers such as a servo driver."
- moved on the sheet: C23, C24, C25, C29, C30, C31, C35, C36, C37, C41, C42, C43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

Commit message: Before adding CAN
Parts:
- renumbered C23 to C20, C24 to C21, C25 to C22, C29 to C23, C30 to C24, C31 to C25, C35 to C26, C36 to C27, C37 to C28, C41 to C29, C42 to C30, C43 to C31, C45 to C32, CN5 to CN3, D30 to D11, D29 to D12, L2 to L1, L4 to L2, L6 to L3, L8 to L4, L10 to L5, R17 to R22, R19 to R23, U3 to U2
Changed lines of the file:
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@@
 		(in_pos_files yes)
 		(dnp no)
-		(property "Reference" "L2"
+		(property "Reference" "L1"
 			(at 94.996 35.814 0)
 			(show_name no)
@@
 			(project "rcm_dish_controller"
 				(path "/10d7c3e5-be4d-4306-a59e-500b86bd141f/25f87735-bff1-413d-a863-85b2ec3ace75"
-					(reference "L2")
+					(reference "L1")
 					(unit 1)
 				)
@@
 		(in_pos_files yes)
 		(dnp no)
-		(property "Reference" "C30"
+		(property "Reference" "C24"
 			(at 187.198 51.816 90)
 			(show_name no)
@@
 			(project "rcm_dish_controller"
 				(path "/10d7c3e5-be4d-4306-a59e-500b86bd141f/25f87735-bff1-413d-a863-85b2ec3ace75"
-					(reference "C30")
+					(reference "C24")
 					(unit 1)
 				)
@@
 		(in_pos_files yes)
 		(dnp no)
-		(property "Reference" "L8"
+		(property "Reference" "L4"
 			(at 196.596 66.294 0)
 			(show_name no)
@@
 			(project "rcm_dish_controller"
 				(path "/10d7c3e5-be4d-4306-a59e-500b86bd141f/25f87735-bff1-413d-a863-85b2ec3ace75"
-					(reference "L8")
+					(reference "L4")
 					(unit 1)
 				)
@@
 		(in_pos_files yes)
 		(dnp no)
-		(property "Reference" "L10"
+		(property "Reference" "L5"
 			(at 198.12 86.36 0)
 			(show_name no)
@@
 			(project "rcm_dish_controller"
 				(path "/10d7c3e5-be4d-4306-a59e-500b86bd141f/25f87735-bff1-413d-a863-85b2ec3ace75"
-					(reference "L10")
+					(reference "L5")
 					(unit 1)
 				)
@@
 		(in_pos_files yes)
 		(dnp no)
-		(property "Reference" "D30"
+		(property "Reference" "D11"
 			(at 173.99 23.368 0)
 			(show_name no)
@@
 			(project "rcm_dish_controller"
 				(path "/10d7c3e5-be4d-4306-a59e-500b86bd141f/25f87735-bff1-413d-a863-85b2ec3ace75"
-					(reference "D30")
+					(reference "D11")
 					(unit 1)
 				)
@@
 		(in_pos_files yes)
 		(dnp no)
-		(property "Reference" "#PWR076"
+		(property "Reference" "#PWR022"
 			(at 173.99 39.37 0)
 			(hide yes)
@@
 			(project "rcm_dish_controller"
 				(path "/10d7c3e5-be4d-4306-a59e-500b86bd141f/25f87735-bff1-413d-a863-85b2ec3ace75"
-					(reference "#PWR076")
+					(reference "#PWR022")
 					(unit 1)
 				)
@@
 		(in_pos_files yes)
 		(dnp no)
-		(property "Reference" "C24"
+		(property "Reference" "C21"
 			(at 107.188 45.466 90)
 			(show_name no)
@@
 			(project "rcm_dish_controller"
 				(path "/10d7c3e5-be4d-4306-a59e-500b86bd141f/25f87735-bff1-413d-a863-85b2ec3ace75"
-					(reference "C24")
+					(reference "C21")
 					(unit 1)
 				)
@@
 		(in_pos_files yes)
 		(dnp no)
-		(property "Reference" "L6"
+		(property "Reference" "L3"
 			(at 100.584 63.5 0)
 			(show_name no)
@@
 			(project "rcm_dish_controller"
 				(path "/10d7c3e5-be4d-4306-a59e-500b86bd141f/25f87735-bff1-413d-a863-85b2ec3ace75"
-					(reference "L6")
+					(reference "L3")
 					(unit 1)
 				)
@@
 		(in_pos_files yes)
 		(dnp no)
-		(property "Reference" "C23"
+		(property "Reference" "C20"
 			(at 97.028 46.482 0)
 			(show_name no)
@@
 			(project "rcm_dish_controller"
 				(path "/10d7c3e5-be4d-4306-a59e-500b86bd141f/25f87735-bff1-413d-a863-85b2ec3ace75"
-					(reference "C23")
+					(reference "C20")
 					(unit 1)
 				)
@@
 		(in_pos_files yes)
 		(dnp no)
-		(property "Reference" "C37"
+		(property "Reference" "C28"
 			(at 128.27 66.802 0)
 			(show_name no)
@@
 			(project "rcm_dish_controller"
 				(path "/10d7c3e5-be4d-4306-a59e-500b86bd141f/25f87735-bff1-413d-a863-85b2ec3ace75"
-					(reference "C37")
+					(reference "C28")
 					(unit 1)
 				)
@@
 		(in_pos_files yes)
 		(dnp no)
-		(property "Reference" "L4"
+		(property "Reference" "L2"
 			(at 179.832 49.022 0)
 			(show_name no)
@@
 			(project "rcm_dish_controller"
 				(path "/10d7c3e5-be4d-4306-a59e-500b86bd141f/25f87735-bff1-413d-a863-85b2ec3ace75"
-					(reference "L4")
+					(reference "L2")
 					(unit 1)
 				)
@@
 		(in_pos_files yes)
 		(dnp no)
-		(property "Reference" "C35"
+		(property "Reference" "C26"
 			(at 109.728 66.802 0)
 			(show_name no)
@@
 			(project "rcm_dish_controller"
 				(path "/10d7c3e5-be4d-4306-a59e-500b86bd141f/25f87735-bff1-413d-a863-85b2ec3ace75"
-					(reference "C35")
+					(reference "C26")
 					(unit 1)
 				)
@@
 		(in_pos_files yes)
 		(dnp no)
-		(property "Reference" "R17"
+		(property "Reference" "R22"
 			(at 192.532 40.894 0)
 			(show_name no)
@@
 			(project "rcm_dish_controller"
 				(path "/10d7c3e5-be4d-4306-a59e-500b86bd141f/25f87735-bff1-413d-a863-85b2ec3ace75"
-					(reference "R17")
+					(reference "R22")
 					(unit 1)
 				)
@@
 		(in_pos_files yes)
 		(dnp no)
-		(property "Reference" "C31"
+		(property "Reference" "C25"
 			(at 197.358 52.832 0)
 			(show_name no)
@@
 			(project "rcm_dish_controller"
 				(path "/10d7c3e5-be4d-4306-a59e-500b86bd141f/25f87735-bff1-413d-a863-85b2ec3ace75"
-					(reference "C31")
+					(reference "C25")
 					(unit 1)
 				)
@@
 		(in_pos_files yes)
 		(dnp no)
-		(property "Reference" "C45"
+		(property "Reference" "C32"
 			(at 162.56 131.572 90)
 			(show_name no)
@@
 			(project "rcm_dish_controller"
 				(path "/10d7c3e5-be4d-4306-a59e-500b86bd141f/25f87735-bff1-413d-a863-85b2ec3ace75"
-					(reference "C45")
+					(reference "C32")
 					(unit 1)
 				)
@@
 		(in_pos_files yes)
 		(dnp no)
-		(property "Reference" "C25"
+		(property "Reference" "C22"
 			(at 115.316 45.974 90)
 			(show_name no)
@@
 			(project "rcm_dish_controller"
 				(path "/10d7c3e5-be4d-4306-a59e-500b86bd141f/25f87735-bff1-413d-a863-85b2ec3ace75"
-					(reference "C25")
+					(reference "C22")
 					(unit 1)
 				)
@@
 		(in_pos_files yes)
 		(dnp no)
-		(property "Reference" "D29"
+		(property "Reference" "D12"
 			(at 147.828 131.572 90)
 			(show_name no)
@@
 			(project "rcm_dish_controller"
 				(path "/10d7c3e5-be4d-4306-a59e-500b86bd141f/25f87735-bff1-413d-a863-85b2ec3ace75"
-					(reference "D29")
+					(reference "D12")
 					(unit 1)
 				)
@@
 		(in_pos_files yes)
 		(dnp no)
-		(property "Reference" "C43"
+		(property "Reference" "C31"
 			(at 191.008 73.152 0)
 			(show_name no)
@@
 			(project "rcm_dish_controller"
 				(path "/10d7c3e5-be4d-4306-a59e-500b86bd141f/25f87735-bff1-413d-a863-85b2ec3ace75"
-					(reference "C43")
+					(reference "C31")
 					(unit 1)
 				)
@@
 		(dnp no)
 		(fields_autoplaced yes)
-		(property "Reference" "#PWR027"
+		(property "Reference" "#PWR025"
 			(at 134.62 82.55 0)
 			(hide yes)
@@
 			(project "rcm_dish_controller"
 				(path "/10d7c3e5-be4d-4306-a59e-500b86bd141f/25f87735-bff1-413d-a863-85b2ec3ace75"
-					(reference "#PWR027")
+					(reference "#PWR025")
 					(unit 1)
 				)
@@
 		(in_pos_files yes)
 		(dnp no)
-		(property "Reference" "#PWR029"
+		(property "Reference" "#PWR026"
 			(at 195.58 99.06 0)
 			(hide yes)
@@
 			(project "rcm_dish_controller"
 				(path "/10d7c3e5-be4d-4306-a59e-500b86bd141f/25f87735-bff1-413d-a863-85b2ec3ace75"
-					(reference "#PWR029")
+					(reference "#PWR026")
 					(unit 1)
 				)
@@
 		(in_pos_files yes)
 		(dnp no)
-		(property "Reference" "#PWR025"
+		(property "Reference" "#PWR024"
 			(at 184.15 68.58 0)
 			(hide yes)
@@
 			(project "rcm_dish_controller"
 				(path "/10d7c3e5-be4d-4306-a59e-500b86bd141f/25f87735-bff1-413d-a863-85b2ec3ace75"
-					(reference "#PWR025")
+					(reference "#PWR024")
 					(unit 1)
 				)
@@
 		(in_pos_files yes)
 		(dnp no)
-		(property "Reference" "R19"
+		(property "Reference" "R23"
 			(at 84.074 48.514 0)
 			(show_name no)
@@
 			(project "rcm_dish_controller"
 				(path "/10d7c3e5-be4d-4306-a59e-500b86bd141f/25f87735-bff1-413d-a863-85b2ec3ace75"
-					(reference "R19")
+					(reference "R23")
 					(unit 1)
 				)
@@
 		(in_pos_files yes)
 		(dnp no)
-		(property "Reference" "C29"
+		(property "Reference" "C23"
 			(at 177.546 52.324 90)
 			(show_name no)
@@
 			(project "rcm_dish_controller"
 				(path "/10d7c3e5-be4d-4306-a59e-500b86bd141f/25f87735-bff1-413d-a863-85b2ec3ace75"
-					(reference "C29")
+					(reference "C23")
 					(unit 1)
 				)
@@
 		(in_pos_files yes)
 		(dnp no)
-		(property "Reference" "C36"
+		(property "Reference" "C27"
 			(at 119.888 65.786 90)
 			(show_name no)
@@
 			(project "rcm_dish_controller"
 				(path "/10d7c3e5-be4d-4306-a59e-500b86bd141f/25f87735-bff1-413d-a863-85b2ec3ace75"
-					(reference "C36")
+					(reference "C27")
 					(unit 1)
 				)
@@
 		(in_pos_files yes)
 		(dnp no)
-		(property "Reference" "CN5"
+		(property "Reference" "CN3"
 			(at 75.692 129.794 0)
 			(show_name no)
@@
 			(project "rcm_dish_controller"
 				(path "/10d7c3e5-be4d-4306-a59e-500b86bd141f/25f87735-bff1-413d-a863-85b2ec3ace75"
-					(reference "CN5")
+					(reference "CN3")
 					(unit 1)
 				)
@@
 		(in_pos_files yes)
 		(dnp no)
-		(property "Reference" "U3"
+		(property "Reference" "U2"
 			(at 150.876 53.594 0)
 			(show_name no)
@@
 			(project "rcm_dish_controller"
 				(path "/10d7c3e5-be4d-4306-a59e-500b86bd141f/25f87735-bff1-413d-a863-85b2ec3ace75"
-					(reference "U3")
+					(reference "U2")
 					(unit 1)
 				)
@@
 		(in_pos_files yes)
 		(dnp no)
-		(property "Reference" "C41"
+		(property "Reference" "C29"
 			(at 173.482 72.898 0)
 			(show_name no)
@@
 			(project "rcm_dish_controller"
 				(path "/10d7c3e5-be4d-4306-a59e-500b86bd141f/25f87735-bff1-413d-a863-85b2ec3ace75"
-					(reference "C41")
+					(reference "C29")
 					(unit 1)
 				)
@@
 		(in_pos_files yes)
 		(dnp no)
-		(property "Reference" "C42"
+		(property "Reference" "C30"
 			(at 182.626 72.898 90)
 			(show_name no)
@@
 			(project "rcm_dish_controller"
 				(path "/10d7c3e5-be4d-4306-a59e-500b86bd141f/25f87735-bff1-413d-a863-85b2ec3ace75"
-					(reference "C42")
+					(reference "C30")
 					(unit 1)
 				)
