File: kicad/rcm_dish_controller.kicad_sch (KiCad schematic)
At the start: 24 parts, among them J1 Conn_ST_STDC14, SW1 DSHP04TSGER, U1 STM32G474RET6, X1 NX2016SA-16MHZ-EXS00A-CS07826

Commit message: Updates to power
Parts:
- R2, R70: LCSC C173683 -> C25744
Other:
- added sheet RCM4 (RCM4.kicad_sch)
Changed lines of the file:
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@@
 	)
 	(rectangle
-		(start 74.93 148.59)
-		(end 111.76 177.8)
+		(start 73.66 147.32)
+		(end 116.84 177.8)
 		(stroke
 			(width 0)
@@
 	(wire
 		(pts
+			(xy 100.33 163.83) (xy 100.33 171.45)
+		)
+		(stroke
+			(width 0)
+			(type default)
+		)
+	)
+	(wire
+		(pts
 			(xy 87.63 20.32) (xy 87.63 36.83)
 		)
@@
 	(wire
 		(pts
-			(xy 81.28 163.83) (xy 81.28 171.45)
+			(xy 78.74 163.83) (xy 78.74 171.45)
 		)
 		(stroke
@@
 	(wire
 		(pts
-			(xy 92.71 163.83) (xy 92.71 171.45)
+			(xy 90.17 163.83) (xy 90.17 171.45)
 		)
 		(stroke
@@
 	(wire
 		(pts
-			(xy 104.14 163.83) (xy 104.14 171.45)
+			(xy 110.49 163.83) (xy 110.49 171.45)
 		)
 		(stroke
@@
 	(global_label "GND"
 		(shape input)
-		(at 104.14 163.83 90)
+		(at 110.49 163.83 90)
 		(fields_autoplaced yes)
 		(effects
@@
 		)
 		(property "Intersheetrefs" "${INTERSHEET_REFS}"
-			(at 104.14 156.9743 90)
+			(at 110.49 156.9743 90)
 			(hide yes)
 			(show_name no)
@@
 	(global_label "12V"
 		(shape input)
-		(at 81.28 163.83 90)
+		(at 78.74 163.83 90)
 		(fields_autoplaced yes)
 		(effects
@@
 		)
 		(property "Intersheetrefs" "${INTERSHEET_REFS}"
-			(at 81.28 157.3372 90)
+			(at 78.74 157.3372 90)
 			(hide yes)
 			(show_name no)
@@
 	(global_label "3V3"
 		(shape input)
-		(at 92.71 163.83 90)
+		(at 90.17 163.83 90)
 		(fields_autoplaced yes)
 		(effects
@@
 		)
 		(property "Intersheetrefs" "${INTERSHEET_REFS}"
-			(at 92.71 156.7324 90)
+			(at 90.17 156.7324 90)
 			(hide yes)
 			(show_name no)
@@
 		)
 	)
+	(global_label "5V"
+		(shape input)
+		(at 100.33 163.83 90)
+		(fields_autoplaced yes)
+		(effects
+			(font
+				(size 1.27 1.27)
+			)
+			(justify left)
+		)
+		(property "Intersheetrefs" "${INTERSHEET_REFS}"
+			(at 100.33 158.5467 90)
+			(hide yes)
+			(show_name no)
+			(do_not_autoplace no)
+			(effects
+				(font
+					(size 1.27 1.27)
+				)
+				(justify left)
+			)
+		)
+	)
 	(global_label "3V3"
 		(shape input)
@@
 			)
 		)
-		(property "Datasheet" "https://www.lcsc.com/datasheet/lcsc_datasheet_2411221126_UNI-ROYAL-Uniroyal-Elec-0402WGF1002TCE_C173683.pdf"
+		(property "Datasheet" "https://www.lcsc.com/datasheet/lcsc_datasheet_2411221126_UNI-ROYAL-Uniroyal-Elec-0402WGF1002TCE_C25744.pdf"
 			(at 40.64 52.07 0)
 			(hide yes)
@@
 			)
 		)
-		(property "LCSC" "C173683"
+		(property "LCSC" "C25744"
 			(at 40.64 52.07 0)
 			(hide yes)
@@
 	(symbol
 		(lib_id "power:PWR_FLAG")
-		(at 104.14 171.45 180)
+		(at 110.49 171.45 180)
 		(unit 1)
 		(body_style 1)
@@
 		(dnp no)
 		(property "Reference" "#FLG03"
-			(at 104.14 173.355 0)
+			(at 110.49 173.355 0)
 			(hide yes)
 			(show_name no)
@@
 		)
 		(property "Value" "PWR_FLAG"
-			(at 104.14 175.26 0)
+			(at 110.49 175.26 0)
 			(show_name no)
 			(do_not_autoplace no)
@@
 		)
 		(property "Footprint" ""
-			(at 104.14 171.45 0)
+			(at 110.49 171.45 0)
 			(hide yes)
 			(show_name no)
@@
 		)
 		(property "Datasheet" ""
-			(at 104.14 171.45 0)
+			(at 110.49 171.45 0)
 			(hide yes)
 			(show_name no)
@@
 		)
 		(property "Description" "Special symbol for telling ERC where power comes from"
-			(at 104.14 171.45 0)
+			(at 110.49 171.45 0)
 			(hide yes)
 			(show_name no)
@@
 	(symbol
 		(lib_id "power:PWR_FLAG")
-		(at 81.28 171.45 180)
+		(at 78.74 171.45 180)
 		(unit 1)
 		(body_style 1)
@@
 		(dnp no)
 		(property "Reference" "#FLG01"
-			(at 81.28 173.355 0)
+			(at 78.74 173.355 0)
 			(hide yes)
 			(show_name no)
@@
 		)
 		(property "Value" "PWR_FLAG"
-			(at 81.28 175.26 0)
+			(at 78.74 175.26 0)
 			(show_name no)
 			(do_not_autoplace no)
@@
 		)
 		(property "Footprint" ""
-			(at 81.28 171.45 0)
+			(at 78.74 171.45 0)
 			(hide yes)
 			(show_name no)
@@
 		)
 		(property "Datasheet" ""
-			(at 81.28 171.45 0)
+			(at 78.74 171.45 0)
 			(hide yes)
 			(show_name no)
@@
 		)
 		(property "Description" "Special symbol for telling ERC where power comes from"
-			(at 81.28 171.45 0)
+			(at 78.74 171.45 0)
 			(hide yes)
 			(show_name no)
@@
 	(symbol
 		(lib_id "power:PWR_FLAG")
-		(at 92.71 171.45 180)
+		(at 90.17 171.45 180)
 		(unit 1)
 		(body_style 1)
@@
 		(dnp no)
 		(property "Reference" "#FLG02"
-			(at 92.71 173.355 0)
+			(at 90.17 173.355 0)
 			(hide yes)
 			(show_name no)
@@
 		)
 		(property "Value" "PWR_FLAG"
-			(at 92.71 175.26 0)
+			(at 90.17 175.26 0)
 			(show_name no)
 			(do_not_autoplace no)
@@
 		)
 		(property "Footprint" ""
-			(at 92.71 171.45 0)
+			(at 90.17 171.45 0)
 			(hide yes)
 			(show_name no)
@@
 		)
 		(property "Datasheet" ""
-			(at 92.71 171.45 0)
+			(at 90.17 171.45 0)
 			(hide yes)
 			(show_name no)
@@
 		)
 		(property "Description" "Special symbol for telling ERC where power comes from"
-			(at 92.71 171.45 0)
+			(at 90.17 171.45 0)
 			(hide yes)
 			(show_name no)
@@
 	)
 	(symbol
+		(lib_id "power:PWR_FLAG")
+		(at 100.33 171.45 180)
+		(unit 1)
+		(body_style 1)
+		(exclude_from_sim no)
+		(in_bom no)
+		(on_board no)
+		(in_pos_files yes)
+		(dnp no)
+		(property "Reference" "#FLG07"
+			(at 100.33 173.355 0)
+			(hide yes)
+			(show_name no)
+			(do_not_autoplace no)
+			(effects
+				(font
+					(size 1.27 1.27)
+				)
+			)
+		)
+		(property "Value" "PWR_FLAG"
+			(at 100.33 175.26 0)
+			(show_name no)
+			(do_not_autoplace no)
+			(effects
+				(font
+					(size 1.27 1.27)
+				)
+			)
+		)
+		(property "Footprint" ""
+			(at 100.33 171.45 0)
+			(hide yes)
+			(show_name no)
+			(do_not_autoplace no)
+			(effects
+				(font
+					(size 1.27 1.27)
+				)
+			)
+		)
+		(property "Datasheet" ""
+			(at 100.33 171.45 0)
+			(hide yes)
+			(show_name no)
+			(do_not_autoplace no)
+			(effects
+				(font
+					(size 1.27 1.27)
+				)
+			)
+		)
+		(property "Description" "Special symbol for telling ERC where power comes from"
+			(at 100.33 171.45 0)
+			(hide yes)
+			(show_name no)
+			(do_not_autoplace no)
+			(effects
+				(font
+					(size 1.27 1.27)
+				)
+			)
+		)
+		(pin "1"
+		)
+		(instances
+			(project "rcm_dish_controller"
+				(path "/10d7c3e5-be4d-4306-a59e-500b86bd141f"
+					(reference "#FLG07")
+					(unit 1)
+				)
+			)
+		)
+	)
+	(symbol
 		(lib_id "PCM_JLCPCB-Resistors:0402,10kΩ")
 		(at 130.81 52.07 180)
@@
 			)
 		)
-		(property "Datasheet" "https://www.lcsc.com/datasheet/lcsc_datasheet_2411221126_UNI-ROYAL-Uniroyal-Elec-0402WGF1002TCE_C173683.pdf"
+		(property "Datasheet" "https://www.lcsc.com/datasheet/lcsc_datasheet_2411221126_UNI-ROYAL-Uniroyal-Elec-0402WGF1002TCE_C25744.pdf"
 			(at 130.81 52.07 0)
 			(hide yes)
@@
 			)
 		)
-		(property "LCSC" "C173683"
+		(property "LCSC" "C25744"
 			(at 130.81 52.07 0)
 			(hide yes)
@@
 				)
 			)
+		)
+	)
+	(sheet
+		(at 208.28 148.59)
+		(size 16.51 13.97)
+		(exclude_from_sim no)
+		(in_bom yes)
+		(on_board yes)
+		(dnp no)
+		(fields_autoplaced yes)
+		(stroke
+			(width 0.1524)
+			(type solid)
+		)
+		(fill
+			(color 0 0 0 0)
+		)
+		(property "Sheetname" "RCM4"
+			(at 208.28 147.8784 0)
+			(show_name no)
+			(do_not_autoplace no)
+			(effects
+				(font
+					(size 1.27 1.27)
+				)
+				(justify left bottom)
+			)
+		)
+		(property "Sheetfile" "RCM4.kicad_sch"
+			(at 208.28 163.1446 0)
+			(show_name no)
+			(do_not_autoplace no)
+			(effects
+				(font
+					(size 1.27 1.27)
+				)
+				(justify left top)
+			)
+		)
+		(instances
+			(project "rcm_dish_controller"
+				(path "/10d7c3e5-be4d-4306-a59e-500b86bd141f"
+					(page "11")
+				)
+			)

Commit message: CM4 schematic changes, before renumbering
Connections:
- net ADDR0 renamed SW1
- net ADDR1 renamed SW2
- net ADDR2 renamed SW3
- net CONFIG_SW renamed SW4
- net RS232_RX_MCU renamed GPS_RX_MCU
- net RS232_TX_MCU renamed GPS_TX_MCU
- net RS485_1_DE_MCU: no longer names the net of U1.58 (PB5)
- net RS485_1_RX_MCU renamed CM4_RX
- net RS485_1_TX_MCU renamed CM4_TX
- no-connect marks 8 -> 9
Other:
- sheet Axis Control - 1 ports: added DIR1_MCU, ENABLE1_MCU, ENC1_A_MCU, ENC1_B_MCU, ENC1_Z_MCU, LIMIT1_SW1_MCU, LIMIT1_SW2_MCU, PUL1_MCU; removed none
- sheet Axis Control - 2 ports: added DIR2_MCU, ENABLE2_MCU, ENC2_A_MCU, ENC2_B_MCU, ENC2_Z_MCU, LIMIT2_SW1_MCU, LIMIT2_SW2_MCU, PUL2_MCU; removed none
- sheet Fan ports: added FAN_MCU; removed none
- sheet GPS ports: added 1PPS_MCU, GPS_RX_MCU, GPS_TX_MCU; removed none
- sheet I2C and EEPROM ports: added FLASH_CS_MCU, SCL_MCU, SDA_MCU, SPI2_MISO_MCU, SPI2_MOSI_MCU, SPI2_SCK_MCU; removed none
- sheet RCM4 ports: added 1PPS_MCU, CM4_RX, CM4_TX; removed none
- sheet RS485 ports: added RS485_2_DE_MCU, RS485_2_RX_MCU, RS485_2_TX_MCU; removed none
- sheet User Switches ports: added USER_SW_1_MCU, USER_SW_2_MCU, USER_SW_3_MCU, USER_SW_4_MCU; removed none
- note added: "Switch: SW1,2,3,4 are the are general purpose config switches for possible future use."
- note removed: "Purpose: Control 2 Axes of a motor controlled system. - Modbus commands over isolated RS485. - MCU outputs motor PWM, direction, enable/disable - Input from encoder connected to motor output - Host provides configuration and position commands - MCU runs a PID loop to position/move motor - Onboard temperature sensor, MCU can turn fan on/off - I2C extender for sensors placed at the axis - 3V3 UART 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"
- note removed: "Switch: Pins 1,2,3 are the address of this board on the RS485_1 bus. Pin 4 is an extra pin that may be of future use, but not used now."

Commit message: Before adding CAN
Parts:
- renumbered C18 to C12, R70 to R1, TP4 to TP1, TP5 to TP2
Other:
- added sheet CAN (can.kicad_sch)
Changed lines of the file:
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@@
 		(in_pos_files yes)
 		(dnp no)
-		(property "Reference" "R70"
+		(property "Reference" "R1"
 			(at 35.56 50.546 0)
 			(show_name no)
@@
 			(project "rcm_dish_controller"
 				(path "/10d7c3e5-be4d-4306-a59e-500b86bd141f"
-					(reference "R70")
+					(reference "R1")
 					(unit 1)
 				)
@@
 		(dnp no)
 		(fields_autoplaced yes)
-		(property "Reference" "#PWR073"
+		(property "Reference" "#PWR09"
 			(at 68.58 142.24 0)
 			(hide yes)
@@
 			(project "rcm_dish_controller"
 				(path "/10d7c3e5-be4d-4306-a59e-500b86bd141f"
-					(reference "#PWR073")
+					(reference "#PWR09")
 					(unit 1)
 				)
@@
 		(in_pos_files yes)
 		(dnp no)
-		(property "Reference" "#FLG03"
+		(property "Reference" "#FLG04"
 			(at 110.49 173.355 0)
 			(hide yes)
@@
 			(project "rcm_dish_controller"
 				(path "/10d7c3e5-be4d-4306-a59e-500b86bd141f"
-					(reference "#FLG03")
+					(reference "#FLG04")
 					(unit 1)
 				)
@@
 		(dnp no)
 		(fields_autoplaced yes)
-		(property "Reference" "TP4"
+		(property "Reference" "TP1"
 			(at 110.49 132.0799 0)
 			(show_name no)
@@
 			(project "rcm_dish_controller"
 				(path "/10d7c3e5-be4d-4306-a59e-500b86bd141f"
-					(reference "TP4")
+					(reference "TP1")
 					(unit 1)
 				)
@@
 		(in_pos_files yes)
 		(dnp no)
-		(property "Reference" "#FLG07"
+		(property "Reference" "#FLG03"
 			(at 100.33 173.355 0)
 			(hide yes)
@@
 			(project "rcm_dish_controller"
 				(path "/10d7c3e5-be4d-4306-a59e-500b86bd141f"
-					(reference "#FLG07")
+					(reference "#FLG03")
 					(unit 1)
 				)
@@
 		(in_pos_files yes)
 		(dnp no)
-		(property "Reference" "C18"
+		(property "Reference" "C12"
 			(at 25.4 149.6059 0)
 			(show_name no)
@@
 			(project "rcm_dish_controller"
 				(path "/10d7c3e5-be4d-4306-a59e-500b86bd141f"
-					(reference "C18")
+					(reference "C12")
 					(unit 1)
 				)
@@
 		(dnp no)
 		(fields_autoplaced yes)
-		(property "Reference" "#PWR015"
+		(property "Reference" "#PWR011"
 			(at 127 175.26 0)
 			(hide yes)
@@
 			(project "rcm_dish_controller"
 				(path "/10d7c3e5-be4d-4306-a59e-500b86bd141f"
-					(reference "#PWR015")
+					(reference "#PWR011")
 					(unit 1)
 				)
@@
 		(dnp no)
 		(fields_autoplaced yes)
-		(property "Reference" "#PWR021"
+		(property "Reference" "#PWR012"
 			(at 165.1 175.26 0)
 			(hide yes)
@@
 			(project "rcm_dish_controller"
 				(path "/10d7c3e5-be4d-4306-a59e-500b86bd141f"
-					(reference "#PWR021")
+					(reference "#PWR012")
 					(unit 1)
 				)
@@
 		(dnp no)
 		(fields_autoplaced yes)
-		(property "Reference" "TP5"
+		(property "Reference" "TP2"
 			(at 78.74 133.3499 0)
 			(show_name no)
@@
 			(project "rcm_dish_controller"
 				(path "/10d7c3e5-be4d-4306-a59e-500b86bd141f"
-					(reference "TP5")
+					(reference "TP2")
 					(unit 1)
 				)
@@
 		(dnp no)
 		(fields_autoplaced yes)
-		(property "Reference" "#PWR011"
+		(property "Reference" "#PWR013"
 			(at 40.64 186.69 0)
 			(hide yes)
@@
 			(project "rcm_dish_controller"
 				(path "/10d7c3e5-be4d-4306-a59e-500b86bd141f"
-					(reference "#PWR011")
+					(reference "#PWR013")
 					(unit 1)
 				)
@@
 				)
 			)
+		)
+	)
+	(sheet
+		(at 176.53 136.525)
+		(size 22.86 13.335)
+		(exclude_from_sim no)
+		(in_bom yes)
+		(on_board yes)
+		(dnp no)
+		(fields_autoplaced yes)
+		(stroke
+			(width 0.1524)
+			(type solid)
+		)
+		(fill
+			(color 0 0 0 0)
+		)
+		(property "Sheetname" "CAN"
+			(at 176.53 135.8134 0)
+			(show_name no)
+			(do_not_autoplace no)
+			(effects
+				(font
+					(size 1.27 1.27)
+				)
+				(justify left bottom)
+			)
+		)
+		(property "Sheetfile" "can.kicad_sch"
+			(at 176.53 150.4446 0)
+			(show_name no)
+			(do_not_autoplace no)
+			(effects
+				(font
+					(size 1.27 1.27)
+				)
+				(justify left top)
+			)
+		)
+		(instances
+			(project "rcm_dish_controller"
+				(path "/10d7c3e5-be4d-4306-a59e-500b86bd141f"
+					(page "17")
+				)
+			)

Commit message: More mods
Connections:
- net RS485_2_TX_MCU is gone; now on net SW1: U1.52 (PC10)
- net SW1: no longer U1.45 (PA11)
- net CAN_TX: now reaches U1.46 (PA12)
- net CAN_TX: no longer R3.1
- net RS485_2_DE_MCU renamed MCU_nIRQ
- net RS485_2_RX_MCU renamed STATUS_LED
- net STATUS_LED: now also R3.1
- new net CAN_RX: U1.45 (PA11)
Other:
- removed sheet RS485
- sheet CAN ports: added CAN_RX, CAN_TX; removed none
- sheet RCM4 ports: added MCU_nIRQ; removed none
- note added: "PA8,9,10 and PC10 should be configured to internal pull-up."
- note removed: "PA8,9,10,11 should be configured to internal pull-up."
- moved on the sheet: LED1, R3
