File: kicad/rcm_dish_controller.kicad_pcb (KiCad board)
At the start: 4 copper layers, 100 x 100 mm, 248 parts, among them CN1 KF2EDGR-2.54-9P, CN12 KF2EDGR-2.54-9P, CN13 KF2EDGR-2.54-6P, CN14 KF2EDGR-2.54-6P, CN17 SMA-KWE_C7498154, CN2 KF2EDGR-2.54-6P, CN3 KF2EDGR-2.54-4P, CN4 KF2EDGR-2.54-4P, CN5 KF2EDGR-2.54-4P, CN7 SM04B-SRSS-TB (LF)(SN), CN8 SM04B-SRSS-TB (LF)(SN), CN9 KF2EDGR-2.54-2P, J1 Conn_ST_STDC14, M1 MountingHole_2.7mm_M2.5_ISO14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, Q1 AO3407A, Q2 AO3400A, Q4 AO3407A, Q5 BSS138, Q6 BSS138, Q7 BSS138, Q8 BSS138, SW1 DSHP04TSGER, SW2 SS-12F49-G050, U1 STM32G474RET6, U2 ISOW1432BDFMR, U3 ISOW1432BDFMR, U4 MP2322GQH-Z, U5 LTC4311ISC6#TRPBF, U6 LM75BIMX-3/NOPB, U7 W25Q32JVSSIQ_C179173, U8 MAX-M10S-00B, X1 NX2016SA-16MHZ-EXS00A-CS07826

Commit message: CM4 schematic changes, before renumbering
Parts:
- removed C20, C28, C32, C40: 10uF, MyParts:C0805
- removed C21, C27, C33, C39: 1uF, MyParts:C0603
- removed C22, C26: 100nF, MyParts:C0402
- removed C34, C38: 10nF, MyParts:C0402
- removed C44: 10nF, MyParts:CAP-TH_L13.0-W6.0-P10.00-D1.2
- removed CN3, CN4: KF2EDGR-2.54-4P, MyParts:CONN-TH_4P-P2.54_KF2EDGR-2.54-4P
- removed D27: SM712_SOT23, Package_TO_SOT_SMD:SOT-23
- removed D28: SMAJ15CA, Diode_SMD:D_SMA
- removed H2: 210S-1*2P L=11.6MMGold-plated black, MyParts:HDR-TH_2P-P2.54-V-M-1
- removed L1, L5, L7, L9: BLM15EX331SN1D, MyParts:L0402
- removed L3: Choke, MyParts:FILTER-SMD_4P-L2.0-W1.2-BL
- removed U2: ISOW1432BDFMR, MyParts:SOIC-20_L12.8-W7.5-P1.27-LS10.3-BL
- added C100: 10uF 35V, MyParts:C0805, F.Cu at (47.1, 121.3)
- added C101: 10uF 35V, MyParts:C0805, F.Cu at (65.8, 124.2)
- added C102: 100nF, PCM_JLCPCB:C_0402, F.Cu at (54.1, 130.2)
- added C103: 10uF 35V, MyParts:C0805, F.Cu at (70.9, 109.5)
- added C104: 56pF, MyParts:C0402, F.Cu at (59.3, 117.6)
- added C105: 2.7nF 50V, MyParts:C0402, F.Cu at (59.3, 119.8)
- added C106: 100nF, PCM_JLCPCB:C_0402, F.Cu at (54.1, 132.1)
- added C107: DNP, MyParts:C0402, F.Cu at (59.3, 121.9)
- added C108: 10uF 10V, MyParts:C0805, F.Cu at (108.0, 60.2)
- added C109: 10uF 10V, MyParts:C0805, F.Cu at (108.0, 63.2)
- added C110: 100uF 6.3V, Capacitor_Tantalum_SMD:CP_EIA-7343-31_Kemet-D, F.Cu at (44.5, 128.6)
- added C111: 10uF 35V, MyParts:C0805, F.Cu at (70.9, 112.4)
- added C112: 10uF 35V, MyParts:C0805, F.Cu at (70.9, 115.4)
- added C113: 10uF 35V, MyParts:C0805, F.Cu at (70.9, 118.3)
- added C114: 10uF 35V, MyParts:C0805, F.Cu at (70.9, 121.3)
- added C115: 100nF, PCM_JLCPCB:C_0402, F.Cu at (77.9, 130.2)
- added C116: 100nF, PCM_JLCPCB:C_0402, F.Cu at (77.9, 132.1)
- added C117: 100uF 6.3V, Capacitor_Tantalum_SMD:CP_EIA-7343-31_Kemet-D, F.Cu at (68.3, 128.6)
- added C46: 100nF, PCM_JLCPCB:C_0402, F.Cu at (108.6, 87.8)
- added C47: 10uF 10V, MyParts:C0805, F.Cu at (42.1, 109.5)
- added C48: 10uF 10V, MyParts:C0805, F.Cu at (42.1, 112.4)
- added C49: 10uF 10V, MyParts:C0805, F.Cu at (42.1, 115.4)
- added C50: 10uF 10V, MyParts:C0805, F.Cu at (42.1, 118.3)
- added C51: 100nF, MyParts:C0805, F.Cu at (42.1, 121.3)
- added C52: 10uF 10V, MyParts:C0805, F.Cu at (65.8, 109.5)
- added C53: 10uF 10V, MyParts:C0805, F.Cu at (65.8, 112.4)
- added C54: 10uF 10V, MyParts:C0805, F.Cu at (65.8, 115.4)
- added C77: 10uF 10V, MyParts:C0805, F.Cu at (65.8, 118.3)
- added C78: 100nF, MyParts:C0805, F.Cu at (65.8, 121.3)
- added C80: 100uF 6.3V, Capacitor_Tantalum_SMD:CP_EIA-7343-31_Kemet-D, F.Cu at (110.5, 75.7)
- added C81: DNP, MyParts:C0402, F.Cu at (83.1, 117.6)
- added C82: 1.2nF, MyParts:C0402, F.Cu at (83.1, 119.8)
- added C83: DNP, MyParts:C0402, F.Cu at (83.1, 121.9)
- added C85: 22pF, PCM_JLCPCB:C_0402, F.Cu at (115.0, 50.8)
- added C86: 22pF, PCM_JLCPCB:C_0402, F.Cu at (115.0, 52.7)
- added C92: 10uF 10V, MyParts:C0805, F.Cu at (108.0, 51.4)
- added C93: 10uF 10V, MyParts:C0805, F.Cu at (108.0, 54.3)
- added C94: 10uF 10V, MyParts:C0805, F.Cu at (108.0, 57.3)
- added C95: 10uF 35V, MyParts:C0805, F.Cu at (42.1, 124.2)
- added C96: 10uF 35V, MyParts:C0805, F.Cu at (47.1, 109.5)
- added C97: 10uF 35V, MyParts:C0805, F.Cu at (47.1, 112.4)
- added C98: 10uF 35V, MyParts:C0805, F.Cu at (47.1, 115.4)
- added C99: 10uF 35V, MyParts:C0805, F.Cu at (47.1, 118.3)
- added DC1: DC007B-2.5-J, MyParts:DC-IN-TH_HX-DC007B-2.5, F.Cu at (96.5, 130.0)
- added F1: SMD1812P300TF/16, MyParts:F1812, F.Cu at (79.8, 126.7)
- added F3: 1812L110/48QR, MyParts:F1812, F.Cu at (56.1, 126.7)
- added H1: Header-Male-2.54_1x3, MyParts:HDR-TH_3P-P2.54-V-M-1, F.Cu at (106.7, 116.2)
- added H5: 210S-1*2P L=11.6MMGold-plated black, MyParts:HDR-TH_2P-P2.54-V-M-1, F.Cu at (99.1, 116.2)
- added H6: 210S-1*2P L=11.6MMGold-plated black, MyParts:HDR-TH_2P-P2.54-V-M-1, F.Cu at (99.1, 120.0)
- added J3: Header-Male-2.54_2x3, MyParts:HDR-TH_6P-P2.54-V-M-R2-C3-S2.54-1, F.Cu at (91.5, 117.5)
- added L15: SRN6045TA-3R3Y, MyParts:IND-SMD_L6.0-W6.0, F.Cu at (53.8, 120.3)
- added L16: SRN6045TA-3R3Y, MyParts:IND-SMD_L6.0-W6.0, F.Cu at (77.5, 120.3)
- added LED3: XL-0805QBC, MyParts:LED0805-R-RD, F.Cu at (83.5, 57.1)
- added LED4: LTST-S270KGKT, MyParts:LED-SMD_L1.7-W0.6-RD, F.Cu at (115.7, 115.8)
- added Module1: ComputeModule4-CM4, CM4_Parts:Raspberry-Pi-4-Compute-Module, F.Cu at (41.0, 90.5)
- added Q11: DMP3013SFV-7, MyParts:DFN-8_L3.3-W3.3-P0.65-BL, F.Cu at (103.1, 139.2)
- added Q12: DMP3013SFV-7, MyParts:DFN-8_L3.3-W3.3-P0.65-BL, F.Cu at (107.6, 139.2)
- added R13: 2.2kΩ, MyParts:R0402, F.Cu at (75.0, 125.2)
- added R20: 1.5kΩ, PCM_JLCPCB:R_0402, F.Cu at (82.1, 52.7)
- added R21: 10kΩ, PCM_JLCPCB:R_0603, F.Cu at (103.2, 129.2)
- added R22: 22.1K, MyParts:R0402, F.Cu at (51.2, 125.2)
- added R23: 15kΩ, PCM_JLCPCB:R_0402, F.Cu at (115.0, 54.5)
- added R39: 20kΩ, MyParts:R0402, F.Cu at (75.0, 127.3)
- added R40: 12kΩ, MyParts:R0402, F.Cu at (75.0, 129.5)
- added R41: 1.5kΩ, PCM_JLCPCB:R_0402, F.Cu at (108.6, 89.7)
- added R42: 1.5kΩ, PCM_JLCPCB:R_0402, F.Cu at (108.6, 91.5)
- added R55: 10Ω, MyParts:R1206, F.Cu at (58.4, 130.9)
- added R56: 10Ω, MyParts:R1206, F.Cu at (82.2, 130.9)
- added R63: 10.5KΩ, MyParts:R0402, F.Cu at (51.2, 127.3)
- added R65: 69.8K, MyParts:R0402, F.Cu at (51.2, 129.5)
- added R83: 36K 1%, MyParts:R0402, F.Cu at (112.1, 51.0)
- added R84: 36K 1%, MyParts:R0402, F.Cu at (112.1, 53.1)
- added R85: 36K 1%, MyParts:R0402, F.Cu at (112.1, 55.3)
- added R86: 36K 1%, MyParts:R0402, F.Cu at (112.1, 57.4)
- added R87: 12kΩ, MyParts:R0402, F.Cu at (112.1, 59.6)
- added R88: 2.2kΩ, MyParts:R0402, F.Cu at (112.1, 61.7)
- added R89: 5.1kΩ, PCM_JLCPCB:R_0402, F.Cu at (115.0, 56.4)
- added R90: 5.1kΩ, PCM_JLCPCB:R_0402, F.Cu at (115.0, 58.2)
- added R91: 4.7kΩ, PCM_JLCPCB:R_0402, F.Cu at (112.5, 115.3)
- added R92: 1kΩ, PCM_JLCPCB:R_0402, F.Cu at (112.5, 117.1)
- added R93: 4.7kΩ, PCM_JLCPCB:R_0402, F.Cu at (112.5, 119.0)
- added RJ1: LPJG0926HENL_C22457393, MyParts:RJ45-TH_LPJG0926HENL_C22457393, F.Cu at (97.6, 89.8)
- added SW4: SS-12F49-G050, MyParts:SW-TH_SS-12F45-GXXX, F.Cu at (94.0, 139.3)
- added TP11: RH-5016, MyParts:TESTPOINT-SMD_L3.0-W2.0, F.Cu at (58.8, 110.0)
- added TP12: RH-5016, MyParts:TESTPOINT-SMD_L3.0-W2.0, F.Cu at (82.6, 110.0)
- added TP13: RH-5016, MyParts:TESTPOINT-SMD_L3.0-W2.0, F.Cu at (82.6, 114.1)
- added TP14: RH-5016, MyParts:TESTPOINT-SMD_L3.0-W2.0, F.Cu at (58.8, 114.1)
- added TP2: RH-5016, MyParts:TESTPOINT-SMD_L3.0-W2.0, F.Cu at (103.9, 126.0)
- added U10: TPD4EUSB30DQAR-N, MyParts:DFN-10_L2.5-W1.0-P0.50-BL-A, F.Cu at (115.7, 60.4)
- added U11: TPD4EUSB30DQAR, MyParts:USON-10_L2.5-W1.0-P0.50-BL, F.Cu at (109.0, 82.3)
- added U12: TPD4EUSB30DQAR, MyParts:USON-10_L2.5-W1.0-P0.50-BL, F.Cu at (109.0, 85.2)
- added U13: AP22653W6-7, MyParts:SOT-23-6_L2.9-W1.6-P0.95-LS2.8-BR, F.Cu at (101.4, 76.6)
- added U14: 2541WV-2X12P, MyParts:HDR-TH_24P-P2.54-V-M-R2-C12-S2.54, F.Cu at (103.2, 111.2)
- added U15: 74LVC1G07SE-7, MyParts:SC-88A_L2.0-W1.3-P0.65-LS2.1-BL, F.Cu at (104.1, 120.0)
- added U16: 74LVC1G07SE-7, MyParts:SC-88A_L2.0-W1.3-P0.65-LS2.1-BL, F.Cu at (107.6, 120.0)
- added U17: AP64501SP-13, MyParts:SOIC-8_L4.9-W3.9-P1.27-LS6.0-BL-EP-1, F.Cu at (53.1, 112.3)
- added U18: AP64501SP-13, MyParts:SOIC-8_L4.9-W3.9-P1.27-LS6.0-BL-EP-1, F.Cu at (76.9, 112.3)
- added U4: FSUSB42MUX, MyParts:MSOP-10_L3.0-W3.0-P0.50-LS5.0-BL, F.Cu at (115.6, 68.0)
- added U9: USB2514B-I/M2, MyParts:SQFN-36_L6.0-W6.0-P0.50-BL-EP, F.Cu at (109.4, 68.5)
- added USB1: Double layer DIP 90° black, MyParts:USB-A-TH_USB-M-51, F.Cu at (96.8, 55.0)
- added USBC1: TYPE-C-31-M-12, MyParts:USB-C_SMD-TYPE-C-31-M-12_1, F.Cu at (93.5, 73.4)
- added X2: X322524MOB4SI, MyParts:CRYSTAL-SMD_4P-L3.2-W2.5-BL, F.Cu at (101.8, 72.0)
- C23, C31, C35, C43: value 10uF -> GRM21BR6YA106KE43L
- C24, C30, C36, C42: value 1uF -> CL10A105KA8NNNC
- C25, C29: value 100nF -> CL05B104KO5NNNC
- L4: value Choke -> SMW2012B371BTE
- R18: value 5.1kΩ -> 100Ω
- R46: value 120Ω -> 100Ω; footprint PCM_JLCPCB:R_0805 -> PCM_JLCPCB:R_0402
- moved R18 71.4 mm to (82.1, 50.8), turned to 0 degrees
- moved R46 68.1 mm to (82.1, 54.5), turned to 0 degrees
Connections:
- net /ADDR0 renamed /SW1
- net /ADDR1 renamed /SW2
- net /ADDR2 renamed /SW3
- net /CONFIG_SW renamed /SW4
- net 1PPS_MCU renamed /1PPS_MCU
- net DIR1_MCU renamed /DIR1_MCU
- net DIR2_MCU renamed /DIR2_MCU
- net ENABLE1_MCU renamed /ENABLE1_MCU
- net ENABLE2_MCU renamed /ENABLE2_MCU
- net ENC1_A_MCU renamed /ENC1_A_MCU
- net ENC1_B_MCU renamed /ENC1_B_MCU
- net ENC1_Z_MCU renamed /ENC1_Z_MCU
- net ENC2_A_MCU renamed /ENC2_A_MCU
- net ENC2_B_MCU renamed /ENC2_B_MCU
- net ENC2_Z_MCU renamed /ENC2_Z_MCU
- net FAN_MCU renamed /FAN_MCU
- net FLASH_CS_MCU renamed /FLASH_CS_MCU
- net LIMIT1_SW1_MCU renamed /LIMIT1_SW1_MCU
- net LIMIT1_SW2_MCU renamed /LIMIT1_SW2_MCU
- net LIMIT2_SW1_MCU renamed /LIMIT2_SW1_MCU
- net LIMIT2_SW2_MCU renamed /LIMIT2_SW2_MCU
- net PUL1_MCU renamed /PUL1_MCU
- net PUL2_MCU renamed /PUL2_MCU
- net RS232_RX_MCU renamed /GPS_RX_MCU
- net RS232_TX_MCU renamed /GPS_TX_MCU
- net RS485_2_DE_MCU renamed /RS485_2_DE_MCU
- net RS485_2_RX_MCU renamed /RS485_2_RX_MCU
- net RS485_2_TX_MCU renamed /RS485_2_TX_MCU
- net SCL_MCU renamed /SCL_MCU
- net SDA_MCU renamed /SDA_MCU
- net SPI2_MISO_MCU renamed /SPI2_MISO_MCU
- net SPI2_MOSI_MCU renamed /SPI2_MOSI_MCU
- net SPI2_SCK_MCU renamed /SPI2_SCK_MCU
- net USER_SW_1_MCU renamed /USER_SW_1_MCU
- net USER_SW_2_MCU renamed /USER_SW_2_MCU
- net USER_SW_3_MCU renamed /USER_SW_3_MCU
- net USER_SW_4_MCU renamed /USER_SW_4_MCU
- R18 pad 1: Net-(U2-VIO) -> /CM4_TX
- R46 pad 1: /RS485/RS485_1_RX -> /CM4_RX
- U1 pad 58: RS485_1_DE_MCU -> unconnected-(U1-PB5-Pad58)
- U1 pad 59: RS485_1_TX_MCU -> /CM4_TX
- U1 pad 60: RS485_1_RX_MCU -> /CM4_RX
Routing:
- net /RS485/RS485_1_TX: track 32.5 -> 0.00 mm
- net /RS485/RS485_1_CHASSIS: track 31.5 -> 0.00 mm, vias 1 -> 0
- net /RS485/RS485_1_RX: track 25.6 -> 0.00 mm
- net Net-(U2-GISOIN): track 25.4 -> 0.00 mm, vias 2 -> 0
- net RS485_1_DE_MCU: track 25.1 -> 0.00 mm
- net RS485_1_TX_MCU: track 21.8 -> 0.00 mm
- net RS485_1_RX_MCU: track 20.0 -> 0.00 mm, vias 2 -> 0
- net Net-(U2-VISOIN): track 13.2 -> 0.00 mm
- net Net-(Module1A-GPIO5): track 11.6 -> 0.00 mm, vias 2 -> 0
- net Net-(U2-A): track 9.65 -> 0.00 mm
- net Net-(U2-VIO): track 8.98 -> 0.00 mm
- net RS485_1_GND: track 8.74 -> 0.00 mm, vias 54 -> 0
- net Net-(U2-VISOOUT): track 8.67 -> 0.00 mm
- net Net-(U2-VDD): track 8.60 -> 0.00 mm
- net GND: track 31.6 -> 25.4 mm, vias 465 -> 418
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- removed copper zone on B.Cu, net RS485_1_GND
- removed copper zone on F.Cu, net RS485_1_GND
- removed copper zone on In1.Cu, net RS485_1_GND
- removed copper zone on In2.Cu, net RS485_1_GND
Other:
- board text removed: "Chassis"
- board text removed: "N.C."
- board text removed: "RS485 In"
- board text removed: "RS485 Input"
- board text removed: "RS485 Passthrough"
- board text removed: "RS485 Passthru"
- board text removed: "Rx"
- board text removed: "Tx"

Commit message: Before adding CAN
Parts:
- removed C100, C95, C96, C97, C98, C99: 10uF 35V, MyParts:C0805
- removed C102, C106: 100nF, PCM_JLCPCB:C_0402
- removed C104: 56pF, MyParts:C0402
- removed C107: DNP, MyParts:C0402
- removed C110: 100uF 6.3V, Capacitor_Tantalum_SMD:CP_EIA-7343-31_Kemet-D
- removed the C46 at (126.5, 79.4)
- removed the C47 at (128.8, 80.2)
- removed the C47 at (42.1, 109.5)
- removed the C48 at (125.3, 104.9)
- removed the C48 at (42.1, 112.4)
- removed the C49 at (117.9, 105.5)
- removed the C49 at (42.1, 115.4)
- removed the C50 at (119.9, 105.5)
- removed the C50 at (42.1, 118.3)
- removed the C51 at (121.7, 105.6)
- removed the C52 at (129.1, 109.7)
- removed the C53 at (124.6, 102.8)
- removed the C54 at (123.4, 107.7)
- removed the DC1 at (126.4, 96.2)
- removed the F1 at (132.7, 81.0)
- removed L11: 3.3uH, MyParts:IND-SMD_L3.0-W3.0-1
- removed L15: SRN6045TA-3R3Y, MyParts:IND-SMD_L6.0-W6.0
- removed the Q1 at (120.2, 75.3)
- removed the Q2 at (127.5, 63.8)
- removed the Q4 at (120.2, 79.7)
- removed the R20 at (126.5, 74.4)
- removed the R21 at (129.0, 108.0)
- removed the R22 at (51.2, 125.2)
- removed the R22 at (128.7, 106.4)
- removed the R23 at (125.9, 108.0)
- removed the R55 at (58.4, 130.9)
- removed the R63 at (51.2, 127.3)
- removed the R65 at (51.2, 129.5)
- removed the SW2 at (132.6, 71.4)
- removed the TP2 at (119.3, 113.8)
- removed the TP3 at (136.8, 100.1)
- removed the U17 at (53.1, 112.3)
- removed the U4 at (123.7, 105.7)
- added C56: 100nF, PCM_JLCPCB:C_0402, F.Cu at (131.1, 102.8)
- added C57: 10uF, PCM_JLCPCB:C_0805, F.Cu at (123.1, 100.4)
- added C58: 10uF, PCM_JLCPCB:C_0805, F.Cu at (123.1, 103.5)
- added C59: 100nF, PCM_JLCPCB:C_0603, F.Cu at (127.3, 107.5)
- added C60: 22pF, PCM_JLCPCB:C_0603, F.Cu at (127.3, 109.8)
- added C61: 22uF, PCM_JLCPCB:C_0805, F.Cu at (123.1, 106.5)
- added C62: 1uF, PCM_JLCPCB:C_0402, F.Cu at (131.1, 104.6)
- added C87: 15pF, PCM_JLCPCB:C_0402, F.Cu at (129.9, 144.3)
- added C88: 15pF, PCM_JLCPCB:C_0402, F.Cu at (129.9, 146.1)
- added L8: 3.3uH, MyParts:IND-SMD_L3.0-W3.0-1, F.Cu at (127.5, 104.1)
- added Q5: AO3400A, MyParts:SOT-23-3_L2.9-W1.3-P1.90-LS2.4-BR, F.Cu at (168.9, 51.8)
- added R72: 976kΩ, Resistor_SMD:R_0805_2012Metric, F.Cu at (127.6, 100.4)
- added R73: 100kΩ, PCM_JLCPCB:R_0603, F.Cu at (131.0, 107.5)
- added R74: 220kΩ, PCM_JLCPCB:R_0603, F.Cu at (131.0, 109.8)
- added R81: 2.2kΩ, MyParts:R0402, F.Cu at (130.0, 148.1)
- added U7: MP2322GQH-Z, MyParts:QFN-8_L2.0-W1.5-P0.50-BL, F.Cu at (122.7, 109.5)
- moved LED3 152.0 mm to (-68.4, 62.0)
- moved R69 152.0 mm to (-69.8, 57.6)
- moved R70 152.0 mm to (-69.8, 55.7)
- moved R71 152.0 mm to (-69.8, 59.4)
- moved C81 142.8 mm to (-34.7, 57.6)
- moved C82 142.8 mm to (-32.2, 70.2)
- moved C83 142.8 mm to (-34.7, 45.8)
- moved C84 142.8 mm to (-34.7, 48.7)
- moved C85 142.8 mm to (-34.7, 51.7)
- moved C86 142.8 mm to (-34.7, 54.6)
- moved U11 142.8 mm to (-41.3, 71.1)
- moved U12 142.8 mm to (-27.0, 54.8)
- moved U14 142.8 mm to (-33.3, 62.9)
- moved X2 142.8 mm to (-40.9, 66.4)
- moved C85 142.8 mm to (-27.7, 45.2)
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- renumbered C18 to C12, C66 to C18, C70 to C19, C23 to C20, C24 to C21, C25 to C22, C29 to C23, C30 to C24, C31 to C25, C35 to C26, C36 to C27, C37 to C28, C41 to C29, C42 to C30, C43 to C31, C45 to C32, C55 to C33, C56 to C34, C57 to C35, C58 to C36, C59 to C37, C60 to C38, C61 to C39, C63 to C40, C19 to C41, C62 to C42, C64 to C43, C65 to C44, C12 to C45, C67 to C46, C68 to C47, C69 to C48, C71 to C49, C76 to C50, C72 to C51, C73 to C52, C74 to C53, C75 to C54, C51 to C55, C78 to C63, C115 to C64, C52 to C65, C53 to C66, C54 to C67, C77 to C68, C117 to C69, C83 to C70, C101 to C71, C105 to C71, C103 to C72, C111 to C73, C112 to C74, C113 to C75, C114 to C76, C116 to C77, C81 to C78, C82 to C79, C46 to C80, C109 to C81, C80 to C82, C92 to C83, C93 to C84, C94 to C85, C108 to C86, CN14 to CN10, CN5 to CN3, CN7 to CN4, CN8 to CN5, CN9 to CN6, CN17 to CN7, CN12 to CN8, CN13 to CN9, D20 to D10, D30 to D11, D29 to D12, D25 to D13, D26 to D14, D17 to D15, D6 to D17, D35 to D18, D7 to D19, D8 to D20, D9 to D21, D10 to D22, D11 to D23, D33 to D24, D34 to D25, D21 to D26, D22 to D27, D23 to D28, D12 to D29, D13 to D30, D14 to D31, D15 to D32, D31 to D6, D32 to D7, D18 to D8, D19 to D9, F4 to F1, F5 to F2, F1 to F4, H3 to H1, H4 to H2, H1 to H3, H5 to H4, H6 to H5, J3 to J2, L2 to L1, L4 to L2, L6 to L3, L8 to L4, L10 to L5, L13 to L6, L14 to L7, L16 to L9, M1 to M2, M1 to M3, M1 to M4, Q5 to Q1, Q6 to Q2, Q11 to Q3, Q12 to Q4, Q7 to Q6, Q8 to Q7, R70 to R1, R14 to R10, R57 to R11, R15 to R12, R73 to R13, R76 to R14, R58 to R15, R59 to R17, R72 to R18, R75 to R19, R71 to R20, R74 to R21, R17 to R22, R19 to R23, R21 to R24, R24 to R25, R25 to R26, R26 to R27, R64 to R28, R27 to R29, R66 to R30, R68 to R31, R28 to R32, R67 to R33, R69 to R34, R29 to R35, R30 to R36, R11 to R37, R10 to R38, R31 to R39, R1 to R40, R12 to R41, R32 to R42, R33 to R43, R34 to R44, R35 to R45, R36 to R46, R37 to R47, R38 to R48, R43 to R49, R60 to R50, R79 to R51, R82 to R52, R44 to R53, R61 to R54, R45 to R55, R62 to R56, R78 to R57, R81 to R58, R77 to R59, R80 to R60, R47 to R61, R48 to R62, R49 to R63, R50 to R64, R51 to R65, R52 to R66, R53 to R67, R54 to R68, R20 to R69, R18 to R70, R46 to R71, R56 to R75, R40 to R76, R39 to R77, R13 to R78, R42 to R79, R41 to R80, R23 to R82, R89 to R83, R90 to R84, R88 to R85, R87 to R86, R83 to R87, R84 to R88, R85 to R89, R86 to R90, R92 to R91, R91 to R92, SW4 to SW2, TP4 to TP1, TP5 to TP2, TP1 to TP3, TP2 to TP4, TP7 to TP5, TP14 to TP6, TP11 to TP7, TP13 to TP8, TP12 to TP9, U12 to U10, U13 to U11, U10 to U12, U4 to U13, U9 to U14, U14 to U17, U3 to U2, U5 to U3, U6 to U4, U7 to U5, U8 to U6, U18 to U8, U11 to U9
Connections:
- H4 pad 1: /RCM4/PWM0 -> /RCM4/I2C1_SDA
- H5 pad 1: /RCM4/PWM1 -> /RCM4/I2C1_SCL
- U14 pad 32: Net-(U9-XTALOUT) -> Net-(U14-XTALOUT)
- U14 pad 33: Net-(U9-XTALIN/CLKIN) -> Net-(U14-XTALIN/CLKIN)
- USBC1 pad A4B9: /RCM4/usb/VBUS -> Net-(R81-Pad2)
- USBC1 pad B4A9: /RCM4/usb/VBUS -> Net-(R81-Pad2)
- X2 pad 1: Net-(U9-XTALIN/CLKIN) -> Net-(U14-XTALIN/CLKIN)
- X2 pad 3: Net-(U9-XTALOUT) -> Net-(U14-XTALOUT)
Routing:
- net /USER_SW_4_MCU: track 64.3 -> 4.97 mm, vias 2 -> 1
- net /FAN_MCU: track 49.1 -> 3.65 mm, vias 2 -> 0
- net /ENC1_A_MCU: track 39.0 -> 3.97 mm
- net /ENC2_A_MCU: track 46.2 -> 11.1 mm
- net /ENC2_B_MCU: track 47.6 -> 13.4 mm
- net /ENC1_B_MCU: track 36.3 -> 3.00 mm
- net /USER_SW_1_MCU: track 70.6 -> 38.1 mm
- net /ENC1_Z_MCU: track 35.6 -> 3.65 mm
- net /USER_SW_2_MCU: track 51.2 -> 19.3 mm, vias 2 -> 1
- net /USER_SW_3_MCU: track 52.2 -> 20.5 mm, vias 2 -> 1
- net /1PPS_MCU: track 38.4 -> 7.09 mm
- net /ENC2_Z_MCU: track 46.4 -> 15.5 mm
- net /GPS_TX_MCU: track 46.9 -> 19.2 mm
- net /FLASH_CS_MCU: track 27.3 -> 1.73 mm
- net /LIMIT1_SW1_MCU: track 28.4 -> 3.34 mm
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- removed copper zone on F.Cu, net 12V
- removed copper zone on In2.Cu, net 12V
- removed copper zone on F.Cu, net 3V3
- removed copper zone on In2.Cu, net 3V3
- removed copper zone on B.Cu, net GND
- removed copper zone on F.Cu, net GND
- removed copper zone on In1.Cu, net GND
- removed copper zone on F.Cu, net Net-(U4-SW)
Other:
- board size 100 x 100 mm -> 130 x 100 mm
- board text removed: "12V IN"
- board text removed: "12V IN - 1Amp Center 12V"
- board text removed: "3.3V"
- board text removed: "ADDR0"
- board text removed: "ADDR1"
- board text removed: "ADDR2"
- board text removed: "Axis Commander V1.1 JRSeti www.jrseti.com"
- board text removed: "CONFIG"
- board text removed: "Fan"
- board text removed: "OFF"
- board text removed: "ON"
- board text removed: "RS485 PINS Rx-Tx-Gnd-Chassis"

Commit message: More mods
Parts:
- added C89: 4.7uF, PCM_JLCPCB:C_1206, F.Cu at (234.5, 48.2)
- added C90: 4.7uF, PCM_JLCPCB:C_1206, F.Cu at (234.5, 51.5)
- added C91: C43Q1103K40C80F, MyParts:CAP-TH_L13.0-W6.0-P10.00-D1.2, F.Cu at (231.5, 35.4)
- added C92: 100nF, PCM_JLCPCB:C_0402, F.Cu at (245.7, 32.7)
- added C93: 100nF, PCM_JLCPCB:C_0402, F.Cu at (245.7, 34.6)
- added C94: 4.7uF, PCM_JLCPCB:C_0805, F.Cu at (233.9, 54.7)
- added C95: 10uF, PCM_JLCPCB:C_0805, F.Cu at (233.9, 57.8)
- added C96: 4.7nF, PCM_JLCPCB:C_0603, F.Cu at (249.1, 37.4)
- added CN11: KF2EDGR-2.54-4P, MyParts:CONN-TH_4P-P2.54_KF2EDGR-2.54-4P, F.Cu at (245.0, 40.9)
- added D33: H24VND3BA, PCM_JLCPCB:D_SOD-323, F.Cu at (249.5, 52.1)
- added D34: H24VND3BA, PCM_JLCPCB:D_SOD-323, F.Cu at (249.5, 55.0)
- added D35: SMAJ14A, PCM_JLCPCB:D_SMA, F.Cu at (228.5, 64.5)
- added D36: SMF6.0A, PCM_JLCPCB:D_SOD-123FL, F.Cu at (256.5, 50.5)
- added D37: TPESD0402G05V, MyParts:D0402-BI, F.Cu at (255.4, 41.4)
- added D38: TPESD0402G05V, MyParts:D0402-BI, F.Cu at (255.4, 43.5)
- added D39: TPESD0402G05V, MyParts:D0402-BI, F.Cu at (255.4, 45.7)
- added D40: TPESD0402G05V, MyParts:D0402-BI, F.Cu at (255.4, 32.9)
- added D41: TPESD0402G05V, MyParts:D0402-BI, F.Cu at (255.4, 35.1)
- added D42: TPESD0402G05V, MyParts:D0402-BI, F.Cu at (255.4, 37.2)
- added D43: PESD0402-140, MyParts:D0402-BI, F.Cu at (255.4, 63.7)
- added L10: CYA0630-10UH, MyParts:IND-SMD_L7.2-W6.6_GPSR07X0, F.Cu at (242.8, 54.5)
- added L11: SMW2012B371BTE, MyParts:FILTER-SMD_4P-L2.0-W1.2-BL, F.Cu at (240.1, 36.9)
- added R94: 10kΩ, PCM_JLCPCB:R_0402, F.Cu at (245.7, 36.4)
- added R95: 180Ω, PCM_JLCPCB:R_1206, F.Cu at (241.5, 33.5)
- added R96: 56Ω, PCM_JLCPCB:R_0603, F.Cu at (249.0, 32.9)
- added R97: 56Ω, PCM_JLCPCB:R_0603, F.Cu at (249.0, 35.2)
- added R98: 100Ω, PCM_JLCPCB:R_0402, F.Cu at (255.1, 57.9)
- added R99: 10kΩ, PCM_JLCPCB:R_0402, F.Cu at (255.1, 59.7)
- added U18: B1205S-1WR3_C5365649, MyParts:PWRM-TH_4P-L11.5-W6.0-P2.54_B1503S, F.Cu at (231.9, 45.1)
- added U20: ISO1042DWVR, MyParts:SOIC-8_L7.5-W5.9-P1.27-LS11.5-BL, F.Cu at (228.1, 53.4)
- added U21: TPD4EUSB30DQAR-N, MyParts:DFN-10_L2.5-W1.0-P0.50-BL-A, F.Cu at (255.8, 53.4)
Connections:
- Module1 pad 30: unconnected-(Module1A-GPIO6-Pad30) -> Net-(Module1A-GPIO6)
- R3 pad 1: Net-(U1-PA12) -> /STATUS_LED
- U1 pad 45: /SW1 -> /CAN_RX
- U1 pad 46: Net-(U1-PA12) -> /CAN_TX
- U1 pad 52: /RS485_2_TX_MCU -> /SW1
- U1 pad 53: /RS485_2_RX_MCU -> /STATUS_LED
- U1 pad 55: /RS485_2_DE_MCU -> /MCU_nIRQ
Routing:
- net /MCU_nIRQ: track 0.00 -> 8.21 mm, vias 0 -> 1
- net /RS485_2_DE_MCU: track 47.8 -> 39.6 mm, vias 1 -> 0
- net /SW1: track 2.30 -> 5.40 mm
- net /RS485_2_TX_MCU: track 35.3 -> 32.2 mm
- net /STATUS_LED: track 0.00 -> 2.15 mm
- net /RS485_2_RX_MCU: track 40.7 -> 38.5 mm

Commit message: Part positioning of PWR, USB, Ethernet
Parts:
- removed C29: 10nF, MyParts:C0402
- removed C30: CL10A105KA8NNNC, MyParts:C0603
- removed C31: GRM21BR6YA106KE43L, MyParts:C0805
- removed C32: 10nF, MyParts:CAP-TH_L13.0-W6.0-P10.00-D1.2
- removed the C71 at (-80.1, 134.8)
- removed the C85 at (-27.7, 45.2)
- removed the C86 at (-27.7, 47.1)
- removed CN3: KF2EDGR-2.54-4P, MyParts:CONN-TH_4P-P2.54_KF2EDGR-2.54-4P
- removed D11: SM712_SOT23, Package_TO_SOT_SMD:SOT-23
- removed D12: SMAJ15CA, Diode_SMD:D_SMA
- removed L1, L3, L4, L5: BLM15EX331SN1D, MyParts:L0402
- removed L2: SMW2012B371BTE, MyParts:FILTER-SMD_4P-L2.0-W1.2-BL
- removed R22: 120Ω, PCM_JLCPCB:R_0805
- removed R23: 5.1kΩ, PCM_JLCPCB:R_0402
- removed TP7: RH-5016, MyParts:TESTPOINT-SMD_L3.0-W2.0
- removed U2: ISOW1432BDFMR, MyParts:SOIC-20_L12.8-W7.5-P1.27-LS10.3-BL
- C20: value GRM21BR6YA106KE43L -> 220uF; footprint MyParts:C0805 -> MyParts:CAP-SMD_BD6.3-L6.6-W6.6-FD
- C21: value CL10A105KA8NNNC -> 10uF 10V; footprint MyParts:C0603 -> MyParts:C0805
- C22: value CL05B104KO5NNNC -> 10uF 10V; footprint MyParts:C0402 -> MyParts:C0805
- C23: value CL05B104KO5NNNC -> 100nF; footprint MyParts:C0402 -> PCM_JLCPCB:C_0402
- C24, C27: value CL10A105KA8NNNC -> 100n; footprint MyParts:C0603 -> Capacitor_SMD:C_0402_1005Metric
- C25, C26: value GRM21BR6YA106KE43L -> 100n; footprint MyParts:C0805 -> Capacitor_SMD:C_0402_1005Metric
- C28: value 10nF -> 100n; footprint MyParts:C0402 -> Capacitor_SMD:C_0402_1005Metric
- C91: value C43Q1103K40C80F -> 10nF, 300V
- D33, D34: value H24VND3BA -> 7A 50V
- moved C63 238.9 mm to (152.6, 59.3), turned to 90 degrees
- moved C71 236.7 mm to (148.0, 55.9), turned to -90 degrees
- moved F4 231.5 mm to (156.1, 57.5), turned to -90 degrees
- moved C68 231.0 mm to (147.3, 65.9), turned to -90 degrees
- moved C67 228.0 mm to (145.1, 65.9), turned to -90 degrees
- moved C74 227.6 mm to (148.0, 60.1), turned to 90 degrees
- moved C75 226.6 mm to (145.9, 60.1), turned to 90 degrees
- moved C76 225.6 mm to (143.8, 60.1), turned to 90 degrees
- moved C66 225.2 mm to (143.1, 65.9), turned to -90 degrees
- moved C72 225.1 mm to (145.9, 55.9), turned to -90 degrees
- moved C73 224.0 mm to (143.8, 55.9), turned to -90 degrees
- moved TP8 223.0 mm to (156.1, 62.8)
- moved C65 222.4 mm to (141.0, 65.9), turned to -90 degrees
- moved C77 221.9 mm to (140.0, 54.2), turned to 180 degrees
- moved R78 218.5 mm to (136.3, 53.8)
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Connections:
- C20 pad 1: GND -> 12V
- C20 pad 2: Net-(U2-VIO) -> GND
- C21 pad 1: Net-(U2-VIO) -> GND
- C21 pad 2: GND -> 3V3_CM4
- C22 pad 1: Net-(U2-VIO) -> GND
- C22 pad 2: GND -> 3V3_CM4
- C23 pad 1: Net-(U2-VISOIN) -> 3V3_CM4
- C23 pad 2: RS485_2_GND -> GND
- C24 pad 1: Net-(U2-VISOIN) -> 3V3_CM4
- C24 pad 2: RS485_2_GND -> GND
- C25 pad 1: RS485_2_GND -> 3V3_CM4
- C25 pad 2: Net-(U2-VISOIN) -> GND
- C26 pad 1: GND -> 3V3_CM4
- C26 pad 2: Net-(U2-VDD) -> GND
- C27 pad 1: Net-(U2-VDD) -> 3V3_CM4
- C28 pad 1: Net-(U2-VDD) -> 3V3_CM4
Routing:
- net (no net): track 0.00 -> 67.2 mm, vias 0 -> 4
- net /RS485_2_DE_MCU: track 39.6 -> 0.00 mm
- net /RS485_2_RX_MCU: track 38.5 -> 0.00 mm
- net /RS485_2_TX_MCU: track 32.2 -> 0.00 mm
- net Net-(U2-GISOIN): track 24.4 -> 0.00 mm, vias 2 -> 0
- net /RS485/RS485_2_CHASSIS: track 22.7 -> 0.00 mm
- net /RS485/RS485_2_RX: track 14.4 -> 0.00 mm
- net /RS485/RS485_2_TX: track 13.7 -> 0.00 mm
- net Net-(U2-VISOIN): track 12.9 -> 0.00 mm
- net Net-(U2-EN/FLT): track 11.8 -> 0.00 mm, vias 2 -> 0
- net Net-(U2-A): track 10.5 -> 0.00 mm
- net Net-(U2-VIO): track 9.72 -> 0.00 mm
- net 3V3: track 75.0 -> 84.1 mm, vias 47 -> 52
- net Net-(U2-VDD): track 9.09 -> 0.00 mm
- net Net-(U2-VISOOUT): track 8.06 -> 0.00 mm
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- added copper zone on B.Cu, net (none)
- added copper zone on F.Cu, net (none)
- added copper zone on In1.Cu, net (none)
- added copper zone on In2.Cu, net (none)
- added copper zone on F.Cu, net 3V3
- added copper zone on F.Cu, net Net-(U7-SW)
- removed copper zone on B.Cu, net RS485_2_GND
- removed copper zone on F.Cu, net RS485_2_GND
- removed copper zone on In1.Cu, net RS485_2_GND
- removed copper zone on In2.Cu, net RS485_2_GND
Other:
- board size 130 x 100 mm -> 140 x 100 mm
- board text added: "CAN Isolation"
- board text removed: "C34"
- board text removed: "RS485 Isolation"
- board text removed: "RS485 Leader"
