File: kicad/rcm_dish_controller.kicad_pcb (KiCad board)
At the start: 4 copper layers, 140 x 100 mm, 310 parts, among them CN1 KF2EDGR-2.54-9P, CN10 KF2EDGR-2.54-6P, CN11 KF2EDGR-2.54-4P, CN2 KF2EDGR-2.54-6P, CN4 SM04B-SRSS-TB (LF)(SN), CN5 SM04B-SRSS-TB (LF)(SN), CN6 KF2EDGR-2.54-2P, CN7 SMA-KWE_C7498154, CN8 KF2EDGR-2.54-9P, CN9 KF2EDGR-2.54-6P, J1 Conn_ST_STDC14, J2 Header-Male-2.54_2x3, M1 MountingHole_2.7mm_M2.5_ISO14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, M2 MountingHole_2.7mm_M2.5_ISO14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, M3 MountingHole_2.7mm_M2.5_ISO14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, M4 MountingHole_2.7mm_M2.5_ISO14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, Q1 BSS138, Q2 BSS138, Q3 DMP3013SFV-7, Q4 DMP3013SFV-7, Q5 AO3400A, Q6 BSS138, Q7 BSS138, SW1 DSHP04TSGER, SW2 SS-12F49-G050, U1 STM32G474RET6, U10 TPD4EUSB30DQAR, U11 AP22653W6-7, U12 TPD4EUSB30DQAR-N, U13 FSUSB42MUX, U14 USB2514B-I/M2, U15 74LVC1G07SE-7, U16 74LVC1G07SE-7, U17 2541WV-2X12P, U18 B1205S-1WR3_C5365649, U20 ISO1042DWVR, U21 TPD4EUSB30DQAR-N, U3 LTC4311ISC6#TRPBF, U4 LM75BIMX-3/NOPB, U5 W25Q32JVSSIQ_C179173, U6 MAX-M10S-00B, U7 MP2322GQH-Z, U8 AP64501SP-13, U9 TPD4EUSB30DQAR, X1 NX2016SA-16MHZ-EXS00A-CS07826, X2 X322524MOB4SI

Commit message: CAN looks complete in schematic
Parts:
- removed C93: 100nF, PCM_JLCPCB:C_0402
- removed C94: 4.7uF, PCM_JLCPCB:C_0805
- removed C95: 10uF, PCM_JLCPCB:C_0805
- removed C96: 4.7nF, PCM_JLCPCB:C_0603
- removed CN11: KF2EDGR-2.54-4P, MyParts:CONN-TH_4P-P2.54_KF2EDGR-2.54-4P
- removed D33, D34: 7A 50V, PCM_JLCPCB:D_SOD-323
- removed L10: CYA0630-10UH, MyParts:IND-SMD_L7.2-W6.6_GPSR07X0
- removed L11: SMW2012B371BTE, MyParts:FILTER-SMD_4P-L2.0-W1.2-BL
- removed R96, R97: 56Ω, PCM_JLCPCB:R_0603
- removed U18: B1205S-1WR3_C5365649, MyParts:PWRM-TH_4P-L11.5-W6.0-P2.54_B1503S
- removed U20: ISO1042DWVR, MyParts:SOIC-8_L7.5-W5.9-P1.27-LS11.5-BL
- added C29: 100nF, MyParts:C0402, F.Cu at (241.0, 47.0)
- added C30: 10uF, MyParts:C0805, F.Cu at (236.6, 53.9)
- added C31: 10nF, MyParts:C0603, F.Cu at (244.4, 47.3)
- added C32: 100nF, MyParts:C0402, F.Cu at (241.0, 49.2)
- added C97: 4.7nF, MyParts:C0805, F.Cu at (236.6, 56.8)
- added CN3: KF2EDGR-2.54-3P, MyParts:CONN-TH_3P-P2.54_KF2EDGR-2.54-3P, F.Cu at (188.5, 41.5)
- added D12: NUP2105LT1G, MyParts:SOT-23-3_L2.9-W1.3-P1.90-LS2.4-BL-2, F.Cu at (227.3, 58.3)
- added J3: Header-Male-2.54_2x2, MyParts:HDR-TH_4P-P2.54-V-M-R2-C2-S2.54-1, F.Cu at (232.2, 81.7)
- added J4: Header-Male-2.54_1x3, MyParts:HDR-TH_3P-P2.54-V-M-1, F.Cu at (233.4, 74.7)
- added L1: BLM15HD182SN1D, MyParts:L0402, F.Cu at (231.1, 57.2)
- added L12: 370R@100MHz, MyParts:FILTER-SMD_4P-L2.0-W1.2-BL, F.Cu at (243.8, 50.4)
- added L2: BLM15HD182SN1D, MyParts:L0402, F.Cu at (231.1, 59.4)
- added R22: 60.4Ω, MyParts:R0805, F.Cu at (241.4, 53.9)
- added R23: 60.4Ω, MyParts:R0805, F.Cu at (241.4, 56.9)
- added U2: ADM3057EBRWZ-RL, MyParts:SOIC-20_L13.0-W7.6-P1.27-LS10.3-BL, F.Cu at (188.5, 53.0)
- C89: value 4.7uF -> 100nF; footprint PCM_JLCPCB:C_1206 -> MyParts:C0402
- C90: value 4.7uF -> 10uF; footprint PCM_JLCPCB:C_1206 -> MyParts:C0805
- C91: value 10nF, 300V -> 10nF; footprint MyParts:CAP-TH_L13.0-W6.0-P10.00-D1.2 -> MyParts:C0603
- C92: footprint PCM_JLCPCB:C_0402 -> MyParts:C0402
- LED3: value XL-0805QBC -> RED
- LED4: value LTST-S270KGKT -> GREEN; footprint MyParts:LED-SMD_L1.7-W0.6-RD -> MyParts:LED0805-R-RD
- R94: value 10kΩ -> 0Ω; footprint PCM_JLCPCB:R_0402 -> MyParts:R0402
- R95: value 180Ω -> 47KΩ; footprint PCM_JLCPCB:R_1206 -> MyParts:R0805
- moved R98 137.4 mm to (118.2, 69.7)
- moved R99 134.7 mm to (120.8, 69.7), turned to 180 degrees
- moved D37 130.2 mm to (151.2, 119.5), turned to 90 degrees
- moved D38 124.8 mm to (156.3, 119.5), turned to 90 degrees
- moved D39 119.6 mm to (161.3, 119.5), turned to 90 degrees
- moved R93 106.8 mm to (84.0, 41.3)
- moved R92 103.4 mm to (80.7, 41.3), turned to 180 degrees
- moved D41 103.1 mm to (196.3, 119.5), turned to 90 degrees
- moved D42 98.4 mm to (201.5, 119.5), turned to 90 degrees
- moved LED4 84.3 mm to (88.2, 60.6), turned to 180 degrees
- moved U16 84.1 mm to (88.3, 64.6)
- moved U15 84.0 mm to (85.8, 64.7), turned to 180 degrees
- moved R91 83.5 mm to (88.3, 62.4)
- moved R70 74.8 mm to (149.1, 85.0)
- moved R71 74.3 mm to (152.2, 85.0)
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Connections:
- C89 pad 1: 12V -> GND
- C89 pad 2: GND -> 5V
- C90 pad 1: Net-(U18-+VIN) -> GND
- C90 pad 2: GND -> 5V
- C91 pad 2: CAN_GND -> 3V3
- C92 pad 1: 3V3 -> GND
- C92 pad 2: GND -> 3V3
- LED4 pad 1: Net-(LED4-K) -> 3V3_CM4
- LED4 pad 2: 3V3_CM4 -> Net-(LED4-K)
- R94 pad 1: 3V3 -> /CAN_RX
- R94 pad 2: /CAN_TX -> Net-(U2-RXD)
- R95 pad 1: /CAN/CAN_5V -> CAN_GND
- R95 pad 2: CAN_GND -> Net-(U2-RS)
Routing:
- net (no net): track 67.2 -> 48.2 mm, vias 4 -> 0
- net 12V: track 102.7 -> 98.1 mm
- net Net-(D18-K): track 1.61 -> 4.10 mm
- net Net-(D41-K): track 2.14 -> 4.34 mm
- net 3V3: track 84.1 -> 82.0 mm, vias 52 -> 50
- net Net-(D42-K): track 2.33 -> 4.47 mm
- net Net-(D40-K): track 2.13 -> 4.23 mm
- net Net-(D38-K): track 2.23 -> 4.32 mm
- net Net-(D39-K): track 2.23 -> 4.29 mm
- net Net-(D37-K): track 2.55 -> 4.28 mm
- net /FAN_MCU: track 3.65 -> 2.35 mm
- net GND: vias 274 -> 255
- removed copper zone on B.Cu, net (none)
- removed copper zone on In1.Cu, net (none)
- removed copper zone on In2.Cu, net (none)
Other:
- board text added: "CM4 Activity"
- board text added: "CM4 Power"
- board text added: "Ethernet"
- board text added: "OFF"
- board text added: "ON"
- board text added: "Raspberry Pi Compute Module 4"

Commit message: Add CAN JR45 - still working on it
Parts:
- removed the H3 at (80.6, 67.7)
- moved J3 153.2 mm to (80.4, 67.9), turned to -90 degrees
- moved J4 69.1 mm to (178.3, 38.5), turned to 180 degrees
- moved R96 66.4 mm to (176.5, 43.2), turned to 90 degrees
- moved C89 65.2 mm to (187.1, 60.2), turned to 180 degrees
- moved R97 63.7 mm to (178.6, 43.2), turned to 90 degrees
- moved R94 62.3 mm to (189.1, 60.2), turned to 180 degrees
- moved C90 60.3 mm to (187.4, 61.7), turned to 180 degrees
- moved C93 59.8 mm to (177.5, 47.4), turned to -90 degrees
- moved C88 57.6 mm to (183.4, 47.0)
- moved C91 56.0 mm to (188.4, 45.5), turned to 180 degrees
- moved C87 55.0 mm to (182.4, 44.2)
- moved R95 54.9 mm to (194.1, 46.1), turned to 180 degrees
- moved L7 53.0 mm to (191.0, 46.1)
- moved C92 52.5 mm to (188.5, 47.0), turned to 180 degrees
- moved L6 51.1 mm to (181.6, 46.4), turned to 90 degrees
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- renumbered C33 to C21, C34 to C22, C35 to C23, C36 to C24, C37 to C25, C38 to C26, C39 to C27, C40 to C28, C41 to C29, C42 to C30, C43 to C31, C44 to C32, C45 to C33, C46 to C34, C47 to C35, C48 to C36, C49 to C37, C50 to C38, C51 to C39, C52 to C40, C53 to C41, C54 to C42, C55 to C43, C56 to C44, C57 to C45, C58 to C46, C59 to C47, C60 to C48, C61 to C49, C62 to C50, C63 to C51, C64 to C52, C65 to C53, C66 to C54, C67 to C55, C68 to C56, C69 to C57, C70 to C58, C71 to C59, C72 to C60, C73 to C61, C74 to C62, C75 to C63, C76 to C64, C77 to C65, C78 to C66, C79 to C67, C80 to C68, C81 to C69, C82 to C70, C83 to C71, C84 to C72, C85 to C73, C86 to C74, C87 to C75, C88 to C76, C21 to C77, C22 to C78, C23 to C79, C24 to C80, C25 to C81, C26 to C82, C27 to C83, C28 to C84, C90 to C85, C89 to C86, C30 to C87, C29 to C88, C92 to C89, C91 to C90, C31 to C91, C32 to C92, C97 to C93, CN3 to CN10, CN4 to CN3, CN5 to CN4, CN6 to CN5, CN7 to CN6, CN8 to CN7, CN9 to CN8, CN10 to CN9, D37 to D10, D8 to D11, D9 to D12, D10 to D13, D35 to D14, D13 to D15, D14 to D16, D15 to D17, D16 to D18, D17 to D19, D18 to D20, D43 to D21, D19 to D22, D20 to D23, D21 to D24, D22 to D25, D23 to D26, D24 to D27, D25 to D28, D42 to D29, D41 to D30, D40 to D31, D26 to D32, D27 to D33, D28 to D34, D29 to D35, D30 to D36, D31 to D37, D32 to D38, D36 to D39, D12 to D40, D39 to D8, D38 to D9, H4 to H3, H5 to H4, J4 to J3, J3 to J4, L6 to L1, L7 to L2, L8 to L3, L9 to L4, L1 to L5, L2 to L6, L12 to L7, R24 to R22, R25 to R23, R26 to R24, R27 to R25, R28 to R26, R29 to R27, R30 to R28, R31 to R29, R32 to R30, R33 to R31, R34 to R32, R35 to R33, R36 to R34, R37 to R35, R38 to R36, R39 to R37, R40 to R38, R41 to R39, R42 to R40, R43 to R41, R44 to R42, R45 to R43, R46 to R44, R47 to R45, R48 to R46, R49 to R47, R50 to R48, R51 to R49, R52 to R50, R53 to R51, R54 to R52, R55 to R53, R56 to R54, R57 to R55, R58 to R56, R59 to R57, R60 to R58, R61 to R59, R62 to R60, R63 to R61, R64 to R62, R65 to R63, R66 to R64, R67 to R65, R68 to R66, R69 to R67, R99 to R68, R98 to R69, R23 to R96, R22 to R97, TP8 to TP7, TP9 to TP8, U11 to U10, U12 to U11, U13 to U12, U14 to U13, U21 to U14, U2 to U18, U3 to U2, U4 to U3, U5 to U4, U6 to U5, U7 to U6, U8 to U7, U9 to U8, U10 to U9
Connections:
- net Net-(C97-Pad1) renamed /CAN/CANHL_C
- net Net-(CN1-Pad1) renamed /Axis Control - 1/12VENC
- net Net-(CN8-Pad1) renamed /Axis Control - 2/12VENC
- net Net-(D14-K) renamed /I2C and EEPROM/SDA
- net Net-(D26-K) renamed /Axis Control - 2/PUL2-
- net Net-(D27-K) renamed /Axis Control - 2/DIR2-
- net Net-(D28-K) renamed /Axis Control - 2/ENABLE2-
- net Net-(D40-K) renamed /Axis Control - 2/PUL2+
- net Net-(D41-K) renamed /Axis Control - 2/DIR2+
- net Net-(D42-K) renamed /Axis Control - 2/ENABLE2+
- net Net-(J3-Pad2) renamed /CAN/CANH_T
- net Net-(J3-Pad4) renamed /CAN/CANL_T
- net Net-(U2-CANH) renamed /CAN/CH
- net Net-(U2-CANL) renamed /CAN/CL
- net Net-(U2-RS) renamed /CAN/RS
- net Net-(U2-RXD) renamed /CAN/RXD
- net Net-(U4-OS) renamed /I2C and EEPROM/OS
- C29 pad 1: Net-(U6-VCC) (its old number) -> /GPS/VCC
- C30 pad 1: Net-(U6-VCC) (its old number) -> /GPS/VCC
- C31 pad 1: Net-(U6-VCC) (its old number) -> /GPS/VCC
- CN10 pad 1: /CAN/CANH -> /CAN/CANL
- CN10 pad 2: /CAN/CANL -> /CAN/CANH
- CN3 pad 4: Net-(D13-K) (its old number) -> /I2C and EEPROM/SCL
- D15 pad 1: Net-(D13-K) (its old number) -> /I2C and EEPROM/SCL
- L1 pad 2: Net-(U6-VCC) (its old number) -> /GPS/VCC
- R28 pad 2: Net-(D13-K) (its old number) -> /I2C and EEPROM/SCL
- U5 pad 7: Net-(U6-VCC) (its old number) -> /GPS/VCC
- U5 pad 8: Net-(U6-VCC) (its old number) -> /GPS/VCC
Routing:
- net Net-(D13-K) (its old number): track 7.94 -> 0.00 mm, vias 2 -> 0
- net /I2C and EEPROM/SCL: track 0.00 -> 7.94 mm, vias 0 -> 2
- net Net-(U6-VCC) (its old number): track 7.60 -> 0.00 mm
- net /GPS/VCC: track 0.00 -> 7.60 mm
- added copper zone on F.Cu, net Net-(U7-SW)
- removed copper zone on F.Cu, net Net-(U6-SW)
Other:
- board text added: "CAN Termination"

Commit message: Updates
Parts:
- added C94: 1nF, MyParts:C0603, F.Cu at (159.2, 44.2)
- added R98: 1MΩ, PCM_JLCPCB:R_0402, F.Cu at (159.6, 47.6)
- added RJ2: KH-RJ45-58-8P8C, MyParts:RJ45-TH_KH-RJ45-58-8P8C, F.Cu at (168.4, 43.7)
- moved R80 87.8 mm to (107.9, 127.0)
- moved R79 87.1 mm to (89.4, 126.3), turned to -90 degrees
- moved H3 76.8 mm to (80.2, 121.4)
- moved H4 76.8 mm to (83.6, 121.4)
- moved R92 76.5 mm to (80.2, 117.8)
- moved R93 76.5 mm to (83.5, 117.8)
- moved RJ1 73.3 mm to (98.2, 119.1), turned to 0 degrees
- moved C68 63.0 mm to (106.9, 112.3), turned to -90 degrees
- moved U9 61.4 mm to (108.6, 119.0), turned to 90 degrees
- moved U8 57.9 mm to (108.6, 116.0), turned to 90 degrees
- moved C70 21.5 mm to (85.0, 54.5)
- moved C71 21.5 mm to (87.6, 51.0)
- moved C72 21.5 mm to (87.6, 48.9)
- moved C81 21.5 mm to (92.7, 46.4)
- moved C69 21.5 mm to (92.0, 58.0)
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- renumbered U17 to J5
Routing:
- net GND: vias 255 -> 252
Other:
- board text added: "Axis Commander with RPCM4 V1.0 -JRSeti-"
- board text added: "CAN Port 1"
- board text added: "CAN Port 2"
