File: kicad/axis_control_1.kicad_sch (KiCad schematic)
At the start: 41 parts, among them CN1 KF2EDGR-2.54-9P, CN2 KF2EDGR-2.54-6P, Q1 BSS138, Q2 BSS138

Commit message: Add CAN JR45 - still working on it
Parts:
- renumbered D37 to D10, D8 to D11, D9 to D12, D10 to D13, D39 to D8, D38 to D9
Connections:
- net 12VENC: now reaches CN1.1, F1.2
Other:
- moved on the sheet: CN1
Changed lines of the file:
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@@
 	(text "Limit Switch 1 Return"
 		(exclude_from_sim no)
-		(at 220.98 64.135 0)
+		(at 224.79 64.77 0)
 		(effects
 			(font
@@
 	(text "Encoder B"
 		(exclude_from_sim no)
-		(at 220.98 57.15 0)
+		(at 224.79 57.15 0)
 		(effects
 			(font
@@
 	(text "Limit Switch 2 Return"
 		(exclude_from_sim no)
-		(at 220.98 69.215 0)
+		(at 224.79 69.85 0)
 		(effects
 			(font
@@
 	(text "Encoder A"
 		(exclude_from_sim no)
-		(at 220.98 54.61 0)
+		(at 224.79 54.61 0)
 		(effects
 			(font
@@
 	(text "Encoder Gnd"
 		(exclude_from_sim no)
-		(at 220.98 52.07 0)
+		(at 224.79 52.07 0)
 		(effects
 			(font
@@
 	(text "Limit Switch 2 Out"
 		(exclude_from_sim no)
-		(at 220.98 67.31 0)
+		(at 224.79 67.31 0)
 		(effects
 			(font
@@
 	(text "Encoder 12V"
 		(exclude_from_sim no)
-		(at 220.98 49.53 0)
+		(at 224.79 49.53 0)
 		(effects
 			(font
@@
 	(text "Encoder Z"
 		(exclude_from_sim no)
-		(at 220.98 59.69 0)
+		(at 224.79 59.69 0)
 		(effects
 			(font
@@
 	(text "Limit Switch 1 Out"
 		(exclude_from_sim no)
-		(at 220.98 62.23 0)
+		(at 224.79 62.23 0)
 		(effects
 			(font
@@
 	)
 	(junction
+		(at 215.9 49.53)
+		(diameter 0)
+		(color 0 0 0 0)
+	)
+	(junction
 		(at 236.22 148.59)
 		(diameter 0)
@@
 	(wire
 		(pts
-			(xy 187.96 62.23) (xy 213.36 62.23)
+			(xy 187.96 62.23) (xy 217.17 62.23)
 		)
 		(stroke
@@
 	(wire
 		(pts
-			(xy 207.01 69.85) (xy 213.36 69.85)
+			(xy 207.01 69.85) (xy 217.17 69.85)
 		)
 		(stroke
@@
 	(wire
 		(pts
-			(xy 212.09 45.72) (xy 212.09 49.53)
+			(xy 215.9 45.72) (xy 215.9 49.53)
 		)
 		(stroke
@@
 	(wire
 		(pts
-			(xy 212.09 35.56) (xy 212.09 34.29)
+			(xy 215.9 35.56) (xy 215.9 34.29)
 		)
 		(stroke
@@
 	(wire
 		(pts
-			(xy 194.31 64.77) (xy 213.36 64.77)
+			(xy 194.31 64.77) (xy 217.17 64.77)
 		)
 		(stroke
@@
 	(wire
 		(pts
-			(xy 212.09 52.07) (xy 213.36 52.07)
+			(xy 212.09 52.07) (xy 217.17 52.07)
 		)
 		(stroke
@@
 	(wire
 		(pts
-			(xy 168.91 54.61) (xy 213.36 54.61)
+			(xy 168.91 54.61) (xy 217.17 54.61)
 		)
 		(stroke
@@
 	(wire
 		(pts
-			(xy 212.09 34.29) (xy 213.36 34.29)
+			(xy 215.9 34.29) (xy 217.17 34.29)
 		)
 		(stroke
@@
 	(wire
 		(pts
+			(xy 214.63 49.53) (xy 215.9 49.53)
+		)
+		(stroke
+			(width 0)
+			(type default)
+		)
+	)
+	(wire
+		(pts
 			(xy 170.18 138.43) (xy 173.99 138.43)
 		)
@@
 	(wire
 		(pts
-			(xy 181.61 59.69) (xy 213.36 59.69)
+			(xy 181.61 59.69) (xy 217.17 59.69)
 		)
 		(stroke
@@
 	(wire
 		(pts
-			(xy 200.66 67.31) (xy 213.36 67.31)
+			(xy 200.66 67.31) (xy 217.17 67.31)
 		)
 		(stroke
@@
 	(wire
 		(pts
-			(xy 175.26 57.15) (xy 213.36 57.15)
+			(xy 175.26 57.15) (xy 217.17 57.15)
 		)
 		(stroke
@@
 	(wire
 		(pts
-			(xy 212.09 49.53) (xy 213.36 49.53)
+			(xy 215.9 49.53) (xy 217.17 49.53)
 		)
 		(stroke
@@
 		)
 	)
+	(label "12VENC"
+		(at 214.63 49.53 180)
+		(effects
+			(font
+				(size 1.27 1.27)
+			)
+			(justify right bottom)
+		)
+	)
 	(label "ENC1_A"
 		(at 43.18 62.23 180)
@@
 	(global_label "12V"
 		(shape input)
-		(at 213.36 34.29 0)
+		(at 217.17 34.29 0)
 		(fields_autoplaced yes)
 		(effects
@@
 		)
 		(property "Intersheetrefs" "${INTERSHEET_REFS}"
-			(at 219.8528 34.29 0)
+			(at 223.6628 34.29 0)
 			(hide yes)
 			(show_name no)
@@
 		(in_pos_files yes)
 		(dnp no)
-		(property "Reference" "D8"
+		(property "Reference" "D11"
 			(at 68.834 143.764 90)
 			(show_name no)
@@
 			(project "rcm_dish_controller"
 				(path "/10d7c3e5-be4d-4306-a59e-500b86bd141f/9493fd2e-7ff6-4d8c-93a5-d9e42c2785c7"
-					(reference "D8")
+					(reference "D11")
 					(unit 1)
 				)
@@
 		(in_pos_files yes)
 		(dnp no)
-		(property "Reference" "D39"
+		(property "Reference" "D8"
 			(at 102.87 108.458 270)
 			(show_name no)
@@
 			(project "rcm_dish_controller"
 				(path "/10d7c3e5-be4d-4306-a59e-500b86bd141f/9493fd2e-7ff6-4d8c-93a5-d9e42c2785c7"
-					(reference "D39")
+					(reference "D8")
 					(unit 1)
 				)
@@
 	(symbol
 		(lib_id "MyParts:KF2EDGR-2.54-9P")
-		(at 218.44 59.69 0)
+		(at 222.25 59.69 0)
 		(unit 1)
 		(body_style 1)
@@
 		(dnp no)
 		(property "Reference" "CN1"
-			(at 216.408 45.974 0)
+			(at 220.218 45.974 0)
 			(show_name no)
 			(do_not_autoplace no)
@@
 		)
 		(property "Value" "KF2EDGR-2.54-9P"
-			(at 215.646 73.406 0)
+			(at 219.456 73.406 0)
 			(show_name no)
 			(do_not_autoplace no)
@@
 		)
 		(property "Footprint" "MyParts:CONN-TH_9P-P2.54_KF2EDGR-2.54-9P"
-			(at 218.44 77.47 0)
+			(at 222.25 77.47 0)
 			(hide yes)
 			(show_name no)
@@
 		)
 		(property "Datasheet" "https://www.lcsc.com/datasheet/C577601.pdf?spm=wm.sxq.inf.ggs&lcsc_vid=FFBaV1wHQFldUVICFgBfBVJTQVJWXgBfEQRYBAFQE1YxVlNRQFRcVVFfT1NbUjtW"
-			(at 218.44 80.01 0)
+			(at 222.25 80.01 0)
 			(hide yes)
 			(show_name no)
@@
 		)
 		(property "Description" "9 Position Board Side/Socket - Closed 2.54mm Pitch Right-Angle Pin"
-			(at 218.44 59.69 0)
+			(at 222.25 59.69 0)
 			(hide yes)
 			(show_name no)
@@
 		)
 		(property "LCSC Part" "C577601"
-			(at 218.44 82.55 0)
+			(at 222.25 82.55 0)
 			(hide yes)
 			(show_name no)
@@
 		(dnp no)
 		(fields_autoplaced yes)
-		(property "Reference" "#PWR021"
+		(property "Reference" "#PWR022"
 			(at 232.41 156.21 0)
 			(hide yes)
@@
 			(project "rcm_dish_controller"
 				(path "/10d7c3e5-be4d-4306-a59e-500b86bd141f/9493fd2e-7ff6-4d8c-93a5-d9e42c2785c7"
-					(reference "#PWR021")
+					(reference "#PWR022")
 					(unit 1)
 				)
@@
 		(in_pos_files yes)
 		(dnp no)
-		(property "Reference" "#PWR0216"
+		(property "Reference" "#PWR019"
 			(at 109.22 100.33 0)
 			(hide yes)
@@
 			(project "rcm_dish_controller"
 				(path "/10d7c3e5-be4d-4306-a59e-500b86bd141f/9493fd2e-7ff6-4d8c-93a5-d9e42c2785c7"
-					(reference "#PWR0216")
+					(reference "#PWR019")
 					(unit 1)
 				)
@@
 		(in_pos_files yes)
 		(dnp no)
-		(property "Reference" "D9"
+		(property "Reference" "D12"
 			(at 74.93 143.764 90)
 			(show_name no)
@@
 			(project "rcm_dish_controller"
 				(path "/10d7c3e5-be4d-4306-a59e-500b86bd141f/9493fd2e-7ff6-4d8c-93a5-d9e42c2785c7"
-					(reference "D9")
+					(reference "D12")
 					(unit 1)
 				)
@@
 		(in_pos_files yes)
 		(dnp no)
-		(property "Reference" "#PWR019"
+		(property "Reference" "#PWR020"
 			(at 73.66 156.21 0)
 			(hide yes)
@@
 			(project "rcm_dish_controller"
 				(path "/10d7c3e5-be4d-4306-a59e-500b86bd141f/9493fd2e-7ff6-4d8c-93a5-d9e42c2785c7"
-					(reference "#PWR019")
+					(reference "#PWR020")
 					(unit 1)
 				)
@@
 		(in_pos_files yes)
 		(dnp no)
-		(property "Reference" "D38"
+		(property "Reference" "D9"
 			(at 109.22 108.458 270)
 			(show_name no)
@@
 			(project "rcm_dish_controller"
 				(path "/10d7c3e5-be4d-4306-a59e-500b86bd141f/9493fd2e-7ff6-4d8c-93a5-d9e42c2785c7"
-					(reference "D38")
+					(reference "D9")
 					(unit 1)
 				)
@@
 		(in_pos_files yes)
 		(dnp no)
-		(property "Reference" "D37"
+		(property "Reference" "D10"
 			(at 115.57 108.458 270)
 			(show_name no)
@@
 			(project "rcm_dish_controller"
 				(path "/10d7c3e5-be4d-4306-a59e-500b86bd141f/9493fd2e-7ff6-4d8c-93a5-d9e42c2785c7"
-					(reference "D37")
+					(reference "D10")
 					(unit 1)
 				)
@@
 	(symbol
 		(lib_id "MyParts:MF-USMF020-2")
-		(at 212.09 40.64 270)
+		(at 215.9 40.64 270)
 		(unit 1)
 		(body_style 1)
@@
 		(fields_autoplaced yes)
 		(property "Reference" "F1"
-			(at 214.63 39.3699 90)
+			(at 218.44 39.3699 90)
 			(show_name no)
 			(do_not_autoplace no)
@@
 		)
 		(property "Value" "MF-USMF020-2"
-			(at 214.63 41.9099 90)
+			(at 218.44 41.9099 90)
 			(show_name no)
 			(do_not_autoplace no)
@@
 		)
 		(property "Footprint" "MyParts:F1210"
-			(at 204.47 40.64 0)
+			(at 208.28 40.64 0)
 			(hide yes)
 			(show_name no)
@@
 		)
 		(property "Datasheet" "https://lcsc.com/product-detail/Surface-Mount-Fuses_BOURNS_MF-USMF020-2_BOURNS-MF-USMF020-2_C210829.html"
-			(at 201.93 40.64 0)
+			(at 205.74 40.64 0)
 			(hide yes)
 			(show_name no)
@@
 		)
 		(property "Description" ""
-			(at 212.09 40.64 0)
+			(at 215.9 40.64 0)
 			(hide yes)
 			(show_name no)
@@
 		)
 		(property "Manufacturer" "BOURNS"
-			(at 199.39 40.64 0)
+			(at 203.2 40.64 0)
 			(hide yes)
 			(show_name no)
@@
 		)
 		(property "MPN" "MF-USMF020-2"
-			(at 196.85 40.64 0)
+			(at 200.66 40.64 0)
 			(hide yes)
 			(show_name no)
@@
 		)
 		(property "LCSC Part" "C210829"
-			(at 194.31 40.64 0)
+			(at 198.12 40.64 0)
 			(hide yes)
 			(show_name no)
@@
 		(in_pos_files yes)
 		(dnp no)
-		(property "Reference" "D10"
+		(property "Reference" "D13"
 			(at 82.296 143.764 90)
 			(show_name no)
@@
 			(project "rcm_dish_controller"
 				(path "/10d7c3e5-be4d-4306-a59e-500b86bd141f/9493fd2e-7ff6-4d8c-93a5-d9e42c2785c7"
-					(reference "D10")
+					(reference "D13")
 					(unit 1)
 				)
@@
 		(dnp no)
 		(fields_autoplaced yes)
-		(property "Reference" "#PWR020"
+		(property "Reference" "#PWR021"
 			(at 170.18 156.21 0)
 			(hide yes)
@@
 			(project "rcm_dish_controller"
 				(path "/10d7c3e5-be4d-4306-a59e-500b86bd141f/9493fd2e-7ff6-4d8c-93a5-d9e42c2785c7"
-					(reference "#PWR020")
+					(reference "#PWR021")
 					(unit 1)
 				)
