File: kicad/axis_control_2.kicad_sch (KiCad schematic)
At the start: 38 parts, among them CN12 KF2EDGR-2.54-9P, CN13 KF2EDGR-2.54-6P, Q7 BSS138, Q8 BSS138

Commit message: Updates to power
Parts:
- R78, R79, R81, R82: LCSC C173683 -> C25744
Changed lines of the file:
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@@
 			)
 		)
-		(property "Datasheet" "https://www.lcsc.com/datasheet/lcsc_datasheet_2411221126_UNI-ROYAL-Uniroyal-Elec-0402WGF1002TCE_C173683.pdf"
+		(property "Datasheet" "https://www.lcsc.com/datasheet/lcsc_datasheet_2411221126_UNI-ROYAL-Uniroyal-Elec-0402WGF1002TCE_C25744.pdf"
 			(at 231.14 137.16 0)
 			(hide yes)
@@
 			)
 		)
-		(property "LCSC" "C173683"
+		(property "LCSC" "C25744"
 			(at 231.14 137.16 0)
 			(hide yes)
@@
 			)
 		)
-		(property "Datasheet" "https://www.lcsc.com/datasheet/lcsc_datasheet_2411221126_UNI-ROYAL-Uniroyal-Elec-0402WGF1002TCE_C173683.pdf"
+		(property "Datasheet" "https://www.lcsc.com/datasheet/lcsc_datasheet_2411221126_UNI-ROYAL-Uniroyal-Elec-0402WGF1002TCE_C25744.pdf"
 			(at 257.81 127 0)
 			(hide yes)
@@
 			)
 		)
-		(property "LCSC" "C173683"
+		(property "LCSC" "C25744"
 			(at 257.81 127 0)
 			(hide yes)
@@
 			)
 		)
-		(property "Datasheet" "https://www.lcsc.com/datasheet/lcsc_datasheet_2411221126_UNI-ROYAL-Uniroyal-Elec-0402WGF1002TCE_C173683.pdf"
+		(property "Datasheet" "https://www.lcsc.com/datasheet/lcsc_datasheet_2411221126_UNI-ROYAL-Uniroyal-Elec-0402WGF1002TCE_C25744.pdf"
 			(at 195.58 127 0)
 			(hide yes)
@@
 			)
 		)
-		(property "LCSC" "C173683"
+		(property "LCSC" "C25744"
 			(at 195.58 127 0)
 			(hide yes)
@@
 			)
 		)
-		(property "Datasheet" "https://www.lcsc.com/datasheet/lcsc_datasheet_2411221126_UNI-ROYAL-Uniroyal-Elec-0402WGF1002TCE_C173683.pdf"
+		(property "Datasheet" "https://www.lcsc.com/datasheet/lcsc_datasheet_2411221126_UNI-ROYAL-Uniroyal-Elec-0402WGF1002TCE_C25744.pdf"
 			(at 168.91 137.16 0)
 			(hide yes)
@@
 			)
 		)
-		(property "LCSC" "C173683"
+		(property "LCSC" "C25744"
 			(at 168.91 137.16 0)
 			(hide yes)

Commit message: CM4 schematic changes, before renumbering
Parts:
- CN13: MPN (none) -> KF2EDGR-2.54-6P; Manufacturer (none) -> KEFA(科发)
Changed lines of the file:
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@@
 	(title_block
 		(title "Encoder/Motor/Limit Switch - Axis2")
-		(date "2026-07-11")
-		(rev "1.1")
+		(date "2026-08-18")
+		(rev "2.0")
 		(company "JRSeti")
 	)
@@
 		)
 	)
-	(global_label "DIR2_MCU"
-		(shape input)
-		(at 53.34 132.08 180)
-		(fields_autoplaced yes)
-		(effects
-			(font
-				(size 1.27 1.27)
-			)
-			(justify right)
-		)
-		(property "Intersheetrefs" "${INTERSHEET_REFS}"
-			(at 40.981 132.08 0)
-			(hide yes)
-			(show_name no)
-			(do_not_autoplace no)
-			(effects
-				(font
-					(size 1.27 1.27)
-				)
-				(justify right)
-			)
-		)
-	)
 	(global_label "3V3"
 		(shape input)
@@
 		)
 	)
-	(global_label "ENABLE2_MCU"
+	(global_label "3V3"
 		(shape input)
-		(at 53.34 137.16 180)
+		(at 256.54 121.92 180)
 		(fields_autoplaced yes)
 		(effects
@@
 		)
 		(property "Intersheetrefs" "${INTERSHEET_REFS}"
-			(at 37.1106 137.16 0)
+			(at 250.0472 121.92 0)
 			(hide yes)
 			(show_name no)
@@
 		)
 	)
-	(global_label "PUL2_MCU"
+	(global_label "12V"
 		(shape input)
-		(at 53.34 127 180)
+		(at 218.44 34.29 0)
 		(fields_autoplaced yes)
 		(effects
@@
 				(size 1.27 1.27)
 			)
-			(justify right)
-		)
-		(property "Intersheetrefs" "${INTERSHEET_REFS}"
-			(at 40.4972 127 0)
-			(hide yes)
-			(show_name no)
-			(do_not_autoplace no)
-			(effects
-				(font
-					(size 1.27 1.27)
-				)
-				(justify right)
-			)
-		)
-	)
-	(global_label "LIMIT2_SW1_MCU"
-		(shape input)
-		(at 196.85 132.08 0)
-		(fields_autoplaced yes)
-		(effects
-			(font
-				(size 0.762 0.762)
-			)
 			(justify left)
 		)
 		(property "Intersheetrefs" "${INTERSHEET_REFS}"
-			(at 208.076 132.08 0)
+			(at 224.9328 34.29 0)
 			(hide yes)
 			(show_name no)
@@
 		)
 	)
-	(global_label "ENC2_Z_MCU"
+	(global_label "12V"
 		(shape input)
-		(at 121.92 64.77 0)
+		(at 193.04 45.72 90)
 		(fields_autoplaced yes)
 		(effects
@@
 		)
 		(property "Intersheetrefs" "${INTERSHEET_REFS}"
-			(at 137.0608 64.77 0)
+			(at 193.04 39.2272 90)
 			(hide yes)
 			(show_name no)
@@
 	(global_label "3V3"
 		(shape input)
-		(at 256.54 121.92 180)
+		(at 85.09 124.46 180)
 		(fields_autoplaced yes)
 		(effects
@@
 		)
 		(property "Intersheetrefs" "${INTERSHEET_REFS}"
-			(at 250.0472 121.92 0)
+			(at 78.5972 124.46 0)
 			(hide yes)
 			(show_name no)
@@
 		)
 	)
-	(global_label "12V"
+	(hierarchical_label "DIR2_MCU"
 		(shape input)
-		(at 218.44 34.29 0)
-		(fields_autoplaced yes)
+		(at 53.34 132.08 180)
 		(effects
 			(font
 				(size 1.27 1.27)
 			)
-			(justify left)
-		)
-		(property "Intersheetrefs" "${INTERSHEET_REFS}"
-			(at 224.9328 34.29 0)
-			(hide yes)
-			(show_name no)
-			(do_not_autoplace no)
-			(effects
-				(font
-					(size 1.27 1.27)
-				)
-				(justify left)
-			)
+			(justify right)
 		)
 	)
-	(global_label "LIMIT2_SW2_MCU"
+	(hierarchical_label "ENABLE2_MCU"
 		(shape input)
-		(at 259.08 132.08 0)
-		(fields_autoplaced yes)
+		(at 53.34 137.16 180)
 		(effects
 			(font
-				(size 0.762 0.762)
-			)
-			(justify left)
-		)
-		(property "Intersheetrefs" "${INTERSHEET_REFS}"
-			(at 270.306 132.08 0)
-			(hide yes)
-			(show_name no)
-			(do_not_autoplace no)
-			(effects
-				(font
-					(size 1.27 1.27)
-				)
-				(justify left)
+				(size 1.27 1.27)
 			)
+			(justify right)
 		)
 	)
-	(global_label "12V"
+	(hierarchical_label "PUL2_MCU"
 		(shape input)
-		(at 193.04 45.72 90)
-		(fields_autoplaced yes)
+		(at 53.34 127 180)
 		(effects
 			(font
 				(size 1.27 1.27)
 			)
-			(justify left)
+			(justify right)
 		)
-		(property "Intersheetrefs" "${INTERSHEET_REFS}"
-			(at 193.04 39.2272 90)
-			(hide yes)
-			(show_name no)
-			(do_not_autoplace no)
-			(effects
-				(font
-					(size 1.27 1.27)
-				)
-				(justify left)
+	)
+	(hierarchical_label "LIMIT2_SW1_MCU"
+		(shape output)
+		(at 196.85 132.08 0)
+		(effects
+			(font
+				(size 0.762 0.762)
 			)
+			(justify left)
 		)
 	)
-	(global_label "ENC2_B_MCU"
-		(shape input)
-		(at 86.36 64.77 0)
-		(fields_autoplaced yes)
+	(hierarchical_label "ENC2_Z_MCU"
+		(shape output)
+		(at 121.92 64.77 0)
 		(effects
 			(font
@@
 			(justify left)
 		)
-		(property "Intersheetrefs" "${INTERSHEET_REFS}"
-			(at 101.5613 64.77 0)
-			(hide yes)
-			(show_name no)
-			(do_not_autoplace no)
-			(effects
-				(font
-					(size 1.27 1.27)
-				)
-				(justify left)
+	)
+	(hierarchical_label "LIMIT2_SW2_MCU"
+		(shape output)
+		(at 259.08 132.08 0)
+		(effects
+			(font
+				(size 0.762 0.762)
 			)
+			(justify left)
 		)
 	)
-	(global_label "ENC2_A_MCU"
-		(shape input)
-		(at 50.8 64.77 0)
-		(fields_autoplaced yes)
+	(hierarchical_label "ENC2_B_MCU"
+		(shape output)
+		(at 86.36 64.77 0)
 		(effects
 			(font
@@
 			(justify left)
 		)
-		(property "Intersheetrefs" "${INTERSHEET_REFS}"
-			(at 65.8199 64.77 0)
-			(hide yes)
-			(show_name no)
-			(do_not_autoplace no)
-			(effects
-				(font
-					(size 1.27 1.27)
-				)
-				(justify left)
-			)
-		)
 	)
-	(global_label "3V3"
-		(shape input)
-		(at 85.09 124.46 180)
-		(fields_autoplaced yes)
+	(hierarchical_label "ENC2_A_MCU"
+		(shape output)
+		(at 50.8 64.77 0)
 		(effects
 			(font
 				(size 1.27 1.27)
 			)
-			(justify right)
-		)
-		(property "Intersheetrefs" "${INTERSHEET_REFS}"
-			(at 78.5972 124.46 0)
-			(hide yes)
-			(show_name no)
-			(do_not_autoplace no)
-			(effects
-				(font
-					(size 1.27 1.27)
-				)
-				(justify right)
-			)
+			(justify left)
 		)
 	)
@@
 	(symbol
 		(lib_id "MyParts:KF2EDGR-2.54-6P")
-		(at 100.33 130.81 0)
+		(at 99.06 130.81 0)
 		(unit 1)
 		(body_style 1)
@@
 		(dnp no)
 		(property "Reference" "CN13"
-			(at 100.076 120.904 0)
+			(at 98.806 120.904 0)
 			(show_name no)
 			(do_not_autoplace no)
@@
 		)
 		(property "Value" "KF2EDGR-2.54-6P"
-			(at 99.314 141.478 0)
+			(at 98.044 141.478 0)
 			(show_name no)
 			(do_not_autoplace no)
@@
 		)
 		(property "Footprint" "MyParts:CONN-TH_KF2EDGR-2.54-6P"
-			(at 100.33 144.78 0)
+			(at 99.06 144.78 0)
 			(hide yes)
 			(show_name no)
@@
 			)
 		)
-		(property "Datasheet" "https://www.lcsc.com/datasheet/C577598.pdf?spm=wm.sxq.inf.ggs&lcsc_vid=FFBaV1wHQFldUVICFgBfBVJTQVJWXgBfEQRYBAFQE1YxVlNRQFRcVVJfR1FdVTtW"
-			(at 100.33 147.32 0)
+		(property "Datasheet" "https://lcsc.com/product-detail/Pluggable-System-Terminal-Block_Cixi-Kefa-Elec-KF2EDGR-2-54-6P_C577598.html"
+			(at 99.06 147.32 0)
 			(hide yes)
 			(show_name no)
@@
 		)
 		(property "Description" "6 Position Board Side/Socket - Closed 2.54mm Pitch Right-Angle Pin"
-			(at 100.33 130.81 0)
+			(at 99.06 130.81 0)
 			(hide yes)
 			(show_name no)
@@
 		)
 		(property "LCSC Part" "C577598"
-			(at 100.33 149.86 0)
+			(at 99.06 149.86 0)
+			(hide yes)
+			(show_name no)
+			(do_not_autoplace no)
+			(effects
+				(font
+					(size 1.27 1.27)
+				)
+			)
+		)
+		(property "Manufacturer" "KEFA(科发)"
+			(at 99.06 149.86 0)
+			(hide yes)
+			(show_name no)
+			(do_not_autoplace no)
+			(effects
+				(font
+					(size 1.27 1.27)
+				)
+			)
+		)
+		(property "MPN" "KF2EDGR-2.54-6P"
+			(at 99.06 152.4 0)
 			(hide yes)
 			(show_name no)

Commit message: Before adding CAN
Parts:
- renumbered C67 to C46, C68 to C47, C69 to C48, C71 to C49, C76 to C50, CN12 to CN8, CN13 to CN9, D7 to D19, D8 to D20, D9 to D21, D10 to D22, D11 to D23, D33 to D24, D34 to D25, D21 to D26, D22 to D27, D23 to D28, F5 to F2, Q7 to Q6, Q8 to Q7, R33 to R43, R34 to R44, R35 to R45, R36 to R46, R37 to R47, R38 to R48, R43 to R49, R60 to R50, R79 to R51, R82 to R52, R44 to R53, R61 to R54, R45 to R55, R62 to R56, R78 to R57, R81 to R58, R77 to R59, R80 to R60

Commit message: More mods
Parts:
- added D40, D41, D42: TPESD0402G05V, MyParts:D0402-BI, symbol MyParts:TPESD0402G05V
Connections:
- net GND: now also D40.2 (A), D41.2 (A), D42.2 (A)
- net at CN9.3, R53.2: now also D41.1 (K)
- net at CN9.1, R49.2: now also D40.1 (K)
- net at CN9.5, R55.2: now also D42.1 (K)
Other:
- note added: "CN9 pins 1/3/5 are the 3V3 common-anode feed to the driver optos - TVS at the connector, matching pins 2/4/6."
- moved on the sheet: CN9

Commit message: Add CAN JR45 - still working on it
Parts:
- renumbered C46 to C34, C47 to C35, C48 to C36, C49 to C37, C50 to C38, CN8 to CN7, CN9 to CN8, D19 to D22, D20 to D23, D21 to D24, D22 to D25, D23 to D26, D24 to D27, D25 to D28, D42 to D29, D41 to D30, D40 to D31, D26 to D32, D27 to D33, D28 to D34, R43 to R41, R44 to R42, R45 to R43, R46 to R44, R47 to R45, R48 to R46, R49 to R47, R50 to R48, R51 to R49, R52 to R50, R53 to R51, R54 to R52, R55 to R53, R56 to R54, R57 to R55, R58 to R56, R59 to R57, R60 to R58
Connections:
- net DIR2-: now reaches CN8.4, D33.1 (K), R52.2
- net DIR2+: now reaches CN8.3, D30.1 (K), R51.2
- net PUL2+: now reaches CN8.1, D31.1 (K), R47.2
- net 12VENC: now reaches CN7.1, F2.2
- net PUL2-: now reaches CN8.2, D32.1 (K), R48.2
- net ENABLE2+: now reaches CN8.5, D29.1 (K), R53.2
- net ENABLE2-: now reaches CN8.6, D34.1 (K), R54.2
Other:
- note added: "Limit Switch 1 Out"
- note added: "Limit Switch 1 Return"
- moved on the sheet: CN7
