File: kicad/power_3v3.kicad_sch (KiCad schematic)
At the start: 26 parts, among them U17 AP64501SP-13

Commit message: Before adding CAN
Parts:
- removed C100, C95, C96, C97, C98, C99: 10uF 35V, MyParts:C0805, symbol MyParts:GRM21BC8YA106KE11L
- removed C102, C106: 100nF, PCM_JLCPCB:C_0402, symbol PCM_JLCPCB-Capacitors:0402,100nF
- removed C104: 56pF, MyParts:C0402, symbol MyParts:CL05C560JB51PNC
- removed C105: 2.7nF 50V, MyParts:C0402, symbol MyParts:CC0402KRX7R9BB272
- removed C107: DNP, MyParts:C0402, symbol Device:C
- removed C110: 100uF 6.3V, Capacitor_Tantalum_SMD:CP_EIA-7343-31_Kemet-D, symbol Device:C_Polarized
- removed C47, C48, C49, C50: 10uF 10V, MyParts:C0805, symbol MyParts:CL21B106KPQNNNE
- removed L15: SRN6045TA-3R3Y, MyParts:IND-SMD_L6.0-W6.0, symbol MyParts:SRN6045TA-3R3Y
- removed R22: 22.1K, MyParts:R0402, symbol MyParts:FRC0402F2212TS
- removed R55: 10Ω, MyParts:R1206, symbol MyParts:1206W4F100JT5E
- removed R63: 10.5KΩ, MyParts:R0402, symbol MyParts:0402WGF1052TCE
- removed R65: 69.8K, MyParts:R0402, symbol MyParts:0402WGF6982TCE
- removed U17: AP64501SP-13, MyParts:SOIC-8_L4.9-W3.9-P1.27-LS6.0-BL-EP-1, symbol MyParts:AP64501SP-13
- added C56: 100nF, PCM_JLCPCB:C_0402, symbol PCM_JLCPCB-Capacitors:0402,100nF,(2)
- added C57, C58: 10uF, PCM_JLCPCB:C_0805, symbol PCM_JLCPCB-Capacitors:0805,10uF,(2)
- added C59: 100nF, PCM_JLCPCB:C_0603, symbol PCM_JLCPCB-Capacitors:0603,100nF
- added C60: 22pF, PCM_JLCPCB:C_0603, symbol PCM_JLCPCB-Capacitors:0603,22pF
- added C61: 22uF, PCM_JLCPCB:C_0805, symbol PCM_JLCPCB-Capacitors:0805,22uF
- added C62: 1uF, PCM_JLCPCB:C_0402, symbol PCM_JLCPCB-Capacitors:0402,1uF
- added L8: 3.3uH, MyParts:IND-SMD_L3.0-W3.0-1, symbol MyParts:ANR3015T4R7M
- added R72: 976kΩ, Resistor_SMD:R_0805_2012Metric, symbol Device:R
- added R73: 100kΩ, PCM_JLCPCB:R_0603, symbol PCM_JLCPCB-Resistors:0603,100kΩ
- added R74: 220kΩ, PCM_JLCPCB:R_0603, symbol PCM_JLCPCB-Resistors:0603,220kΩ
- added U7: MP2322GQH-Z, MyParts:QFN-8_L2.0-W1.5-P0.50-BL, symbol MyParts:MP2322GQH-Z
- renumbered C51 to C55, TP14 to TP6, TP11 to TP7
Connections:
- net 12V_MCU: now also C57.1, C58.1, C59.1, U7.2 (IN), U7.3 (EN)
- net 3V3: now also C60.1, C61.1, L8.2, R72.1
- net GND: now also C57.2, C58.2, C59.2, C61.2, C62.2, R74.2, U7.1 (GND)
- new net: R73.1, U7.6 (PG)
- new net: C62.1, R73.2, U7.4 (VCC)
- new net: C60.2, R72.2, R74.1, U7.5 (FB)
- new net: C56.2, U7.7 (BST)
- new net: C56.1, L8.1, U7.8 (SW)
Other:
- note added: "0.1%"
- note added: "1%"
- note added: "12V to 3V3 Buck"
- note removed: "3V3 @ 1A"
- note removed: "3V3 @ 1A PSU ( 7.5v-28v Input )"
- moved on the sheet: TP7

Commit message: Part positioning of PWR, USB, Ethernet
Parts:
- removed TP7: RH-5016, MyParts:TESTPOINT-SMD_L3.0-W2.0, symbol MyParts:RH-5016
Changed lines of the file:
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@@
 	(wire
 		(pts
-			(xy 195.58 80.01) (xy 196.85 80.01)
-		)
-		(stroke
-			(width 0)
-			(type default)
-		)
-	)
-	(wire
-		(pts
 			(xy 196.85 118.11) (xy 172.72 118.11)
 		)
@@
 	(global_label "3V3"
 		(shape input)
-		(at 195.58 80.01 180)
-		(fields_autoplaced yes)
-		(effects
-			(font
-				(size 1.27 1.27)
-			)
-			(justify right)
-		)
-		(property "Intersheetrefs" "${INTERSHEET_REFS}"
-			(at 189.0872 80.01 0)
-			(hide yes)
-			(show_name no)
-			(do_not_autoplace no)
-			(effects
-				(font
-					(size 1.27 1.27)
-				)
-				(justify right)
-			)
-		)
-	)
-	(global_label "3V3"
-		(shape input)
 		(at 198.12 92.71 0)
 		(fields_autoplaced yes)
@@
 					(unit 1)
 				)
-			)
-		)
-	)
-	(symbol
-		(lib_id "MyParts:RH-5016")
-		(at 200.66 80.01 0)
-		(unit 1)
-		(body_style 1)
-		(exclude_from_sim no)
-		(in_bom yes)
-		(on_board yes)
-		(in_pos_files yes)
-		(dnp no)
-		(fields_autoplaced yes)
-		(property "Reference" "TP7"
-			(at 205.74 78.7399 0)
-			(show_name no)
-			(do_not_autoplace no)
-			(effects
-				(font
-					(size 1.27 1.27)
-				)
-				(justify left)
-			)
-		)
-		(property "Value" "RH-5016"
-			(at 205.74 81.2799 0)
-			(show_name no)
-			(do_not_autoplace no)
-			(effects
-				(font
-					(size 1.27 1.27)
-				)
-				(justify left)
-			)
-		)
-		(property "Footprint" "MyParts:TESTPOINT-SMD_L3.0-W2.0"
-			(at 200.66 87.63 0)
-			(hide yes)
-			(show_name no)
-			(do_not_autoplace no)
-			(effects
-				(font
-					(size 1.27 1.27)
-				)
-			)
-		)
-		(property "Datasheet" "https://www.lcsc.com/datasheet/C5199799.pdf"
-			(at 200.66 90.17 0)
-			(hide yes)
-			(show_name no)
-			(do_not_autoplace no)
-			(effects
-				(font
-					(size 1.27 1.27)
-				)
-			)
-		)
-		(property "Description" ""
-			(at 200.66 80.01 0)
-			(hide yes)
-			(show_name no)
-			(do_not_autoplace no)
-			(effects
-				(font
-					(size 1.27 1.27)
-				)
-			)
-		)
-		(property "Manufacturer" "荣和"
-			(at 200.66 92.71 0)
-			(hide yes)
-			(show_name no)
-			(do_not_autoplace no)
-			(effects
-				(font
-					(size 1.27 1.27)
-				)
-			)
-		)
-		(property "MPN" "RH-5016"
-			(at 200.66 95.25 0)
-			(hide yes)
-			(show_name no)
-			(do_not_autoplace no)
-			(effects
-				(font
-					(size 1.27 1.27)
-				)
-			)
-		)
-		(property "LCSC Part" "C5199799"
-			(at 200.66 97.79 0)
-			(hide yes)
-			(show_name no)
-			(do_not_autoplace no)
-			(effects
-				(font
-					(size 1.27 1.27)
-				)
-			)
-		)
-		(pin "1"
-		)
-		(instances
-			(project "rcm_dish_controller"
-				(path "/10d7c3e5-be4d-4306-a59e-500b86bd141f/f4424325-c15a-4f12-b98c-68501db44bed/28ecc382-76c0-468b-9943-cf450709a5af"
-					(reference "TP7")
-					(unit 1)
-				)

Commit message: Add CAN JR45 - still working on it
Parts:
- renumbered C55 to C43, C56 to C44, C57 to C45, C58 to C46, C59 to C47, C60 to C48, C61 to C49, C62 to C50, L8 to L3, U7 to U6
Changed lines of the file:
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@@
 		(dnp no)
 		(fields_autoplaced yes)
-		(property "Reference" "#PWR070"
+		(property "Reference" "#PWR069"
 			(at 104.14 113.03 0)
 			(hide yes)
@@
 			(project "rcm_dish_controller"
 				(path "/10d7c3e5-be4d-4306-a59e-500b86bd141f/f4424325-c15a-4f12-b98c-68501db44bed/28ecc382-76c0-468b-9943-cf450709a5af"
-					(reference "#PWR070")
+					(reference "#PWR069")
 					(unit 1)
 				)
@@
 		(dnp no)
 		(fields_autoplaced yes)
-		(property "Reference" "#PWR072"
+		(property "Reference" "#PWR071"
 			(at 132.08 128.27 0)
 			(hide yes)
@@
 			(project "rcm_dish_controller"
 				(path "/10d7c3e5-be4d-4306-a59e-500b86bd141f/f4424325-c15a-4f12-b98c-68501db44bed/28ecc382-76c0-468b-9943-cf450709a5af"
-					(reference "#PWR072")
+					(reference "#PWR071")
 					(unit 1)
 				)
@@
 		(dnp no)
 		(fields_autoplaced yes)
-		(property "Reference" "C62"
+		(property "Reference" "C50"
 			(at 134.62 114.2999 0)
 			(show_name no)
@@
 			(project "rcm_dish_controller"
 				(path "/10d7c3e5-be4d-4306-a59e-500b86bd141f/f4424325-c15a-4f12-b98c-68501db44bed/28ecc382-76c0-468b-9943-cf450709a5af"
-					(reference "C62")
+					(reference "C50")
 					(unit 1)
 				)
@@
 		(in_pos_files yes)
 		(dnp no)
-		(property "Reference" "#PWR068"
+		(property "Reference" "#PWR067"
 			(at 146.05 63.5 0)
 			(hide yes)
@@
 			(project "rcm_dish_controller"
 				(path "/10d7c3e5-be4d-4306-a59e-500b86bd141f/f4424325-c15a-4f12-b98c-68501db44bed/28ecc382-76c0-468b-9943-cf450709a5af"
-					(reference "#PWR068")
+					(reference "#PWR067")
 					(unit 1)
 				)
@@
 		(dnp no)
 		(fields_autoplaced yes)
-		(property "Reference" "#PWR071"
+		(property "Reference" "#PWR070"
 			(at 172.72 125.73 0)
 			(hide yes)
@@
 			(project "rcm_dish_controller"
 				(path "/10d7c3e5-be4d-4306-a59e-500b86bd141f/f4424325-c15a-4f12-b98c-68501db44bed/28ecc382-76c0-468b-9943-cf450709a5af"
-					(reference "#PWR071")
+					(reference "#PWR070")
 					(unit 1)
 				)
@@
 		(dnp no)
 		(fields_autoplaced yes)
-		(property "Reference" "C61"
+		(property "Reference" "C49"
 			(at 199.39 100.3299 0)
 			(show_name no)
@@
 			(project "rcm_dish_controller"
 				(path "/10d7c3e5-be4d-4306-a59e-500b86bd141f/f4424325-c15a-4f12-b98c-68501db44bed/28ecc382-76c0-468b-9943-cf450709a5af"
-					(reference "C61")
+					(reference "C49")
 					(unit 1)
 				)
@@
 		(dnp no)
 		(fields_autoplaced yes)
-		(property "Reference" "C55"
+		(property "Reference" "C43"
 			(at 148.59 49.5299 0)
 			(show_name no)
@@
 			(project "rcm_dish_controller"
 				(path "/10d7c3e5-be4d-4306-a59e-500b86bd141f/f4424325-c15a-4f12-b98c-68501db44bed/28ecc382-76c0-468b-9943-cf450709a5af"
-					(reference "C55")
+					(reference "C43")
 					(unit 1)
 				)
@@
 		(dnp no)
 		(fields_autoplaced yes)
-		(property "Reference" "U7"
+		(property "Reference" "U6"
 			(at 132.08 85.09 0)
 			(show_name no)
@@
 			(project "rcm_dish_controller"
 				(path "/10d7c3e5-be4d-4306-a59e-500b86bd141f/f4424325-c15a-4f12-b98c-68501db44bed/28ecc382-76c0-468b-9943-cf450709a5af"
-					(reference "U7")
+					(reference "U6")
 					(unit 1)
 				)
@@
 		(dnp no)
 		(fields_autoplaced yes)
-		(property "Reference" "L8"
+		(property "Reference" "L3"
 			(at 162.56 86.36 0)
 			(show_name no)
@@
 			(project "rcm_dish_controller"
 				(path "/10d7c3e5-be4d-4306-a59e-500b86bd141f/f4424325-c15a-4f12-b98c-68501db44bed/28ecc382-76c0-468b-9943-cf450709a5af"
-					(reference "L8")
+					(reference "L3")
 					(unit 1)
 				)
@@
 		(dnp no)
 		(fields_autoplaced yes)
-		(property "Reference" "C56"
+		(property "Reference" "C44"
 			(at 149.86 86.36 90)
 			(show_name no)
@@
 			(project "rcm_dish_controller"
 				(path "/10d7c3e5-be4d-4306-a59e-500b86bd141f/f4424325-c15a-4f12-b98c-68501db44bed/28ecc382-76c0-468b-9943-cf450709a5af"
-					(reference "C56")
+					(reference "C44")
 					(unit 1)
 				)
@@
 		(dnp no)
 		(fields_autoplaced yes)
-		(property "Reference" "C60"
+		(property "Reference" "C48"
 			(at 185.42 100.3299 0)
 			(show_name no)
@@
 			(project "rcm_dish_controller"
 				(path "/10d7c3e5-be4d-4306-a59e-500b86bd141f/f4424325-c15a-4f12-b98c-68501db44bed/28ecc382-76c0-468b-9943-cf450709a5af"
-					(reference "C60")
+					(reference "C48")
 					(unit 1)
 				)
@@
 		(in_pos_files yes)
 		(dnp no)
-		(property "Reference" "C59"
+		(property "Reference" "C47"
 			(at 112.014 97.7899 0)
 			(show_name no)
@@
 			(project "rcm_dish_controller"
 				(path "/10d7c3e5-be4d-4306-a59e-500b86bd141f/f4424325-c15a-4f12-b98c-68501db44bed/28ecc382-76c0-468b-9943-cf450709a5af"
-					(reference "C59")
+					(reference "C47")
 					(unit 1)
 				)
@@
 		(in_pos_files yes)
 		(dnp no)
-		(property "Reference" "C57"
+		(property "Reference" "C45"
 			(at 99.06 97.7899 0)
 			(show_name no)
@@
 			(project "rcm_dish_controller"
 				(path "/10d7c3e5-be4d-4306-a59e-500b86bd141f/f4424325-c15a-4f12-b98c-68501db44bed/28ecc382-76c0-468b-9943-cf450709a5af"
-					(reference "C57")
+					(reference "C45")
 					(unit 1)
 				)
@@
 		(in_pos_files yes)
 		(dnp no)
-		(property "Reference" "C58"
+		(property "Reference" "C46"
 			(at 105.664 97.7899 0)
 			(show_name no)
@@
 			(project "rcm_dish_controller"
 				(path "/10d7c3e5-be4d-4306-a59e-500b86bd141f/f4424325-c15a-4f12-b98c-68501db44bed/28ecc382-76c0-468b-9943-cf450709a5af"
-					(reference "C58")
+					(reference "C46")
 					(unit 1)
 				)
@@
 		(dnp no)
 		(fields_autoplaced yes)
-		(property "Reference" "#PWR069"
+		(property "Reference" "#PWR068"
 			(at 119.38 80.01 0)
 			(hide yes)
@@
 			(project "rcm_dish_controller"
 				(path "/10d7c3e5-be4d-4306-a59e-500b86bd141f/f4424325-c15a-4f12-b98c-68501db44bed/28ecc382-76c0-468b-9943-cf450709a5af"
-					(reference "#PWR069")
+					(reference "#PWR068")
 					(unit 1)
 				)
