File: kicad/power_5v.kicad_sch (KiCad schematic)
At the start: 26 parts, among them U18 AP64501SP-13

Commit message: Before adding CAN
Parts:
- renumbered C78 to C63, C115 to C64, C52 to C65, C53 to C66, C54 to C67, C77 to C68, C117 to C69, C83 to C70, C101 to C71, C103 to C72, C111 to C73, C112 to C74, C113 to C75, C114 to C76, C116 to C77, C81 to C78, C82 to C79, F1 to F4, L16 to L9, R56 to R75, R40 to R76, R39 to R77, R13 to R78, TP13 to TP8, TP12 to TP9, U18 to U8

Commit message: Add CAN JR45 - still working on it
Parts:
- renumbered C63 to C51, C64 to C52, C65 to C53, C66 to C54, C67 to C55, C68 to C56, C69 to C57, C70 to C58, C71 to C59, C72 to C60, C73 to C61, C74 to C62, C75 to C63, C76 to C64, C77 to C65, C78 to C66, C79 to C67, L9 to L4, TP8 to TP7, TP9 to TP8, U8 to U7
Changed lines of the file:
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@@
 		(dnp no)
 		(fields_autoplaced yes)
-		(property "Reference" "C77"
+		(property "Reference" "C65"
 			(at 116.84 138.4299 0)
 			(show_name no)
@@
 			(project "rcm_dish_controller"
 				(path "/10d7c3e5-be4d-4306-a59e-500b86bd141f/f4424325-c15a-4f12-b98c-68501db44bed/2b73156f-617f-4ddb-9603-19922a26015d"
-					(reference "C77")
+					(reference "C65")
 					(unit 1)
 				)
@@
 		(in_pos_files yes)
 		(dnp no)
-		(property "Reference" "C72"
+		(property "Reference" "C60"
 			(at 64.516 134.874 90)
 			(show_name no)
@@
 			(project "rcm_dish_controller"
 				(path "/10d7c3e5-be4d-4306-a59e-500b86bd141f/f4424325-c15a-4f12-b98c-68501db44bed/2b73156f-617f-4ddb-9603-19922a26015d"
-					(reference "C72")
+					(reference "C60")
 					(unit 1)
 				)
@@
 		(in_pos_files yes)
 		(dnp no)
-		(property "Reference" "C69"
+		(property "Reference" "C57"
 			(at 225.806 120.0149 0)
 			(show_name no)
@@
 			(project "rcm_dish_controller"
 				(path "/10d7c3e5-be4d-4306-a59e-500b86bd141f/f4424325-c15a-4f12-b98c-68501db44bed/2b73156f-617f-4ddb-9603-19922a26015d"
-					(reference "C69")
+					(reference "C57")
 					(unit 1)
 				)
@@
 		(in_pos_files yes)
 		(dnp no)
-		(property "Reference" "C75"
+		(property "Reference" "C63"
 			(at 96.266 134.874 90)
 			(show_name no)
@@
 			(project "rcm_dish_controller"
 				(path "/10d7c3e5-be4d-4306-a59e-500b86bd141f/f4424325-c15a-4f12-b98c-68501db44bed/2b73156f-617f-4ddb-9603-19922a26015d"
-					(reference "C75")
+					(reference "C63")
 					(unit 1)
 				)
@@
 		(dnp no)
 		(fields_autoplaced yes)
-		(property "Reference" "TP8"
+		(property "Reference" "TP7"
 			(at 157.48 49.5299 0)
 			(show_name no)
@@
 			(project "rcm_dish_controller"
 				(path "/10d7c3e5-be4d-4306-a59e-500b86bd141f/f4424325-c15a-4f12-b98c-68501db44bed/2b73156f-617f-4ddb-9603-19922a26015d"
-					(reference "TP8")
+					(reference "TP7")
 					(unit 1)
 				)
@@
 		(in_pos_files yes)
 		(dnp yes)
-		(property "Reference" "C70"
+		(property "Reference" "C58"
 			(at 176.53 124.46 0)
 			(show_name no)
@@
 			(project "rcm_dish_controller"
 				(path "/10d7c3e5-be4d-4306-a59e-500b86bd141f/f4424325-c15a-4f12-b98c-68501db44bed/2b73156f-617f-4ddb-9603-19922a26015d"
-					(reference "C70")
+					(reference "C58")
 					(unit 1)
 				)
@@
 		(in_pos_files yes)
 		(dnp no)
-		(property "Reference" "C64"
+		(property "Reference" "C52"
 			(at 107.188 118.3639 0)
 			(show_name no)
@@
 			(project "rcm_dish_controller"
 				(path "/10d7c3e5-be4d-4306-a59e-500b86bd141f/f4424325-c15a-4f12-b98c-68501db44bed/2b73156f-617f-4ddb-9603-19922a26015d"
-					(reference "C64")
+					(reference "C52")
 					(unit 1)
 				)
@@
 		(dnp no)
 		(fields_autoplaced yes)
-		(property "Reference" "L9"
+		(property "Reference" "L4"
 			(at 153.67 109.22 0)
 			(show_name no)
@@
 			(project "rcm_dish_controller"
 				(path "/10d7c3e5-be4d-4306-a59e-500b86bd141f/f4424325-c15a-4f12-b98c-68501db44bed/2b73156f-617f-4ddb-9603-19922a26015d"
-					(reference "L9")
+					(reference "L4")
 					(unit 1)
 				)
@@
 		(in_pos_files yes)
 		(dnp no)
-		(property "Reference" "#PWR076"
+		(property "Reference" "#PWR075"
 			(at 138.43 161.29 0)
 			(hide yes)
@@
 			(project "rcm_dish_controller"
 				(path "/10d7c3e5-be4d-4306-a59e-500b86bd141f/f4424325-c15a-4f12-b98c-68501db44bed/2b73156f-617f-4ddb-9603-19922a26015d"
-					(reference "#PWR076")
+					(reference "#PWR075")
 					(unit 1)
 				)
@@
 		(in_pos_files yes)
 		(dnp no)
-		(property "Reference" "#PWR074"
+		(property "Reference" "#PWR073"
 			(at 204.47 134.62 0)
 			(hide yes)
@@
 			(project "rcm_dish_controller"
 				(path "/10d7c3e5-be4d-4306-a59e-500b86bd141f/f4424325-c15a-4f12-b98c-68501db44bed/2b73156f-617f-4ddb-9603-19922a26015d"
-					(reference "#PWR074")
+					(reference "#PWR073")
 					(unit 1)
 				)
@@
 		(in_pos_files yes)
 		(dnp no)
-		(property "Reference" "#PWR073"
+		(property "Reference" "#PWR072"
 			(at 144.78 81.28 0)
 			(hide yes)
@@
 			(project "rcm_dish_controller"
 				(path "/10d7c3e5-be4d-4306-a59e-500b86bd141f/f4424325-c15a-4f12-b98c-68501db44bed/2b73156f-617f-4ddb-9603-19922a26015d"
-					(reference "#PWR073")
+					(reference "#PWR072")
 					(unit 1)
 				)
@@
 		(in_pos_files yes)
 		(dnp no)
-		(property "Reference" "C71"
+		(property "Reference" "C59"
 			(at 54.356 134.874 90)
 			(show_name no)
@@
 			(project "rcm_dish_controller"
 				(path "/10d7c3e5-be4d-4306-a59e-500b86bd141f/f4424325-c15a-4f12-b98c-68501db44bed/2b73156f-617f-4ddb-9603-19922a26015d"
-					(reference "C71")
+					(reference "C59")
 					(unit 1)
 				)
@@
 		(in_pos_files yes)
 		(dnp no)
-		(property "Reference" "C74"
+		(property "Reference" "C62"
 			(at 86.106 134.874 90)
 			(show_name no)
@@
 			(project "rcm_dish_controller"
 				(path "/10d7c3e5-be4d-4306-a59e-500b86bd141f/f4424325-c15a-4f12-b98c-68501db44bed/2b73156f-617f-4ddb-9603-19922a26015d"
-					(reference "C74")
+					(reference "C62")
 					(unit 1)
 				)
@@
 		(in_pos_files yes)
 		(dnp no)
-		(property "Reference" "C67"
+		(property "Reference" "C55"
 			(at 206.756 120.0149 90)
 			(show_name no)
@@
 			(project "rcm_dish_controller"
 				(path "/10d7c3e5-be4d-4306-a59e-500b86bd141f/f4424325-c15a-4f12-b98c-68501db44bed/2b73156f-617f-4ddb-9603-19922a26015d"
-					(reference "C67")
+					(reference "C55")
 					(unit 1)
 				)
@@
 		(in_pos_files yes)
 		(dnp yes)
-		(property "Reference" "C78"
+		(property "Reference" "C66"
 			(at 144.018 141.224 0)
 			(show_name no)
@@
 			(project "rcm_dish_controller"
 				(path "/10d7c3e5-be4d-4306-a59e-500b86bd141f/f4424325-c15a-4f12-b98c-68501db44bed/2b73156f-617f-4ddb-9603-19922a26015d"
-					(reference "C78")
+					(reference "C66")
 					(unit 1)
 				)
@@
 		(dnp no)
 		(fields_autoplaced yes)
-		(property "Reference" "C63"
+		(property "Reference" "C51"
 			(at 147.32 67.3099 0)
 			(show_name no)
@@
 			(project "rcm_dish_controller"
 				(path "/10d7c3e5-be4d-4306-a59e-500b86bd141f/f4424325-c15a-4f12-b98c-68501db44bed/2b73156f-617f-4ddb-9603-19922a26015d"
-					(reference "C63")
+					(reference "C51")
 					(unit 1)
 				)
@@
 		(in_pos_files yes)
 		(dnp no)
-		(property "Reference" "C66"
+		(property "Reference" "C54"
 			(at 197.866 120.0149 90)
 			(show_name no)
@@
 			(project "rcm_dish_controller"
 				(path "/10d7c3e5-be4d-4306-a59e-500b86bd141f/f4424325-c15a-4f12-b98c-68501db44bed/2b73156f-617f-4ddb-9603-19922a26015d"
-					(reference "C66")
+					(reference "C54")
 					(unit 1)
 				)
@@
 		(in_pos_files yes)
 		(dnp no)
-		(property "Reference" "C65"
+		(property "Reference" "C53"
 			(at 188.976 120.0149 90)
 			(show_name no)
@@
 			(project "rcm_dish_controller"
 				(path "/10d7c3e5-be4d-4306-a59e-500b86bd141f/f4424325-c15a-4f12-b98c-68501db44bed/2b73156f-617f-4ddb-9603-19922a26015d"
-					(reference "C65")
+					(reference "C53")
 					(unit 1)
 				)
@@
 		(dnp no)
 		(fields_autoplaced yes)
-		(property "Reference" "TP9"
+		(property "Reference" "TP8"
 			(at 237.49 101.5999 0)
 			(show_name no)
@@
 			(project "rcm_dish_controller"
 				(path "/10d7c3e5-be4d-4306-a59e-500b86bd141f/f4424325-c15a-4f12-b98c-68501db44bed/2b73156f-617f-4ddb-9603-19922a26015d"
-					(reference "TP9")
+					(reference "TP8")
 					(unit 1)
 				)
@@
 		(in_pos_files yes)
 		(dnp no)
-		(property "Reference" "#PWR075"
+		(property "Reference" "#PWR074"
 			(at 52.07 151.13 0)
 			(hide yes)
@@
 			(project "rcm_dish_controller"
 				(path "/10d7c3e5-be4d-4306-a59e-500b86bd141f/f4424325-c15a-4f12-b98c-68501db44bed/2b73156f-617f-4ddb-9603-19922a26015d"
-					(reference "#PWR075")
+					(reference "#PWR074")
 					(unit 1)
 				)
@@
 		(in_pos_files yes)
 		(dnp no)
-		(property "Reference" "C76"
+		(property "Reference" "C64"
 			(at 106.426 134.874 90)
 			(show_name no)
@@
 			(project "rcm_dish_controller"
 				(path "/10d7c3e5-be4d-4306-a59e-500b86bd141f/f4424325-c15a-4f12-b98c-68501db44bed/2b73156f-617f-4ddb-9603-19922a26015d"
-					(reference "C76")
+					(reference "C64")
 					(unit 1)
 				)
@@
 		(in_pos_files yes)
 		(dnp no)
-		(property "Reference" "C73"
+		(property "Reference" "C61"
 			(at 75.946 134.874 90)
 			(show_name no)
@@
 			(project "rcm_dish_controller"
 				(path "/10d7c3e5-be4d-4306-a59e-500b86bd141f/f4424325-c15a-4f12-b98c-68501db44bed/2b73156f-617f-4ddb-9603-19922a26015d"
-					(reference "C73")
+					(reference "C61")
 					(unit 1)
 				)
@@
 		(in_pos_files yes)
 		(dnp no)
-		(property "Reference" "U8"
+		(property "Reference" "U7"
 			(at 125.73 129.032 0)
 			(show_name no)
@@
 			(project "rcm_dish_controller"
 				(path "/10d7c3e5-be4d-4306-a59e-500b86bd141f/f4424325-c15a-4f12-b98c-68501db44bed/2b73156f-617f-4ddb-9603-19922a26015d"
-					(reference "U8")
+					(reference "U7")
 					(unit 1)
 				)
@@
 		(in_pos_files yes)
 		(dnp no)
-		(property "Reference" "C68"
+		(property "Reference" "C56"
 			(at 215.646 120.0149 90)
 			(show_name no)
@@
 			(project "rcm_dish_controller"
 				(path "/10d7c3e5-be4d-4306-a59e-500b86bd141f/f4424325-c15a-4f12-b98c-68501db44bed/2b73156f-617f-4ddb-9603-19922a26015d"
-					(reference "C68")
+					(reference "C56")
 					(unit 1)
 				)
@@
 		(in_pos_files yes)
 		(dnp no)
-		(property "Reference" "C79"
+		(property "Reference" "C67"
 			(at 155.702 147.32 90)
 			(show_name no)
@@
 			(project "rcm_dish_controller"
 				(path "/10d7c3e5-be4d-4306-a59e-500b86bd141f/f4424325-c15a-4f12-b98c-68501db44bed/2b73156f-617f-4ddb-9603-19922a26015d"
-					(reference "C79")
+					(reference "C67")
 					(unit 1)
 				)
