File: kicad/user_switches.kicad_sch (KiCad schematic)
At the start: 17 parts, among them CN14 KF2EDGR-2.54-6P

Commit message: CM4 schematic changes, before renumbering
Parts:
- CN14: MPN (none) -> KF2EDGR-2.54-6P; Manufacturer (none) -> KEFA(科发)
Changed lines of the file:
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@@
 	(title_block
 		(title "User Switches")
-		(date "2026-07-11")
-		(rev "1.1")
+		(date "2026-08-18")
+		(rev "2.0")
 		(company "JRSeti")
 	)
@@
 		)
 	)
-	(global_label "USER_SW_2_MCU"
-		(shape input)
-		(at 140.97 78.74 0)
-		(fields_autoplaced yes)
-		(effects
-			(font
-				(size 1.27 1.27)
-			)
-			(justify left)
-		)
-		(property "Intersheetrefs" "${INTERSHEET_REFS}"
-			(at 159.7393 78.74 0)
-			(hide yes)
-			(show_name no)
-			(do_not_autoplace no)
-			(effects
-				(font
-					(size 1.27 1.27)
-				)
-				(justify left)
-			)
-		)
-	)
 	(global_label "3V3"
 		(shape input)
@@
 		)
 	)
-	(global_label "USER_SW_1_MCU"
-		(shape input)
-		(at 140.97 48.26 0)
-		(fields_autoplaced yes)
-		(effects
-			(font
-				(size 1.27 1.27)
-			)
-			(justify left)
-		)
-		(property "Intersheetrefs" "${INTERSHEET_REFS}"
-			(at 159.7393 48.26 0)
-			(hide yes)
-			(show_name no)
-			(do_not_autoplace no)
-			(effects
-				(font
-					(size 1.27 1.27)
-				)
-				(justify left)
-			)
-		)
-	)
-	(global_label "USER_SW_4_MCU"
-		(shape input)
-		(at 142.24 140.97 0)
-		(fields_autoplaced yes)
-		(effects
-			(font
-				(size 1.27 1.27)
-			)
-			(justify left)
-		)
-		(property "Intersheetrefs" "${INTERSHEET_REFS}"
-			(at 161.0093 140.97 0)
-			(hide yes)
-			(show_name no)
-			(do_not_autoplace no)
-			(effects
-				(font
-					(size 1.27 1.27)
-				)
-				(justify left)
-			)
-		)
-	)
 	(global_label "3V3"
 		(shape input)
@@
 		)
 	)
-	(global_label "USER_SW_3_MCU"
-		(shape input)
-		(at 140.97 109.22 0)
-		(fields_autoplaced yes)
+	(hierarchical_label "USER_SW_2_MCU"
+		(shape output)
+		(at 140.97 78.74 0)
 		(effects
 			(font
@@
 			(justify left)
 		)
-		(property "Intersheetrefs" "${INTERSHEET_REFS}"
-			(at 159.7393 109.22 0)
-			(hide yes)
-			(show_name no)
-			(do_not_autoplace no)
-			(effects
-				(font
-					(size 1.27 1.27)
-				)
-				(justify left)
-			)
+	)
+	(hierarchical_label "USER_SW_1_MCU"
+		(shape output)
+		(at 140.97 48.26 0)
+		(effects
+			(font
+				(size 1.27 1.27)
+			)
+			(justify left)
+		)
+	)
+	(hierarchical_label "USER_SW_4_MCU"
+		(shape output)
+		(at 142.24 140.97 0)
+		(effects
+			(font
+				(size 1.27 1.27)
+			)
+			(justify left)
+		)
+	)
+	(hierarchical_label "USER_SW_3_MCU"
+		(shape output)
+		(at 140.97 109.22 0)
+		(effects
+			(font
+				(size 1.27 1.27)
+			)
+			(justify left)
 		)
 	)
@@
 	(symbol
 		(lib_id "MyParts:KF2EDGR-2.54-6P")
-		(at 86.36 54.61 0)
+		(at 87.63 54.61 0)
 		(mirror y)
 		(unit 1)
@@
 		(dnp no)
 		(property "Reference" "CN14"
-			(at 88.646 44.196 0)
+			(at 89.916 44.196 0)
 			(show_name no)
 			(do_not_autoplace no)
@@
 		)
 		(property "Value" "KF2EDGR-2.54-6P"
-			(at 88.392 65.278 0)
+			(at 89.662 65.278 0)
 			(show_name no)
 			(do_not_autoplace no)
@@
 		)
 		(property "Footprint" "MyParts:CONN-TH_KF2EDGR-2.54-6P"
-			(at 86.36 68.58 0)
-			(hide yes)
-			(show_name no)
-			(do_not_autoplace no)
-			(effects
-				(font
-					(size 1.27 1.27)
-				)
-			)
-		)
-		(property "Datasheet" "https://www.lcsc.com/datasheet/C577598.pdf?spm=wm.sxq.inf.ggs&lcsc_vid=FFBaV1wHQFldUVICFgBfBVJTQVJWXgBfEQRYBAFQE1YxVlNRQFRcVVJfR1FdVTtW"
-			(at 86.36 71.12 0)
+			(at 87.63 68.58 0)
+			(hide yes)
+			(show_name no)
+			(do_not_autoplace no)
+			(effects
+				(font
+					(size 1.27 1.27)
+				)
+			)
+		)
+		(property "Datasheet" "https://lcsc.com/product-detail/Pluggable-System-Terminal-Block_Cixi-Kefa-Elec-KF2EDGR-2-54-6P_C577598.html"
+			(at 87.63 71.12 0)
 			(hide yes)
 			(show_name no)
@@
 		)
 		(property "Description" "6 Position Board Side/Socket - Closed 2.54mm Pitch Right-Angle Pin"
-			(at 86.36 54.61 0)
+			(at 87.63 54.61 0)
 			(hide yes)
 			(show_name no)
@@
 		)
 		(property "LCSC Part" "C577598"
-			(at 86.36 73.66 0)
-			(hide yes)
-			(show_name no)
+			(at 87.63 73.66 0)
+			(hide yes)
+			(show_name no)
+			(do_not_autoplace no)
+			(effects
+				(font
+					(size 1.27 1.27)
+				)
+			)
+		)
+		(property "Manufacturer" "KEFA(科发)"
+			(at 87.63 73.66 0)
+			(hide yes)
+			(show_name no)
+			(do_not_autoplace no)
+			(effects
+				(font
+					(size 1.27 1.27)
+				)
+			)
+		)
+		(property "MPN" "KF2EDGR-2.54-6P"
+			(at 87.63 76.2 0)
+			(hide yes)
+			(show_name no)

Commit message: Before adding CAN
Parts:
- renumbered C72 to C51, C73 to C52, C74 to C53, C75 to C54, CN14 to CN10, D12 to D29, D13 to D30, D14 to D31, D15 to D32, R47 to R61, R48 to R62, R49 to R63, R50 to R64, R51 to R65, R52 to R66, R53 to R67, R54 to R68
Changed lines of the file:
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@@
 		(in_pos_files yes)
 		(dnp no)
-		(property "Reference" "#PWR064"
+		(property "Reference" "#PWR060"
 			(at 139.7 67.31 0)
 			(hide yes)
@@
 			(project "rcm_dish_controller"
 				(path "/10d7c3e5-be4d-4306-a59e-500b86bd141f/7fa68ebc-abbe-49d0-8996-6dde5383e808"
-					(reference "#PWR064")
+					(reference "#PWR060")
 					(unit 1)
 				)
@@
 		(in_pos_files yes)
 		(dnp no)
-		(property "Reference" "D13"
+		(property "Reference" "D30"
 			(at 130.81 84.582 90)
 			(show_name no)
@@
 			(project "rcm_dish_controller"
 				(path "/10d7c3e5-be4d-4306-a59e-500b86bd141f/7fa68ebc-abbe-49d0-8996-6dde5383e808"
-					(reference "D13")
+					(reference "D30")
 					(unit 1)
 				)
@@
 		(in_pos_files yes)
 		(dnp no)
-		(property "Reference" "R50"
+		(property "Reference" "R64"
 			(at 134.874 76.708 90)
 			(show_name no)
@@
 			(project "rcm_dish_controller"
 				(path "/10d7c3e5-be4d-4306-a59e-500b86bd141f/7fa68ebc-abbe-49d0-8996-6dde5383e808"
-					(reference "R50")
+					(reference "R64")
 					(unit 1)
 				)
@@
 		(dnp no)
 		(fields_autoplaced yes)
-		(property "Reference" "C75"
+		(property "Reference" "C54"
 			(at 143.51 143.5099 0)
 			(show_name no)
@@
 			(project "rcm_dish_controller"
 				(path "/10d7c3e5-be4d-4306-a59e-500b86bd141f/7fa68ebc-abbe-49d0-8996-6dde5383e808"
-					(reference "C75")
+					(reference "C54")
 					(unit 1)
 				)
@@
 		(dnp no)
 		(fields_autoplaced yes)
-		(property "Reference" "C74"
+		(property "Reference" "C53"
 			(at 142.24 111.7599 0)
 			(show_name no)
@@
 			(project "rcm_dish_controller"
 				(path "/10d7c3e5-be4d-4306-a59e-500b86bd141f/7fa68ebc-abbe-49d0-8996-6dde5383e808"
-					(reference "C74")
+					(reference "C53")
 					(unit 1)
 				)
@@
 		(in_pos_files yes)
 		(dnp no)
-		(property "Reference" "#PWR066"
+		(property "Reference" "#PWR061"
 			(at 139.7 97.79 0)
 			(hide yes)
@@
 			(project "rcm_dish_controller"
 				(path "/10d7c3e5-be4d-4306-a59e-500b86bd141f/7fa68ebc-abbe-49d0-8996-6dde5383e808"
-					(reference "#PWR066")
+					(reference "#PWR061")
 					(unit 1)
 				)
@@
 		(in_pos_files yes)
 		(dnp no)
-		(property "Reference" "R51"
+		(property "Reference" "R65"
 			(at 129.794 104.14 0)
 			(show_name no)
@@
 			(project "rcm_dish_controller"
 				(path "/10d7c3e5-be4d-4306-a59e-500b86bd141f/7fa68ebc-abbe-49d0-8996-6dde5383e808"
-					(reference "R51")
+					(reference "R65")
 					(unit 1)
 				)
@@
 		(in_pos_files yes)
 		(dnp no)
-		(property "Reference" "#PWR067"
+		(property "Reference" "#PWR062"
 			(at 139.7 128.27 0)
 			(hide yes)
@@
 			(project "rcm_dish_controller"
 				(path "/10d7c3e5-be4d-4306-a59e-500b86bd141f/7fa68ebc-abbe-49d0-8996-6dde5383e808"
-					(reference "#PWR067")
+					(reference "#PWR062")
 					(unit 1)
 				)
@@
 		(in_pos_files yes)
 		(dnp no)
-		(property "Reference" "R54"
+		(property "Reference" "R68"
 			(at 136.144 138.684 90)
 			(show_name no)
@@
 			(project "rcm_dish_controller"
 				(path "/10d7c3e5-be4d-4306-a59e-500b86bd141f/7fa68ebc-abbe-49d0-8996-6dde5383e808"
-					(reference "R54")
+					(reference "R68")
 					(unit 1)
 				)
@@
 		(in_pos_files yes)
 		(dnp no)
-		(property "Reference" "#PWR065"
+		(property "Reference" "#PWR059"
 			(at 107.95 66.04 0)
 			(hide yes)
@@
 			(project "rcm_dish_controller"
 				(path "/10d7c3e5-be4d-4306-a59e-500b86bd141f/7fa68ebc-abbe-49d0-8996-6dde5383e808"
-					(reference "#PWR065")
+					(reference "#PWR059")
 					(unit 1)
 				)
@@
 		(in_pos_files yes)
 		(dnp no)
-		(property "Reference" "CN14"
+		(property "Reference" "CN10"
 			(at 89.916 44.196 0)
 			(show_name no)
@@
 			(project "rcm_dish_controller"
 				(path "/10d7c3e5-be4d-4306-a59e-500b86bd141f/7fa68ebc-abbe-49d0-8996-6dde5383e808"
-					(reference "CN14")
+					(reference "CN10")
 					(unit 1)
 				)
@@
 		(in_pos_files yes)
 		(dnp no)
-		(property "Reference" "D14"
+		(property "Reference" "D31"
 			(at 130.81 115.062 90)
 			(show_name no)
@@
 			(project "rcm_dish_controller"
 				(path "/10d7c3e5-be4d-4306-a59e-500b86bd141f/7fa68ebc-abbe-49d0-8996-6dde5383e808"
-					(reference "D14")
+					(reference "D31")
 					(unit 1)
 				)
@@
 		(in_pos_files yes)
 		(dnp no)
-		(property "Reference" "R53"
+		(property "Reference" "R67"
 			(at 131.318 135.636 0)
 			(show_name no)
@@
 			(project "rcm_dish_controller"
 				(path "/10d7c3e5-be4d-4306-a59e-500b86bd141f/7fa68ebc-abbe-49d0-8996-6dde5383e808"
-					(reference "R53")
+					(reference "R67")
 					(unit 1)
 				)
@@
 		(in_pos_files yes)
 		(dnp no)
-		(property "Reference" "D15"
+		(property "Reference" "D32"
 			(at 132.08 146.812 90)
 			(show_name no)
@@
 			(project "rcm_dish_controller"
 				(path "/10d7c3e5-be4d-4306-a59e-500b86bd141f/7fa68ebc-abbe-49d0-8996-6dde5383e808"
-					(reference "D15")
+					(reference "D32")
 					(unit 1)
 				)
@@
 		(in_pos_files yes)
 		(dnp no)
-		(property "Reference" "R52"
+		(property "Reference" "R66"
 			(at 134.62 106.934 90)
 			(show_name no)
@@
 			(project "rcm_dish_controller"
 				(path "/10d7c3e5-be4d-4306-a59e-500b86bd141f/7fa68ebc-abbe-49d0-8996-6dde5383e808"
-					(reference "R52")
+					(reference "R66")
 					(unit 1)
 				)
@@
 		(in_pos_files yes)
 		(dnp no)
-		(property "Reference" "R48"
+		(property "Reference" "R62"
 			(at 134.366 46.228 90)
 			(show_name no)
@@
 			(project "rcm_dish_controller"
 				(path "/10d7c3e5-be4d-4306-a59e-500b86bd141f/7fa68ebc-abbe-49d0-8996-6dde5383e808"
-					(reference "R48")
+					(reference "R62")
 					(unit 1)
 				)
@@
 		(dnp no)
 		(fields_autoplaced yes)
-		(property "Reference" "C73"
+		(property "Reference" "C52"
 			(at 142.24 81.2799 0)
 			(show_name no)
@@
 			(project "rcm_dish_controller"
 				(path "/10d7c3e5-be4d-4306-a59e-500b86bd141f/7fa68ebc-abbe-49d0-8996-6dde5383e808"
-					(reference "C73")
+					(reference "C52")
 					(unit 1)
 				)
@@
 		(in_pos_files yes)
 		(dnp no)
-		(property "Reference" "R49"
+		(property "Reference" "R63"
 			(at 130.048 73.66 0)
 			(show_name no)
@@
 			(project "rcm_dish_controller"
 				(path "/10d7c3e5-be4d-4306-a59e-500b86bd141f/7fa68ebc-abbe-49d0-8996-6dde5383e808"
-					(reference "R49")
+					(reference "R63")
 					(unit 1)
 				)
@@
 		(in_pos_files yes)
 		(dnp no)
-		(property "Reference" "#PWR068"
+		(property "Reference" "#PWR063"
 			(at 140.97 160.02 0)
 			(hide yes)
@@
 			(project "rcm_dish_controller"
 				(path "/10d7c3e5-be4d-4306-a59e-500b86bd141f/7fa68ebc-abbe-49d0-8996-6dde5383e808"
-					(reference "#PWR068")
+					(reference "#PWR063")
 					(unit 1)
 				)
@@
 		(dnp no)
 		(fields_autoplaced yes)
-		(property "Reference" "C72"
+		(property "Reference" "C51"
 			(at 142.24 50.7999 0)
 			(show_name no)
@@
 			(project "rcm_dish_controller"
 				(path "/10d7c3e5-be4d-4306-a59e-500b86bd141f/7fa68ebc-abbe-49d0-8996-6dde5383e808"
-					(reference "C72")
+					(reference "C51")
 					(unit 1)
 				)
@@
 		(in_pos_files yes)
 		(dnp no)
-		(property "Reference" "R47"
+		(property "Reference" "R61"
 			(at 130.048 43.18 0)
 			(show_name no)
@@
 			(project "rcm_dish_controller"
 				(path "/10d7c3e5-be4d-4306-a59e-500b86bd141f/7fa68ebc-abbe-49d0-8996-6dde5383e808"
-					(reference "R47")
+					(reference "R61")
 					(unit 1)
 				)
@@
 		(in_pos_files yes)
 		(dnp no)
-		(property "Reference" "D12"
+		(property "Reference" "D29"
 			(at 130.81 54.102 90)
 			(show_name no)
@@
 			(project "rcm_dish_controller"
 				(path "/10d7c3e5-be4d-4306-a59e-500b86bd141f/7fa68ebc-abbe-49d0-8996-6dde5383e808"
-					(reference "D12")
+					(reference "D29")
 					(unit 1)
 				)

Commit message: Add CAN JR45 - still working on it
Parts:
- renumbered C51 to C39, C52 to C40, C53 to C41, C54 to C42, CN10 to CN9, D29 to D35, D30 to D36, D31 to D37, D32 to D38, R61 to R59, R62 to R60, R63 to R61, R64 to R62, R65 to R63, R66 to R64, R67 to R65, R68 to R66
Changed lines of the file:
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@@
 		(in_pos_files yes)
 		(dnp no)
-		(property "Reference" "#PWR060"
+		(property "Reference" "#PWR059"
 			(at 139.7 67.31 0)
 			(hide yes)
@@
 			(project "rcm_dish_controller"
 				(path "/10d7c3e5-be4d-4306-a59e-500b86bd141f/7fa68ebc-abbe-49d0-8996-6dde5383e808"
-					(reference "#PWR060")
+					(reference "#PWR059")
 					(unit 1)
 				)
@@
 		(in_pos_files yes)
 		(dnp no)
-		(property "Reference" "D30"
+		(property "Reference" "D36"
 			(at 130.81 84.582 90)
 			(show_name no)
@@
 			(project "rcm_dish_controller"
 				(path "/10d7c3e5-be4d-4306-a59e-500b86bd141f/7fa68ebc-abbe-49d0-8996-6dde5383e808"
-					(reference "D30")
+					(reference "D36")
 					(unit 1)
 				)
@@
 		(in_pos_files yes)
 		(dnp no)
-		(property "Reference" "R64"
+		(property "Reference" "R62"
 			(at 134.874 76.708 90)
 			(show_name no)
@@
 			(project "rcm_dish_controller"
 				(path "/10d7c3e5-be4d-4306-a59e-500b86bd141f/7fa68ebc-abbe-49d0-8996-6dde5383e808"
-					(reference "R64")
+					(reference "R62")
 					(unit 1)
 				)
@@
 		(dnp no)
 		(fields_autoplaced yes)
-		(property "Reference" "C54"
+		(property "Reference" "C42"
 			(at 143.51 143.5099 0)
 			(show_name no)
@@
 			(project "rcm_dish_controller"
 				(path "/10d7c3e5-be4d-4306-a59e-500b86bd141f/7fa68ebc-abbe-49d0-8996-6dde5383e808"
-					(reference "C54")
+					(reference "C42")
 					(unit 1)
 				)
@@
 		(dnp no)
 		(fields_autoplaced yes)
-		(property "Reference" "C53"
+		(property "Reference" "C41"
 			(at 142.24 111.7599 0)
 			(show_name no)
@@
 			(project "rcm_dish_controller"
 				(path "/10d7c3e5-be4d-4306-a59e-500b86bd141f/7fa68ebc-abbe-49d0-8996-6dde5383e808"
-					(reference "C53")
+					(reference "C41")
 					(unit 1)
 				)
@@
 		(in_pos_files yes)
 		(dnp no)
-		(property "Reference" "#PWR061"
+		(property "Reference" "#PWR060"
 			(at 139.7 97.79 0)
 			(hide yes)
@@
 			(project "rcm_dish_controller"
 				(path "/10d7c3e5-be4d-4306-a59e-500b86bd141f/7fa68ebc-abbe-49d0-8996-6dde5383e808"
-					(reference "#PWR061")
+					(reference "#PWR060")
 					(unit 1)
 				)
@@
 		(in_pos_files yes)
 		(dnp no)
-		(property "Reference" "R65"
+		(property "Reference" "R63"
 			(at 129.794 104.14 0)
 			(show_name no)
@@
 			(project "rcm_dish_controller"
 				(path "/10d7c3e5-be4d-4306-a59e-500b86bd141f/7fa68ebc-abbe-49d0-8996-6dde5383e808"
-					(reference "R65")
+					(reference "R63")
 					(unit 1)
 				)
@@
 		(in_pos_files yes)
 		(dnp no)
-		(property "Reference" "#PWR062"
+		(property "Reference" "#PWR061"
 			(at 139.7 128.27 0)
 			(hide yes)
@@
 			(project "rcm_dish_controller"
 				(path "/10d7c3e5-be4d-4306-a59e-500b86bd141f/7fa68ebc-abbe-49d0-8996-6dde5383e808"
-					(reference "#PWR062")
+					(reference "#PWR061")
 					(unit 1)
 				)
@@
 		(in_pos_files yes)
 		(dnp no)
-		(property "Reference" "R68"
+		(property "Reference" "R66"
 			(at 136.144 138.684 90)
 			(show_name no)
@@
 			(project "rcm_dish_controller"
 				(path "/10d7c3e5-be4d-4306-a59e-500b86bd141f/7fa68ebc-abbe-49d0-8996-6dde5383e808"
-					(reference "R68")
+					(reference "R66")
 					(unit 1)
 				)
@@
 		(in_pos_files yes)
 		(dnp no)
-		(property "Reference" "#PWR059"
+		(property "Reference" "#PWR058"
 			(at 107.95 66.04 0)
 			(hide yes)
@@
 			(project "rcm_dish_controller"
 				(path "/10d7c3e5-be4d-4306-a59e-500b86bd141f/7fa68ebc-abbe-49d0-8996-6dde5383e808"
-					(reference "#PWR059")
+					(reference "#PWR058")
 					(unit 1)
 				)
@@
 		(in_pos_files yes)
 		(dnp no)
-		(property "Reference" "CN10"
+		(property "Reference" "CN9"
 			(at 89.916 44.196 0)
 			(show_name no)
@@
 			(project "rcm_dish_controller"
 				(path "/10d7c3e5-be4d-4306-a59e-500b86bd141f/7fa68ebc-abbe-49d0-8996-6dde5383e808"
-					(reference "CN10")
+					(reference "CN9")
 					(unit 1)
 				)
@@
 		(in_pos_files yes)
 		(dnp no)
-		(property "Reference" "D31"
+		(property "Reference" "D37"
 			(at 130.81 115.062 90)
 			(show_name no)
@@
 			(project "rcm_dish_controller"
 				(path "/10d7c3e5-be4d-4306-a59e-500b86bd141f/7fa68ebc-abbe-49d0-8996-6dde5383e808"
-					(reference "D31")
+					(reference "D37")
 					(unit 1)
 				)
@@
 		(in_pos_files yes)
 		(dnp no)
-		(property "Reference" "R67"
+		(property "Reference" "R65"
 			(at 131.318 135.636 0)
 			(show_name no)
@@
 			(project "rcm_dish_controller"
 				(path "/10d7c3e5-be4d-4306-a59e-500b86bd141f/7fa68ebc-abbe-49d0-8996-6dde5383e808"
-					(reference "R67")
+					(reference "R65")
 					(unit 1)
 				)
@@
 		(in_pos_files yes)
 		(dnp no)
-		(property "Reference" "D32"
+		(property "Reference" "D38"
 			(at 132.08 146.812 90)
 			(show_name no)
@@
 			(project "rcm_dish_controller"
 				(path "/10d7c3e5-be4d-4306-a59e-500b86bd141f/7fa68ebc-abbe-49d0-8996-6dde5383e808"
-					(reference "D32")
+					(reference "D38")
 					(unit 1)
 				)
@@
 		(in_pos_files yes)
 		(dnp no)
-		(property "Reference" "R66"
+		(property "Reference" "R64"
 			(at 134.62 106.934 90)
 			(show_name no)
@@
 			(project "rcm_dish_controller"
 				(path "/10d7c3e5-be4d-4306-a59e-500b86bd141f/7fa68ebc-abbe-49d0-8996-6dde5383e808"
-					(reference "R66")
+					(reference "R64")
 					(unit 1)
 				)
@@
 		(in_pos_files yes)
 		(dnp no)
-		(property "Reference" "R62"
+		(property "Reference" "R60"
 			(at 134.366 46.228 90)
 			(show_name no)
@@
 			(project "rcm_dish_controller"
 				(path "/10d7c3e5-be4d-4306-a59e-500b86bd141f/7fa68ebc-abbe-49d0-8996-6dde5383e808"
-					(reference "R62")
+					(reference "R60")
 					(unit 1)
 				)
@@
 		(dnp no)
 		(fields_autoplaced yes)
-		(property "Reference" "C52"
+		(property "Reference" "C40"
 			(at 142.24 81.2799 0)
 			(show_name no)
@@
 			(project "rcm_dish_controller"
 				(path "/10d7c3e5-be4d-4306-a59e-500b86bd141f/7fa68ebc-abbe-49d0-8996-6dde5383e808"
-					(reference "C52")
+					(reference "C40")
 					(unit 1)
 				)
@@
 		(in_pos_files yes)
 		(dnp no)
-		(property "Reference" "R63"
+		(property "Reference" "R61"
 			(at 130.048 73.66 0)
 			(show_name no)
@@
 			(project "rcm_dish_controller"
 				(path "/10d7c3e5-be4d-4306-a59e-500b86bd141f/7fa68ebc-abbe-49d0-8996-6dde5383e808"
-					(reference "R63")
+					(reference "R61")
 					(unit 1)
 				)
@@
 		(in_pos_files yes)
 		(dnp no)
-		(property "Reference" "#PWR063"
+		(property "Reference" "#PWR062"
 			(at 140.97 160.02 0)
 			(hide yes)
@@
 			(project "rcm_dish_controller"
 				(path "/10d7c3e5-be4d-4306-a59e-500b86bd141f/7fa68ebc-abbe-49d0-8996-6dde5383e808"
-					(reference "#PWR063")
+					(reference "#PWR062")
 					(unit 1)
 				)
@@
 		(dnp no)
 		(fields_autoplaced yes)
-		(property "Reference" "C51"
+		(property "Reference" "C39"
 			(at 142.24 50.7999 0)
 			(show_name no)
@@
 			(project "rcm_dish_controller"
 				(path "/10d7c3e5-be4d-4306-a59e-500b86bd141f/7fa68ebc-abbe-49d0-8996-6dde5383e808"
-					(reference "C51")
+					(reference "C39")
 					(unit 1)
 				)
@@
 		(in_pos_files yes)
 		(dnp no)
-		(property "Reference" "R61"
+		(property "Reference" "R59"
 			(at 130.048 43.18 0)
 			(show_name no)
@@
 			(project "rcm_dish_controller"
 				(path "/10d7c3e5-be4d-4306-a59e-500b86bd141f/7fa68ebc-abbe-49d0-8996-6dde5383e808"
-					(reference "R61")
+					(reference "R59")
 					(unit 1)
 				)
@@
 		(in_pos_files yes)
 		(dnp no)
-		(property "Reference" "D29"
+		(property "Reference" "D35"
 			(at 130.81 54.102 90)
 			(show_name no)
@@
 			(project "rcm_dish_controller"
 				(path "/10d7c3e5-be4d-4306-a59e-500b86bd141f/7fa68ebc-abbe-49d0-8996-6dde5383e808"
-					(reference "D29")
+					(reference "D35")
 					(unit 1)
 				)
