File: kicad/RCM4.kicad_sch (KiCad schematic)
At the start: 0 parts

Commit message: Working on CM4 IO
Parts:
- added LED3: XL-0805QBC, MyParts:LED0805-R-RD, symbol MyParts:XL-0805QBC
- added Module1: ComputeModule4-CM4, CM4IO:Raspberry-Pi-4-Compute-Module, symbol CM4_Parts:ComputeModule4-CM4
- added R20: 1.5kΩ, PCM_JLCPCB:R_0402, symbol PCM_JLCPCB-Resistors:0402,1.5kΩ
Connections:
- new net: Module1.21 (PI_nLED_Activity), R20.2
- new net: LED3.2 (K), R20.1
- new net 1PPS_MCU: Module1.29 (GPIO16)
- new net 3V3_CM4: Module1.78 (GPIO_VREF(1.8v/3.3v_Input)), Module1.84 (+3.3v_(Output)), Module1.86 (+3.3v_(Output))
- new net 5V: LED3.1 (A), Module1.77 (+5v_(Input)), Module1.79 (+5v_(Input)), Module1.81 (+5v_(Input)), Module1.83 (+5v_(Input)), Module1.85 (+5v_(Input)), Module1.87 (+5v_(Input))
- new net AIN0: Module1.96 (AnalogIP0)
- new net AIN1: Module1.94 (AnalogIP1)
- new net EEPROM_nWP: Module1.20 (EEPROM_nWP)
- new net EP0+: Module1.12 (Ethernet_Pair0_P)
- new net EP0-: Module1.10 (Ethernet_Pair0_N)
- new net EP1+: Module1.4 (Ethernet_Pair1_P)
- new net EP1-: Module1.6 (Ethernet_Pair1_N)
- new net EP2+: Module1.11 (Ethernet_Pair2_P)
- new net EP2-: Module1.9 (Ethernet_Pair2_N)
- new net EP3+: Module1.3 (Ethernet_Pair3_P)
- new net EP3-: Module1.5 (Ethernet_Pair3_N)
- new net ETH_LEDG: Module1.17 (Ethernet_nLED2(3.3v))
- new net ETH_LEDY: Module1.15 (Ethernet_nLED3(3.3v))
- new net GLOBAL_EN: Module1.99 (Global_EN)
- new net GND: Module1.1 (GND), Module1.107 (GND), Module1.108 (GND), Module1.113 (GND), Module1.114 (GND), Module1.119 (GND), Module1.120 (GND), Module1.125 (GND), Module1.126 (GND), Module1.13 (GND), Module1.131 (GND), Module1.132 (GND), Module1.137 (GND), Module1.138 (GND), Module1.14 (GND), Module1.144 (GND), Module1.150 (GND), Module1.155 (GND), Module1.156 (GND), Module1.161 (GND), Module1.162 (GND), Module1.167 (GND), Module1.168 (GND), Module1.173 (GND), Module1.174 (GND), Module1.179 (GND), Module1.180 (GND), Module1.185 (GND), Module1.186 (GND), Module1.191 (GND), Module1.192 (GND), Module1.197 (GND), Module1.198 (GND), Module1.2 (GND), Module1.22 (GND), Module1.23 (GND), Module1.32 (GND), Module1.33 (GND), Module1.42 (GND), Module1.43 (GND), Module1.52 (GND), Module1.53 (GND), Module1.59 (GND), Module1.60 (GND), Module1.65 (GND), Module1.66 (GND), Module1.7 (GND), Module1.71 (GND), Module1.74 (GND), Module1.8 (GND), Module1.98 (GND)
- new net RUN_PG: Module1.92 (RUN_PG)
- new net SCL0: Module1.80 (SCL0)
- new net SDA0: Module1.82 (SDA0)
- new net SPI0_CE0: Module1.39 (GPIO8)
- new net SPI0_CE1: Module1.37 (GPIO7)
- new net SPI0_MISO: Module1.40 (GPIO9)
- new net SPI0_MOSI: Module1.44 (GPIO10)
- new net SPI0_SCLK: Module1.38 (GPIO11)
- new net STM32_USART1_RX: Module1.54 (GPIO4)
- new net STM32_USART1_TX: Module1.34 (GPIO5)
- new net UART0_RXD: Module1.51 (GPIO15)
- new net UART0_TXD: Module1.55 (GPIO14)
- new net USB2_N: Module1.103 (USB2_N)
- new net USB2_P: Module1.105 (USB2_P)
- new net USB_OTG_ID: Module1.101 (USB_OTG_ID)
- new net nEXTRST: Module1.100 (nEXTRST)
- new net nPWR_LED: Module1.95 (nPI_LED_PWR)
- new net nRPIBOOT: Module1.93 (nRPIBOOT)
- no-connect marks 0 -> 38
Other:
- added sheet CM4_Connectors (cm4_connectors.kicad_sch)
- added sheet ethernet (ethernet.kicad_sch)
- added sheet usb (usb.kicad_sch)
- note added: "1PPS from GPS"

Commit message: CM4 schematic changes, before renumbering
Parts:
- added R18, R46: 100Ω, PCM_JLCPCB:R_0402, symbol PCM_JLCPCB-Resistors:0402,100Ω
- Module1: footprint CM4IO:Raspberry-Pi-4-Compute-Module -> CM4_Parts:Raspberry-Pi-4-Compute-Module
Connections:
- net PWM1: now reaches Module1.28 (GPIO13)
- net PWM0: now reaches Module1.31 (GPIO12)
- net GPIO22: now reaches Module1.46 (GPIO22)
- net I2C1_SCL: now reaches Module1.56 (GPIO3)
- net I2C1_SDA: now reaches Module1.58 (GPIO2)
- net SCL0: no longer names the net of Module1.80 (SCL0)
- net SDA0: no longer names the net of Module1.82 (SDA0)
- net STM32_USART1_RX: no longer names the net of Module1.54 (GPIO4)
- net STM32_USART1_RX: now also R46.2
- net STM32_USART1_TX: no longer names the net of Module1.34 (GPIO5)
- net STM32_USART1_TX: now also R18.2
- net UART0_RXD renamed BOOT_CONSOLE_RXD
- net UART0_TXD renamed BOOT_CONSOLE_TXD
- new net CM4_RX: R46.1
- new net CM4_TX: R18.1
- no-connect marks 38 -> 103
Other:
- sheet CM4_Connectors ports: added AIN0, AIN1, BOOT_CONSOLE_RXD, BOOT_CONSOLE_TXD, EEPROM_nWP, GLOBAL_EN, GPIO22, I2C1_SCL, I2C1_SDA, PWM0, PWM1, RUN_PG, SPI0_CE0, SPI0_CE1, SPI0_MISO, SPI0_MOSI, SPI0_SCLK, nPWR_LED, nRPIBOOT; removed none
- sheet ethernet ports: added EP0+, EP0-, EP1+, EP1-, EP2+, EP2-, EP3+, EP3-, ETH_LEDG, ETH_LEDY; removed none
- sheet usb ports: added USB2_N, USB2_P, USB_OTG_ID, nEXTRST; removed none

Commit message: Before adding CAN
Parts:
- renumbered R20 to R69, R18 to R70, R46 to R71
Changed lines of the file:
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@@
 		(dnp no)
 		(fields_autoplaced yes)
-		(property "Reference" "#PWR09"
+		(property "Reference" "#PWR064"
 			(at 48.26 163.83 0)
 			(hide yes)
@@
 			(project "rcm_dish_controller"
 				(path "/10d7c3e5-be4d-4306-a59e-500b86bd141f/a4b43769-68f4-4111-a02f-817ae260783a"
-					(reference "#PWR09")
+					(reference "#PWR064")
 					(unit 1)
 				)
@@
 		(dnp no)
 		(fields_autoplaced yes)
-		(property "Reference" "#PWR031"
+		(property "Reference" "#PWR067"
 			(at 220.98 163.83 0)
 			(hide yes)
@@
 			(project "rcm_dish_controller"
 				(path "/10d7c3e5-be4d-4306-a59e-500b86bd141f/a4b43769-68f4-4111-a02f-817ae260783a"
-					(reference "#PWR031")
+					(reference "#PWR067")
 					(unit 1)
 				)
@@
 		(dnp no)
 		(fields_autoplaced yes)
-		(property "Reference" "#PWR012"
+		(property "Reference" "#PWR065"
 			(at 114.3 163.83 0)
 			(hide yes)
@@
 			(project "rcm_dish_controller"
 				(path "/10d7c3e5-be4d-4306-a59e-500b86bd141f/a4b43769-68f4-4111-a02f-817ae260783a"
-					(reference "#PWR012")
+					(reference "#PWR065")
 					(unit 1)
 				)
@@
 		(dnp no)
 		(fields_autoplaced yes)
-		(property "Reference" "R20"
+		(property "Reference" "R69"
 			(at 135.89 48.2599 0)
 			(show_name no)
@@
 			(project "rcm_dish_controller"
 				(path "/10d7c3e5-be4d-4306-a59e-500b86bd141f/a4b43769-68f4-4111-a02f-817ae260783a"
-					(reference "R20")
+					(reference "R69")
 					(unit 1)
 				)
@@
 		(dnp no)
 		(fields_autoplaced yes)
-		(property "Reference" "#PWR032"
+		(property "Reference" "#PWR066"
 			(at 154.94 163.83 0)
 			(hide yes)
@@
 			(project "rcm_dish_controller"
 				(path "/10d7c3e5-be4d-4306-a59e-500b86bd141f/a4b43769-68f4-4111-a02f-817ae260783a"
-					(reference "#PWR032")
+					(reference "#PWR066")
 					(unit 1)
 				)
@@
 		(in_pos_files yes)
 		(dnp no)
-		(property "Reference" "R18"
+		(property "Reference" "R70"
 			(at 43.434 66.294 90)
 			(show_name no)
@@
 			(project "rcm_dish_controller"
 				(path "/10d7c3e5-be4d-4306-a59e-500b86bd141f/a4b43769-68f4-4111-a02f-817ae260783a"
-					(reference "R18")
+					(reference "R70")
 					(unit 1)
 				)
@@
 		(in_pos_files yes)
 		(dnp no)
-		(property "Reference" "R46"
+		(property "Reference" "R71"
 			(at 43.434 91.694 90)
 			(show_name no)
@@
 			(project "rcm_dish_controller"
 				(path "/10d7c3e5-be4d-4306-a59e-500b86bd141f/a4b43769-68f4-4111-a02f-817ae260783a"
-					(reference "R46")
+					(reference "R71")
 					(unit 1)
 				)

Commit message: More mods
Parts:
- added R98: 100Ω, PCM_JLCPCB:R_0402, symbol PCM_JLCPCB-Resistors:0402,100Ω
- added R99: 10kΩ, PCM_JLCPCB:R_0402, symbol PCM_JLCPCB-Resistors:0402,10kΩ
Connections:
- net 3V3_CM4: now also R99.1
- net at Module1.30 (GPIO6): now also R98.2
- new net MCU_nIRQ: R98.1, R99.2
- no-connect marks 103 -> 102
Other:
- note added: "MCU_nIRQ (PD2 -> GPIO6): open-drain, active low. Set PD2 OUTPUT_OD; R99 idles the line high on 3V3_CM4. GPIO6 also powers up pulled high."

Commit message: CAN looks complete in schematic
Parts:
- removed LED3: XL-0805QBC, MyParts:LED0805-R-RD, symbol MyParts:XL-0805QBC
- added LED3: RED, MyParts:LED0805-R-RD, symbol MyParts:E6C0805UR
Connections:
- net 5V: now also LED3.1 (A)
- net at R69.1: now also LED3.2 (K)
Changed lines of the file:
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@@
+	)
+	(symbol
+		(lib_id "MyParts:E6C0805UR")
+		(at 134.62 38.1 270)
+		(mirror x)
+		(unit 1)
+		(body_style 1)
+		(exclude_from_sim no)
+		(in_bom yes)
+		(on_board yes)
+		(in_pos_files yes)
+		(dnp no)
+		(property "Reference" "LED3"
+			(at 136.906 37.338 90)
+			(show_name no)
+			(do_not_autoplace no)
+			(effects
+				(font
+					(size 1.27 1.27)
+				)
+				(justify left)
+			)
+		)
+		(property "Value" "RED"
+			(at 136.906 39.116 90)
+			(hide yes)
+			(show_name no)
+			(do_not_autoplace no)
+			(effects
+				(font
+					(size 1.27 1.27)
+				)
+				(justify left)
+			)
+		)
+		(property "Footprint" "MyParts:LED0805-R-RD"
+			(at 125.73 38.1 0)
+			(hide yes)
+			(show_name no)
+			(do_not_autoplace no)
+			(effects
+				(font
+					(size 1.27 1.27)
+				)
+			)
+		)
+		(property "Datasheet" "https://lcsc.com/product-detail/Light-Emitting-Diodes-LED_Red-LED-0805-Highlighted_C2295.html"
+			(at 123.19 38.1 0)
+			(hide yes)
+			(show_name no)
+			(do_not_autoplace no)
+			(effects
+				(font
+					(size 1.27 1.27)
+				)
+			)
+		)
+		(property "Description" "0805"
+			(at 110.49 38.1 0)
+			(hide yes)
+			(show_name no)
+			(do_not_autoplace no)
+			(effects
+				(font
+					(size 1.27 1.27)
+				)
+			)
+		)
+		(property "Manufacturer" "KENTO"
+			(at 120.65 38.1 0)
+			(hide yes)
+			(show_name no)
+			(do_not_autoplace no)
+			(effects
+				(font
+					(size 1.27 1.27)
+				)
+			)
+		)
+		(property "MPN" "KT-0805R"
+			(at 141.986 39.116 90)
+			(hide yes)
+			(show_name no)
+			(do_not_autoplace no)
+			(effects
+				(font
+					(size 1.27 1.27)
+				)
+			)
+		)
+		(property "LCSC Part" "C2295"
+			(at 115.57 38.1 0)
+			(hide yes)
+			(show_name no)
+			(do_not_autoplace no)
+			(effects
+				(font
+					(size 1.27 1.27)
+				)
+			)
+		)
+		(pin "1"
+		)
+		(pin "2"
+		)
+		(instances
+			(project "rcm_dish_controller"
+				(path "/10d7c3e5-be4d-4306-a59e-500b86bd141f/a4b43769-68f4-4111-a02f-817ae260783a"
+					(reference "LED3")
+					(unit 1)
+				)
+			)
+		)
 	)
 	(symbol
@@
 				)
 			)
-		)
-	)
-	(symbol
-		(lib_id "MyParts:XL-0805QBC")
-		(at 134.62 38.1 270)
-		(mirror x)
-		(unit 1)
-		(body_style 1)
-		(exclude_from_sim no)
-		(in_bom yes)
-		(on_board yes)
-		(in_pos_files yes)
-		(dnp no)
-		(fields_autoplaced yes)
-		(property "Reference" "LED3"
-			(at 138.43 38.0999 90)
-			(show_name no)
-			(do_not_autoplace no)
-			(effects
-				(font
-					(size 1.27 1.27)
-				)
-				(justify left)
-			)
-		)
-		(property "Value" "XL-0805QBC"
-			(at 138.43 40.6399 90)
-			(show_name no)
-			(do_not_autoplace no)
-			(effects
-				(font
-					(size 1.27 1.27)
-				)
-				(justify left)
-			)
-		)
-		(property "Footprint" "MyParts:LED0805-R-RD"
-			(at 125.73 38.1 0)
-			(hide yes)
-			(show_name no)
-			(do_not_autoplace no)
-			(effects
-				(font
-					(size 1.27 1.27)
-				)
-			)
-		)
-		(property "Datasheet" "https://lcsc.com/product-detail/Light-Emitting-Diodes-LED_Blue-light_C2293.html"
-			(at 123.19 38.1 0)
-			(hide yes)
-			(show_name no)
-			(do_not_autoplace no)
-			(effects
-				(font
-					(size 1.27 1.27)
-				)
-			)
-		)
-		(property "Description" ""
-			(at 134.62 38.1 0)
-			(hide yes)
-			(show_name no)
-			(do_not_autoplace no)
-			(effects
-				(font
-					(size 1.27 1.27)
-				)
-			)
-		)
-		(property "Manufacturer" "KENTO"
-			(at 120.65 38.1 0)
-			(hide yes)
-			(show_name no)
-			(do_not_autoplace no)
-			(effects
-				(font
-					(size 1.27 1.27)
-				)
-			)
-		)
-		(property "MPN" "KT-0805B"
-			(at 118.11 38.1 0)
-			(hide yes)
-			(show_name no)
-			(do_not_autoplace no)
-			(effects
-				(font
-					(size 1.27 1.27)
-				)
-			)
-		)
-		(property "LCSC Part" "C2293"
-			(at 115.57 38.1 0)
-			(hide yes)
-			(show_name no)
-			(do_not_autoplace no)
-			(effects
-				(font
-					(size 1.27 1.27)
-				)
-			)
-		)
-		(pin "1"
-		)
-		(pin "2"
-		)
-		(instances
-			(project "rcm_dish_controller"
-				(path "/10d7c3e5-be4d-4306-a59e-500b86bd141f/a4b43769-68f4-4111-a02f-817ae260783a"
-					(reference "LED3")
-					(unit 1)
-				)
-			)

Commit message: Add CAN JR45 - still working on it
Parts:
- renumbered R69 to R67, R99 to R68, R98 to R69
Changed lines of the file:
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@@
 		(dnp no)
 		(fields_autoplaced yes)
-		(property "Reference" "#PWR064"
+		(property "Reference" "#PWR063"
 			(at 48.26 163.83 0)
 			(hide yes)
@@
 			(project "rcm_dish_controller"
 				(path "/10d7c3e5-be4d-4306-a59e-500b86bd141f/a4b43769-68f4-4111-a02f-817ae260783a"
-					(reference "#PWR064")
+					(reference "#PWR063")
 					(unit 1)
 				)
@@
 		(dnp no)
 		(fields_autoplaced yes)
-		(property "Reference" "#PWR067"
+		(property "Reference" "#PWR066"
 			(at 220.98 163.83 0)
 			(hide yes)
@@
 			(project "rcm_dish_controller"
 				(path "/10d7c3e5-be4d-4306-a59e-500b86bd141f/a4b43769-68f4-4111-a02f-817ae260783a"
-					(reference "#PWR067")
+					(reference "#PWR066")
 					(unit 1)
 				)
@@
 		(dnp no)
 		(fields_autoplaced yes)
-		(property "Reference" "#PWR065"
+		(property "Reference" "#PWR064"
 			(at 114.3 163.83 0)
 			(hide yes)
@@
 			(project "rcm_dish_controller"
 				(path "/10d7c3e5-be4d-4306-a59e-500b86bd141f/a4b43769-68f4-4111-a02f-817ae260783a"
-					(reference "#PWR065")
+					(reference "#PWR064")
 					(unit 1)
 				)
@@
 		(in_pos_files yes)
 		(dnp no)
-		(property "Reference" "R98"
+		(property "Reference" "R69"
 			(at 36.83 61.976 90)
 			(show_name no)
@@
 			(project "rcm_dish_controller"
 				(path "/10d7c3e5-be4d-4306-a59e-500b86bd141f/a4b43769-68f4-4111-a02f-817ae260783a"
-					(reference "R98")
+					(reference "R69")
 					(unit 1)
 				)
@@
 		(dnp no)
 		(fields_autoplaced yes)
-		(property "Reference" "R69"
+		(property "Reference" "R67"
 			(at 135.89 48.2599 0)
 			(show_name no)
@@
 			(project "rcm_dish_controller"
 				(path "/10d7c3e5-be4d-4306-a59e-500b86bd141f/a4b43769-68f4-4111-a02f-817ae260783a"
-					(reference "R69")
+					(reference "R67")
 					(unit 1)
 				)
@@
 		(in_pos_files yes)
 		(dnp no)
-		(property "Reference" "R99"
+		(property "Reference" "R68"
 			(at 28.702 52.07 0)
 			(show_name no)
@@
 			(project "rcm_dish_controller"
 				(path "/10d7c3e5-be4d-4306-a59e-500b86bd141f/a4b43769-68f4-4111-a02f-817ae260783a"
-					(reference "R99")
+					(reference "R68")
 					(unit 1)
 				)
@@
 		(dnp no)
 		(fields_autoplaced yes)
-		(property "Reference" "#PWR066"
+		(property "Reference" "#PWR065"
 			(at 154.94 163.83 0)
 			(hide yes)
@@
 			(project "rcm_dish_controller"
 				(path "/10d7c3e5-be4d-4306-a59e-500b86bd141f/a4b43769-68f4-4111-a02f-817ae260783a"
-					(reference "#PWR066")
+					(reference "#PWR065")
 					(unit 1)
 				)

Commit message: Before removing CAN 24V
Parts:
- Module1: footprint CM4_Parts:Raspberry-Pi-4-Compute-Module -> CM4IO:Raspberry-Pi-4-Compute-Module
Changed lines of the file:
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@@
 			)
 		)
-		(property "Footprint" "CM4_Parts:Raspberry-Pi-4-Compute-Module"
+		(property "Footprint" "CM4IO:Raspberry-Pi-4-Compute-Module"
 			(at 226.06 110.49 0)
 			(hide yes)
@@
 			)
 		)
-		(property "Footprint" "CM4_Parts:Raspberry-Pi-4-Compute-Module"
+		(property "Footprint" "CM4IO:Raspberry-Pi-4-Compute-Module"
 			(at 190.5 115.57 0)
 			(hide yes)
