File: kicad/cm4_connectors.kicad_sch (KiCad schematic)
At the start: 8 parts, among them CN15 KF2EDGR-2.54-10P, J3 Header-Male-2.54_2x3, U14 2541WV-2X12P, U15 74LVC1G07SE-7, U16 74LVC1G07SE-7

Commit message: CM4 schematic changes, before renumbering
Parts:
- removed CN15: KF2EDGR-2.54-10P, MyParts:CONN-TH_10P-P2.54_KF2EDGR-2.54-10P, symbol MyParts:KF2EDGR-2.54-10P
- added H5, H6: 210S-1*2P L=11.6MMGold-plated black, MyParts:HDR-TH_2P-P2.54-V-M-1, symbol MyParts:210S-1*2PL=11.6MMGold-platedblack
- added R91, R93: 4.7kΩ, PCM_JLCPCB:R_0402, symbol PCM_JLCPCB-Resistors:0402,4.7kΩ
Connections:
- net 3V3_CM4: now also U14.7, R91.1, R93.1
- net 5V: now also U14.5; no longer U15.5 (VCC)
- net AIN0: now also U14.2; no longer U14.3
- net AIN1: now also U14.4; no longer U14.5
- net GND: now also U14.11, U14.13, U14.15, U14.17, U14.19, U14.21, U14.23, U14.3, U14.9; no longer U14.12
- net SPI0_CE0: now also U14.12; no longer U14.8
- net SPI0_CE1: now also U14.14; no longer U14.10
- net SPI0_MISO: now also U14.10; no longer U14.6
- net SPI0_MOSI: now also U14.8; no longer U14.4
- net SPI0_SCLK: now also U14.6; no longer U14.2
- net I2C1_SDA: now reaches U14.16
- net I2C1_SDA: now also H5.1
- net I2C1_SCL: now reaches U14.18
- net I2C1_SCL: now also H6.1
- net PWM0: now reaches U14.20
- net PWM1: now reaches U14.22
- net GPIO22: now reaches U14.24
- net UART0_RXD renamed BOOT_CONSOLE_RXD
- net UART0_TXD renamed BOOT_CONSOLE_TXD
- new net: H6.2, R93.2
- new net: H5.2, R91.2
- new net 3V3: U15.5 (VCC)
Other:
- note added: "Boot/EEPROM_EN/GLOBAL_EN"
- note added: "GPIO Headers"
- note added: "GPIO10"
- note added: "GPIO11"
- note added: "GPIO12"
- note added: "GPIO13"
- note added: "GPIO2"
- note added: "GPIO3"
- note added: "GPIO7"
- note added: "GPIO8"
- note added: "GPIO9"
- note added: "I2C Pull-Ups"
- note added: "Power-On LED"
- note removed: "GPIO"
- moved on the sheet: H1, J3, R92, U14, U15, U16

Commit message: Before adding CAN
Parts:
- renumbered H1 to H3, H5 to H4, H6 to H5, J3 to J2, R92 to R91, R91 to R92, U14 to U17
Changed lines of the file:
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@@
 		(dnp no)
 		(fields_autoplaced yes)
-		(property "Reference" "#PWR0103"
+		(property "Reference" "#PWR0104"
 			(at 165.1 137.16 0)
 			(hide yes)
@@
 			(project "rcm_dish_controller"
 				(path "/10d7c3e5-be4d-4306-a59e-500b86bd141f/a4b43769-68f4-4111-a02f-817ae260783a/ea625b3a-a58b-4ce4-9f3d-01a79f8438bc"
-					(reference "#PWR0103")
+					(reference "#PWR0104")
 					(unit 1)
 				)
@@
 		(dnp no)
 		(fields_autoplaced yes)
-		(property "Reference" "#PWR0106"
+		(property "Reference" "#PWR0103"
 			(at 157.48 109.22 0)
 			(hide yes)
@@
 			(project "rcm_dish_controller"
 				(path "/10d7c3e5-be4d-4306-a59e-500b86bd141f/a4b43769-68f4-4111-a02f-817ae260783a/ea625b3a-a58b-4ce4-9f3d-01a79f8438bc"
-					(reference "#PWR0106")
+					(reference "#PWR0103")
 					(unit 1)
 				)
@@
 		(in_pos_files yes)
 		(dnp no)
-		(property "Reference" "H5"
+		(property "Reference" "H4"
 			(at 83.82 138.684 90)
 			(show_name no)
@@
 			(project "rcm_dish_controller"
 				(path "/10d7c3e5-be4d-4306-a59e-500b86bd141f/a4b43769-68f4-4111-a02f-817ae260783a/ea625b3a-a58b-4ce4-9f3d-01a79f8438bc"
-					(reference "H5")
+					(reference "H4")
 					(unit 1)
 				)
@@
 		(dnp no)
 		(fields_autoplaced yes)
-		(property "Reference" "#PWR057"
+		(property "Reference" "#PWR0102"
 			(at 96.52 107.95 0)
 			(hide yes)
@@
 			(project "rcm_dish_controller"
 				(path "/10d7c3e5-be4d-4306-a59e-500b86bd141f/a4b43769-68f4-4111-a02f-817ae260783a/ea625b3a-a58b-4ce4-9f3d-01a79f8438bc"
-					(reference "#PWR057")
+					(reference "#PWR0102")
 					(unit 1)
 				)
@@
 		(in_pos_files yes)
 		(dnp no)
-		(property "Reference" "U14"
+		(property "Reference" "U17"
 			(at 173.99 108.966 0)
 			(show_name no)
@@
 			(project "rcm_dish_controller"
 				(path "/10d7c3e5-be4d-4306-a59e-500b86bd141f/a4b43769-68f4-4111-a02f-817ae260783a/ea625b3a-a58b-4ce4-9f3d-01a79f8438bc"
-					(reference "U14")
+					(reference "U17")
 					(unit 1)
 				)
@@
 		(in_pos_files yes)
 		(dnp no)
-		(property "Reference" "J3"
+		(property "Reference" "J2"
 			(at 201.676 58.42 0)
 			(show_name no)
@@
 			(project "rcm_dish_controller"
 				(path "/10d7c3e5-be4d-4306-a59e-500b86bd141f/a4b43769-68f4-4111-a02f-817ae260783a/ea625b3a-a58b-4ce4-9f3d-01a79f8438bc"
-					(reference "J3")
+					(reference "J2")
 					(unit 1)
 				)
@@
 		(dnp no)
 		(fields_autoplaced yes)
-		(property "Reference" "#PWR061"
+		(property "Reference" "#PWR099"
 			(at 154.94 68.58 0)
 			(hide yes)
@@
 			(project "rcm_dish_controller"
 				(path "/10d7c3e5-be4d-4306-a59e-500b86bd141f/a4b43769-68f4-4111-a02f-817ae260783a/ea625b3a-a58b-4ce4-9f3d-01a79f8438bc"
-					(reference "#PWR061")
+					(reference "#PWR099")
 					(unit 1)
 				)
@@
 		(dnp no)
 		(fields_autoplaced yes)
-		(property "Reference" "#PWR074"
+		(property "Reference" "#PWR0100"
 			(at 191.77 72.39 0)
 			(hide yes)
@@
 			(project "rcm_dish_controller"
 				(path "/10d7c3e5-be4d-4306-a59e-500b86bd141f/a4b43769-68f4-4111-a02f-817ae260783a/ea625b3a-a58b-4ce4-9f3d-01a79f8438bc"
-					(reference "#PWR074")
+					(reference "#PWR0100")
 					(unit 1)
 				)
@@
 		(in_pos_files yes)
 		(dnp no)
-		(property "Reference" "H6"
+		(property "Reference" "H5"
 			(at 107.95 138.684 90)
 			(show_name no)
@@
 			(project "rcm_dish_controller"
 				(path "/10d7c3e5-be4d-4306-a59e-500b86bd141f/a4b43769-68f4-4111-a02f-817ae260783a/ea625b3a-a58b-4ce4-9f3d-01a79f8438bc"
-					(reference "H6")
+					(reference "H5")
 					(unit 1)
 				)
@@
 		(in_pos_files yes)
 		(dnp no)
-		(property "Reference" "H1"
+		(property "Reference" "H3"
 			(at 101.346 102.616 0)
 			(show_name no)
@@
 			(project "rcm_dish_controller"
 				(path "/10d7c3e5-be4d-4306-a59e-500b86bd141f/a4b43769-68f4-4111-a02f-817ae260783a/ea625b3a-a58b-4ce4-9f3d-01a79f8438bc"
-					(reference "H1")
+					(reference "H3")
 					(unit 1)
 				)
@@
 		(dnp no)
 		(fields_autoplaced yes)
-		(property "Reference" "R92"
+		(property "Reference" "R91"
 			(at 110.49 59.6899 0)
 			(show_name no)
@@
 			(project "rcm_dish_controller"
 				(path "/10d7c3e5-be4d-4306-a59e-500b86bd141f/a4b43769-68f4-4111-a02f-817ae260783a/ea625b3a-a58b-4ce4-9f3d-01a79f8438bc"
-					(reference "R92")
+					(reference "R91")
 					(unit 1)
 				)
@@
 		(dnp no)
 		(fields_autoplaced yes)
-		(property "Reference" "#PWR0104"
+		(property "Reference" "#PWR0101"
 			(at 73.66 74.93 0)
 			(hide yes)
@@
 			(project "rcm_dish_controller"
 				(path "/10d7c3e5-be4d-4306-a59e-500b86bd141f/a4b43769-68f4-4111-a02f-817ae260783a/ea625b3a-a58b-4ce4-9f3d-01a79f8438bc"
-					(reference "#PWR0104")
+					(reference "#PWR0101")
 					(unit 1)
 				)
@@
 		(dnp no)
 		(fields_autoplaced yes)
-		(property "Reference" "R91"
+		(property "Reference" "R92"
 			(at 93.98 133.3499 0)
 			(show_name no)
@@
 			(project "rcm_dish_controller"
 				(path "/10d7c3e5-be4d-4306-a59e-500b86bd141f/a4b43769-68f4-4111-a02f-817ae260783a/ea625b3a-a58b-4ce4-9f3d-01a79f8438bc"
-					(reference "R91")
+					(reference "R92")
 					(unit 1)
 				)

Commit message: CAN looks complete in schematic
Parts:
- removed LED4: LTST-S270KGKT, MyParts:LED-SMD_L1.7-W0.6-RD, symbol MyParts:LTST-S270KGKT
- added LED4: GREEN, MyParts:LED0805-R-RD, symbol MyParts:0805G
- renumbered H3 to J4
Connections:
- net 3V3_CM4: now also LED4.1 (A)
- net at R91.1: now also LED4.2 (K)
Changed lines of the file:
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@@
-	)
-	(symbol
-		(lib_id "MyParts:LTST-S270KGKT")
-		(at 107.95 50.8 270)
-		(mirror x)
-		(unit 1)
-		(body_style 1)
-		(exclude_from_sim no)
-		(in_bom yes)
-		(on_board yes)
-		(in_pos_files yes)
-		(dnp no)
-		(fields_autoplaced yes)
-		(property "Reference" "LED4"
-			(at 113.03 50.7999 90)
-			(show_name no)
-			(do_not_autoplace no)
-			(effects
-				(font
-					(size 1.27 1.27)
-				)
-				(justify left)
-			)
-		)
-		(property "Value" "LTST-S270KGKT"
-			(at 113.03 53.3399 90)
-			(show_name no)
-			(do_not_autoplace no)
-			(effects
-				(font
-					(size 1.27 1.27)
-				)
-				(justify left)
-			)
-		)
-		(property "Footprint" "MyParts:LED-SMD_L1.7-W0.6-RD"
-			(at 100.33 50.8 0)
-			(hide yes)
-			(show_name no)
-			(do_not_autoplace no)
-			(effects
-				(font
-					(size 1.27 1.27)
-				)
-			)
-		)
-		(property "Datasheet" "https://lcsc.com/product-detail/Light-Emitting-Diodes-LED_SMD-green_C125113.html"
-			(at 97.79 50.8 0)
-			(hide yes)
-			(show_name no)
-			(do_not_autoplace no)
-			(effects
-				(font
-					(size 1.27 1.27)
-				)
-			)
-		)
-		(property "Description" ""
-			(at 107.95 50.8 0)
-			(hide yes)
-			(show_name no)
-			(do_not_autoplace no)
-			(effects
-				(font
-					(size 1.27 1.27)
-				)
-			)
-		)
-		(property "LCSC Part" "C125113"
-			(at 95.25 50.8 0)
-			(hide yes)
-			(show_name no)
-			(do_not_autoplace no)
-			(effects
-				(font
-					(size 1.27 1.27)
-				)
-			)
-		)
-		(pin "2"
-		)
-		(pin "1"
-		)
-		(instances
-			(project "rcm_dish_controller"
-				(path "/10d7c3e5-be4d-4306-a59e-500b86bd141f/a4b43769-68f4-4111-a02f-817ae260783a/ea625b3a-a58b-4ce4-9f3d-01a79f8438bc"
-					(reference "LED4")
-					(unit 1)
-				)
-			)
-		)
 	)
 	(symbol
@@
 		(in_pos_files yes)
 		(dnp no)
-		(property "Reference" "H3"
+		(property "Reference" "J4"
 			(at 101.346 102.616 0)
 			(show_name no)
@@
 			(project "rcm_dish_controller"
 				(path "/10d7c3e5-be4d-4306-a59e-500b86bd141f/a4b43769-68f4-4111-a02f-817ae260783a/ea625b3a-a58b-4ce4-9f3d-01a79f8438bc"
-					(reference "H3")
+					(reference "J4")
 					(unit 1)
 				)
@@
 					(unit 1)
 				)
+			)
+		)
+	)
+	(symbol
+		(lib_id "MyParts:0805G")
+		(at 109.22 50.8 270)
+		(mirror x)
+		(unit 1)
+		(body_style 1)
+		(exclude_from_sim no)
+		(in_bom yes)
+		(on_board yes)
+		(in_pos_files yes)
+		(dnp no)
+		(property "Reference" "LED4"
+			(at 115.824 50.038 90)
+			(show_name no)
+			(do_not_autoplace no)
+			(effects
+				(font
+					(size 1.27 1.27)
+				)
+				(justify right)
+			)
+		)
+		(property "Value" "GREEN"
+			(at 117.348 52.07 90)
+			(show_name no)
+			(do_not_autoplace no)
+			(effects
+				(font
+					(size 1.27 1.27)
+				)
+				(justify right)
+			)
+		)
+		(property "Footprint" "MyParts:LED0805-R-RD"
+			(at 100.33 50.8 0)
+			(hide yes)
+			(show_name no)
+			(do_not_autoplace no)
+			(effects
+				(font
+					(size 1.27 1.27)
+				)
+			)
+		)
+		(property "Datasheet" "https://lcsc.com/product-detail/Light-Emitting-Diodes-LED_Green-0805-Highlighted_C2297.html"
+			(at 97.79 50.8 0)
+			(hide yes)
+			(show_name no)
+			(do_not_autoplace no)
+			(effects
+				(font
+					(size 1.27 1.27)
+				)
+			)
+		)
+		(property "Description" "0805"
+			(at 85.09 50.8 0)
+			(hide yes)
+			(show_name no)
+			(do_not_autoplace no)
+			(effects
+				(font
+					(size 1.27 1.27)
+				)
+			)
+		)
+		(property "Manufacturer" "KENTO"
+			(at 95.25 50.8 0)
+			(hide yes)
+			(show_name no)
+			(do_not_autoplace no)
+			(effects
+				(font
+					(size 1.27 1.27)
+				)
+			)
+		)
+		(property "MPN" "KT-0805G"
+			(at 92.71 50.8 0)
+			(hide yes)
+			(show_name no)
+			(do_not_autoplace no)
+			(effects
+				(font
+					(size 1.27 1.27)
+				)
+			)
+		)
+		(property "LCSC Part" "C2297"
+			(at 90.17 50.8 0)
+			(hide yes)
+			(show_name no)
+			(do_not_autoplace no)
+			(effects
+				(font
+					(size 1.27 1.27)
+				)
+			)
+		)
+		(pin "1"
+		)
+		(pin "2"
+		)
+		(instances
+			(project "rcm_dish_controller"
+				(path "/10d7c3e5-be4d-4306-a59e-500b86bd141f/a4b43769-68f4-4111-a02f-817ae260783a/ea625b3a-a58b-4ce4-9f3d-01a79f8438bc"
+					(reference "LED4")
+					(unit 1)
+				)

Commit message: Add CAN JR45 - still working on it
Parts:
- renumbered H4 to H3, H5 to H4, J4 to J3
Changed lines of the file:
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@@
 		(dnp no)
 		(fields_autoplaced yes)
-		(property "Reference" "#PWR0104"
+		(property "Reference" "#PWR0107"
 			(at 165.1 137.16 0)
 			(hide yes)
@@
 			(project "rcm_dish_controller"
 				(path "/10d7c3e5-be4d-4306-a59e-500b86bd141f/a4b43769-68f4-4111-a02f-817ae260783a/ea625b3a-a58b-4ce4-9f3d-01a79f8438bc"
-					(reference "#PWR0104")
+					(reference "#PWR0107")
 					(unit 1)
 				)
@@
 		(dnp no)
 		(fields_autoplaced yes)
-		(property "Reference" "#PWR0103"
+		(property "Reference" "#PWR0106"
 			(at 157.48 109.22 0)
 			(hide yes)
@@
 			(project "rcm_dish_controller"
 				(path "/10d7c3e5-be4d-4306-a59e-500b86bd141f/a4b43769-68f4-4111-a02f-817ae260783a/ea625b3a-a58b-4ce4-9f3d-01a79f8438bc"
-					(reference "#PWR0103")
+					(reference "#PWR0106")
 					(unit 1)
 				)
@@
 		(in_pos_files yes)
 		(dnp no)
-		(property "Reference" "H4"
+		(property "Reference" "H3"
 			(at 83.82 138.684 90)
 			(show_name no)
@@
 			(project "rcm_dish_controller"
 				(path "/10d7c3e5-be4d-4306-a59e-500b86bd141f/a4b43769-68f4-4111-a02f-817ae260783a/ea625b3a-a58b-4ce4-9f3d-01a79f8438bc"
-					(reference "H4")
+					(reference "H3")
 					(unit 1)
 				)
@@
 		(dnp no)
 		(fields_autoplaced yes)
-		(property "Reference" "#PWR0102"
+		(property "Reference" "#PWR0105"
 			(at 96.52 107.95 0)
 			(hide yes)
@@
 			(project "rcm_dish_controller"
 				(path "/10d7c3e5-be4d-4306-a59e-500b86bd141f/a4b43769-68f4-4111-a02f-817ae260783a/ea625b3a-a58b-4ce4-9f3d-01a79f8438bc"
-					(reference "#PWR0102")
+					(reference "#PWR0105")
 					(unit 1)
 				)
@@
 		(dnp no)
 		(fields_autoplaced yes)
-		(property "Reference" "#PWR099"
+		(property "Reference" "#PWR0102"
 			(at 154.94 68.58 0)
 			(hide yes)
@@
 			(project "rcm_dish_controller"
 				(path "/10d7c3e5-be4d-4306-a59e-500b86bd141f/a4b43769-68f4-4111-a02f-817ae260783a/ea625b3a-a58b-4ce4-9f3d-01a79f8438bc"
-					(reference "#PWR099")
+					(reference "#PWR0102")
 					(unit 1)
 				)
@@
 		(dnp no)
 		(fields_autoplaced yes)
-		(property "Reference" "#PWR0100"
+		(property "Reference" "#PWR0103"
 			(at 191.77 72.39 0)
 			(hide yes)
@@
 			(project "rcm_dish_controller"
 				(path "/10d7c3e5-be4d-4306-a59e-500b86bd141f/a4b43769-68f4-4111-a02f-817ae260783a/ea625b3a-a58b-4ce4-9f3d-01a79f8438bc"
-					(reference "#PWR0100")
+					(reference "#PWR0103")
 					(unit 1)
 				)
@@
 		(in_pos_files yes)
 		(dnp no)
-		(property "Reference" "H5"
+		(property "Reference" "H4"
 			(at 107.95 138.684 90)
 			(show_name no)
@@
 			(project "rcm_dish_controller"
 				(path "/10d7c3e5-be4d-4306-a59e-500b86bd141f/a4b43769-68f4-4111-a02f-817ae260783a/ea625b3a-a58b-4ce4-9f3d-01a79f8438bc"
-					(reference "H5")
+					(reference "H4")
 					(unit 1)
 				)
@@
 		(in_pos_files yes)
 		(dnp no)
-		(property "Reference" "J4"
+		(property "Reference" "J3"
 			(at 101.346 102.616 0)
 			(show_name no)
@@
 			(project "rcm_dish_controller"
 				(path "/10d7c3e5-be4d-4306-a59e-500b86bd141f/a4b43769-68f4-4111-a02f-817ae260783a/ea625b3a-a58b-4ce4-9f3d-01a79f8438bc"
-					(reference "J4")
+					(reference "J3")
 					(unit 1)
 				)
@@
 		(dnp no)
 		(fields_autoplaced yes)
-		(property "Reference" "#PWR0101"
+		(property "Reference" "#PWR0104"
 			(at 73.66 74.93 0)
 			(hide yes)
@@
 			(project "rcm_dish_controller"
 				(path "/10d7c3e5-be4d-4306-a59e-500b86bd141f/a4b43769-68f4-4111-a02f-817ae260783a/ea625b3a-a58b-4ce4-9f3d-01a79f8438bc"
-					(reference "#PWR0101")
+					(reference "#PWR0104")
 					(unit 1)
 				)

Commit message: Updates
Parts:
- renumbered U17 to J5
Changed lines of the file:
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@@
 		(in_pos_files yes)
 		(dnp no)
-		(property "Reference" "U17"
+		(property "Reference" "J5"
 			(at 173.99 108.966 0)
 			(show_name no)
@@
 			(project "rcm_dish_controller"
 				(path "/10d7c3e5-be4d-4306-a59e-500b86bd141f/a4b43769-68f4-4111-a02f-817ae260783a/ea625b3a-a58b-4ce4-9f3d-01a79f8438bc"
-					(reference "U17")
+					(reference "J5")
 					(unit 1)
 				)
