File: robo-dc-controller/kicad/cm4-robo-controller/cm4_connectors.kicad_sch (KiCad schematic)
At the start: 0 parts

Commit message: CM4 carrier: GPS sheet integration, U12 expansion header, power fixes
Populate U12 (2x12 expansion header) on the CM4_Connectors sheet:
all 19 CM4 signals plus 3V3_CM4 and four grounds, with 2.2k I2C
pull-ups (R113/R114) on GPIO2/GPIO3. Value matches the CM4IO
reference design, which uses 2.2k on SDA1/SCL1.

Wire the new GPS sheet (MAX-M10S) into the CM4 sheet: add sheet pins
for GPS_RX_MCU, GPS_TX_MCU and 1PPS_MCU. The UART lands on UART3
(GPIO4 = TXD3 to the GPS RXD, GPIO5 = RXD3 from the GPS TXD) and
1PPS on GPIO16. Needs dtoverlay=uart3 in config.txt. The leftover
CM4_TX/CM4_RX/1PPS_MCU hierarchical labels, which pointed at a root
sheet with no matching pins, become local labels on those nets.

Fix the orphaned 3V3 label on the GPS sheet, which left the MS621FE
backup cell with no charge path, and scope 3V3_CM4 to the CM4
hierarchy: local labels in the CM4 sheet, hierarchical labels plus
sheet pins in each consuming sub-sheet. Net membership is unchanged
at 30 nodes.

Add PWR_FLAGs on the 5V rail and on GND. Both are driven through
passive parts (an inductor and ground symbols respectively), so ERC
could not see a driver.

ERC: 55 -> 40 violations. Of the remainder, 30 are the RoboClaw U1,
which is placed on the root sheet but not yet wired.
Parts:
- added R113, R114: 2.2kΩ, PCM_JLCPCB:R_0402, symbol PCM_JLCPCB-Resistors:0402,2.2kΩ
- added U12: 2541WV-2X12P, MyParts:HDR-TH_24P-P2.54-V-M-R2-C12-S2.54, symbol MyParts:2541WV-2X12P
Connections:
- new net 3V3_CM4: R113.1, R114.1, U12.1
- new net AIN0: U12.19
- new net AIN1: U12.20
- new net BOOT_CONSOLE_RXD: U12.14
- new net BOOT_CONSOLE_TXD: U12.13
- new net EEPROM_nWP: U12.24
- new net GLOBAL_EN: U12.23
- new net GND: U12.11, U12.17, U12.2, U12.5
- new net GPIO22: U12.6
- new net I2C1_SCL: R114.2, U12.4
- new net I2C1_SDA: R113.2, U12.3
- new net PWM0: U12.15
- new net PWM1: U12.16
- new net RUN_PG: U12.21
- new net SPI0_CE0: U12.10
- new net SPI0_CE1: U12.12
- new net SPI0_MISO: U12.8
- new net SPI0_MOSI: U12.7
- new net SPI0_SCLK: U12.9
- new net nPWR_LED: U12.18
- new net nRPIBOOT: U12.22

Commit message: Updates
Parts:
- added H1: Header-Male-2.54_1x4, MyParts:HDR-TH_4P-P2.54-V-M, symbol MyParts:Header-Male-2.54_1x4
Changed lines of the file:
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@@
-		)
-	)
-	(hierarchical_label "3V3_CM4"
-		(shape input)
-		(at 130.81 118.11 90)
-		(effects
-			(font
-				(size 1.27 1.27)
-			)
-			(justify left)
-		)
-	)
-	(hierarchical_label "3V3_CM4"
-		(shape input)
-		(at 114.3 73.66 180)
-		(effects
-			(font
-				(size 1.27 1.27)
-			)
-			(justify right)
 		)
 	)
@@
 		)
 	)
+	(hierarchical_label "3V3_CM4"
+		(shape input)
+		(at 130.81 118.11 90)
+		(effects
+			(font
+				(size 1.27 1.27)
+			)
+			(justify left)
+		)
+	)
 	(hierarchical_label "RUN_PG"
 		(shape input)
@@
 		(shape output)
 		(at 114.3 96.52 180)
+		(effects
+			(font
+				(size 1.27 1.27)
+			)
+			(justify right)
+		)
+	)
+	(hierarchical_label "3V3_CM4"
+		(shape input)
+		(at 114.3 73.66 180)
 		(effects
 			(font
@@
 					(unit 1)
 				)
+			)
+		)
+	)
+	(symbol
+		(lib_id "MyParts:Header-Male-2.54_1x4")
+		(at 218.44 85.09 0)
+		(unit 1)
+		(body_style 1)
+		(exclude_from_sim no)
+		(in_bom yes)
+		(on_board yes)
+		(in_pos_files yes)
+		(dnp no)
+		(fields_autoplaced yes)
+		(property "Reference" "H1"
+			(at 224.79 83.8199 0)
+			(show_name no)
+			(do_not_autoplace no)
+			(effects
+				(font
+					(size 1.27 1.27)
+				)
+				(justify left)
+			)
+		)
+		(property "Value" "Header-Male-2.54_1x4"
+			(at 224.79 86.3599 0)
+			(show_name no)
+			(do_not_autoplace no)
+			(effects
+				(font
+					(size 1.27 1.27)
+				)
+				(justify left)
+			)
+		)
+		(property "Footprint" "MyParts:HDR-TH_4P-P2.54-V-M"
+			(at 218.44 96.52 0)
+			(hide yes)
+			(show_name no)
+			(do_not_autoplace no)
+			(effects
+				(font
+					(size 1.27 1.27)
+				)
+			)
+		)
+		(property "Datasheet" "https://www.lcsc.com/datasheet/C124378.pdf?spm=wm.sxq.inf.ggs___wm.ssy.bg.0.cbh&lcsc_vid=FFBaV1wHQFldUVICFgBfBVJTQVJWXgBfEQRYBAFQE1YxVlNRQFZaV1ZfRVdbVjsOAxUeFF5JWBYZEEoKFBINSQcJGk4eFQsCAgIaSgADAwAHC0slRlNaVFNQWQkaCgg%3D"
+			(at 218.44 99.06 0)
+			(hide yes)
+			(show_name no)
+			(do_not_autoplace no)
+			(effects
+				(font
+					(size 1.27 1.27)
+				)
+			)
+		)
+		(property "Description" "CONN HEADER 4POS 2.54mm SINGLE ROW TH"
+			(at 218.44 85.09 0)
+			(hide yes)
+			(show_name no)
+			(do_not_autoplace no)
+			(effects
+				(font
+					(size 1.27 1.27)
+				)
+			)
+		)
+		(property "Manufacturer" "Ckmtw(灿科盟)"
+			(at 218.44 101.6 0)
+			(hide yes)
+			(show_name no)
+			(do_not_autoplace no)
+			(effects
+				(font
+					(size 1.27 1.27)
+				)
+			)
+		)
+		(property "MPN" "B-2100S04P-A110"
+			(at 218.44 104.14 0)
+			(hide yes)
+			(show_name no)
+			(do_not_autoplace no)
+			(effects
+				(font
+					(size 1.27 1.27)
+				)
+			)
+		)
+		(property "LCSC Part" "C124378"
+			(at 218.44 106.68 0)
+			(hide yes)
+			(show_name no)
+			(do_not_autoplace no)
+			(effects
+				(font
+					(size 1.27 1.27)
+				)
+			)
+		)
+		(pin "4"
+		)
+		(pin "1"
+		)
+		(pin "3"
+		)
+		(pin "2"
+		)
+		(instances
+			(project "cm4-robo-controller"
+				(path "/c1285fbe-5f56-49a8-9041-410713cbe619/3cc0f123-2315-4414-aa85-3a1a0bb694eb/ea625b3a-a58b-4ce4-9f3d-01a79f8438bc"
+					(reference "H1")
+					(unit 1)
+				)
