File: robo-dc-controller/kicad/cm4-robo-controller/power_5v.kicad_sch (KiCad schematic)
At the start: 24 parts, among them U9 AP64501SP-13

Commit message: CM4 carrier: GPS sheet integration, U12 expansion header, power fixes
Populate U12 (2x12 expansion header) on the CM4_Connectors sheet:
all 19 CM4 signals plus 3V3_CM4 and four grounds, with 2.2k I2C
pull-ups (R113/R114) on GPIO2/GPIO3. Value matches the CM4IO
reference design, which uses 2.2k on SDA1/SCL1.

Wire the new GPS sheet (MAX-M10S) into the CM4 sheet: add sheet pins
for GPS_RX_MCU, GPS_TX_MCU and 1PPS_MCU. The UART lands on UART3
(GPIO4 = TXD3 to the GPS RXD, GPIO5 = RXD3 from the GPS TXD) and
1PPS on GPIO16. Needs dtoverlay=uart3 in config.txt. The leftover
CM4_TX/CM4_RX/1PPS_MCU hierarchical labels, which pointed at a root
sheet with no matching pins, become local labels on those nets.

Fix the orphaned 3V3 label on the GPS sheet, which left the MS621FE
backup cell with no charge path, and scope 3V3_CM4 to the CM4
hierarchy: local labels in the CM4 sheet, hierarchical labels plus
sheet pins in each consuming sub-sheet. Net membership is unchanged
at 30 nodes.

Add PWR_FLAGs on the 5V rail and on GND. Both are driven through
passive parts (an inductor and ground symbols respectively), so ERC
could not see a driver.

ERC: 55 -> 40 violations. Of the remainder, 30 are the RoboClaw U1,
which is placed on the root sheet but not yet wired.
Parts:
- removed R76: 12kΩ, MyParts:R0402, symbol PCM_JLCPCB-Resistors:0402,12kΩ
- added R76: 11.5kΩ, MyParts:R0402, symbol MyParts:FRC0402F1152TS
- TP8: value RH-5016 -> 5V
Connections:
- net 5V: now also R76.2
- net at C58.2, R78.1, U9.5 (FB): now also R76.1
Other:
- note added: "+5v @ 3A PSU ( 8.3v-28v Input )"
- note added: "12V to 5V Buck - AP64501 (5A, 570kHz, 0.8V reference) Vout = 4.98V, designed for 3A. Input 8.3V-28V (eFuse UVLO cuts in at 8.3V). EN tied to VIN: starts automatically, the eFuse upstream provides the UVLO. Output voltage set by the FB divider Vout = 0.8V x (1 + R76/R78) = 0.8 x (1 + 11.5k/2.2k) = 4.98V R76 11.5k 1% top leg, 5V to FB R78 2.2k 1% bottom leg, FB to GND C58 DNP optional feedforward a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"
- note removed: "+5v @ 3A PSU ( 7.5v-28v Input )"
